File: piparv2/piparv2.kicad_pcb (KiCad board)
At the start: 2 copper layers, 139.4 x 109.8 mm, 109 parts, among them M2 MountingHole_2.2mm_M2, SW1 SW_Wuerth_450301014042

Commit message: adds macropad
Parts:
- added BAT+1: BAT+, TestPoint:TestPoint_THTPad_D2.0mm_Drill1.0mm, F.Cu at (62.8, 130.8)
- added BAT-1: BAT-, TestPoint:TestPoint_THTPad_2.0x2.0mm_Drill1.0mm, F.Cu at (66.9, 130.8)
- added Brd1: SSD1306, SSD1306:128x64OLED_0.91, F.Cu at (63.5, 153.6)
- added CH19: KSwitch, keyswitches:Kailh_socket_PG1350_reversible, F.Cu at (82.8, 165.1)
- added CH20: KSwitch, keyswitches:Kailh_socket_PG1350_reversible, F.Cu at (100.8, 165.1)
- added CH21: KSwitch, keyswitches:Kailh_socket_PG1350_reversible, F.Cu at (118.7, 165.1)
- added CH22: KSwitch, keyswitches:Kailh_socket_PG1350_reversible, F.Cu at (82.8, 148.1)
- added CH23: KSwitch, keyswitches:Kailh_socket_PG1350_reversible, F.Cu at (100.8, 148.1)
- added CH24: KSwitch, keyswitches:Kailh_socket_PG1350_reversible, F.Cu at (118.7, 148.1)
- added CH25: KSwitch, keyswitches:Kailh_socket_PG1350_reversible, F.Cu at (100.8, 131.2)
- added CH26: KSwitch, keyswitches:Kailh_socket_PG1350_reversible, F.Cu at (118.7, 131.2)
- added CH27: RotaryEncoder_Switch, Rotary_Encoder:RotaryEncoder_Bourns_Vertical_PEL11L-4xxxF-Sxxxx_1, F.Cu at (82.6, 131.1)
- added D19: D, Diode_SMD:Nexperia_CFP3_SOD-123W, B.Cu at (78.1, 165.1)
- added D20: D, Diode_SMD:Nexperia_CFP3_SOD-123W, B.Cu at (96.1, 165.1)
- added D21: D, Diode_SMD:Nexperia_CFP3_SOD-123W, B.Cu at (114.0, 165.1)
- added D22: D, Diode_SMD:Nexperia_CFP3_SOD-123W, B.Cu at (78.1, 148.2)
- added D23: D, Diode_SMD:Nexperia_CFP3_SOD-123W, B.Cu at (96.0, 148.1)
- added D24: D, Diode_SMD:Nexperia_CFP3_SOD-123W, B.Cu at (114.1, 148.1)
- added D25: D, Diode_SMD:Nexperia_CFP3_SOD-123W, B.Cu at (96.2, 131.2)
- added D26: D, Diode_SMD:Nexperia_CFP3_SOD-123W, B.Cu at (114.1, 131.2)
- added M2: MountingHole_2.2mm_M2, MountingHole:MountingHole_2.2mm_M2, F.Cu at (66.9, 125.5)
- added M2: MountingHole_2.2mm_M2, MountingHole:MountingHole_2.2mm_M2, F.Cu at (109.7, 173.4)
- added SW2: SW_Wuerth_450301014042, Button_Switch_SMD:SW_SPDT_PCM12, B.Cu at (56.3, 127.6)
- added U2: nice_nano, nice-nano-kicad:nice_nano, F.Cu at (63.4, 155.4)
- moved TP2 115.3 mm to (102.5, 105.9)
- moved D15 115.3 mm to (115.5, 67.1)
- moved D15 115.3 mm to (97.6, 65.5)
- moved D7 115.3 mm to (71.7, 29.8)
- moved CH18 115.3 mm to (122.3, 85.6)
- moved CH7 115.3 mm to (62.9, 31.8)
- moved CH2 115.3 mm to (41.2, 103.4)
- moved D10 115.3 mm to (76.9, 25.1)
- moved SW1 115.3 mm to (143.5, 42.6)
- moved ? 115.3 mm to (109.1, 116.5)
- moved ? 115.3 mm to (107.5, 102.3)
- moved CH17 115.3 mm to (129.8, 69.5)
- moved D2 115.3 mm to (44.7, 111.8)
- moved CH1 115.3 mm to (25.8, 112.3)
- moved ? 115.3 mm to (116.8, 99.5)
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Routing:
- net GND: track 32.9 -> 119.0 mm, vias 2 -> 4
- net Net-(U2-P0.22): track 0.00 -> 85.5 mm, vias 0 -> 2
- net Net-(D21-K): track 0.00 -> 84.6 mm, vias 0 -> 2
- net Net-(U2-P0.17): track 0.00 -> 83.4 mm, vias 0 -> 3
- net Net-(U2-P0.20): track 0.00 -> 81.9 mm, vias 0 -> 3
- net Net-(D20-K): track 0.00 -> 64.3 mm
- net Net-(U2-AIN5/P0.29): track 0.00 -> 50.3 mm, vias 0 -> 2
- net Net-(U2-AIN7/P0.31): track 0.00 -> 50.0 mm
- net Net-(SW2-B): track 0.00 -> 43.5 mm, vias 0 -> 1
- net Net-(U2-RX1/P0.08): track 0.00 -> 40.2 mm, vias 0 -> 3
- net Net-(D21-A): track 0.00 -> 32.8 mm, vias 0 -> 1
- net Net-(D23-A): track 0.00 -> 32.2 mm, vias 0 -> 1
- net Net-(D22-A): track 0.00 -> 32.2 mm, vias 0 -> 1
- net Net-(D19-A): track 0.00 -> 32.2 mm, vias 0 -> 1
- net Net-(D25-A): track 0.00 -> 32.2 mm, vias 0 -> 1
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Other:
- board size 139.4 x 109.8 mm -> 139.4 x 159.1 mm
