File: pcb/pipar.kicad_pcb (KiCad board)
At the start: 2 copper layers, 139.4 x 158.3 mm, 133 parts, among them M2 MountingHole_2.2mm_M2, SW1 SW_Wuerth_450301014042, SW2 SW_Wuerth_450301014042, U2 nice_nano

Commit message: slightly improved PCB design
Parts:
- renumbered BAT+1 to BAT+, BAT-1 to BAT-
Routing:
- net Net-(D19-K): track 23.5 -> 22.9 mm
- net Net-(SW1-B): vias 6 -> 5
Other:
- outline, holes or cut-outs redrawn
- board text added: "Components visible"

Commit message: updates the pcb for flake
Parts:
- moved M2 16.2 mm to (108.2, 156.9)
- moved D21 2.42 mm to (111.9, 165.9)
- moved CH21 2.42 mm to (116.6, 165.8)
- moved D26 2.17 mm to (112.0, 130.1)
- moved CH26 2.17 mm to (116.6, 130.1)
- moved D24 2.10 mm to (112.0, 148.0)
- moved CH24 2.10 mm to (116.6, 148.0)
- moved CH20 1.61 mm to (99.7, 165.8)
- moved D20 1.61 mm to (95.0, 165.8)
- moved CH19 1.22 mm to (82.8, 165.8)
- moved D19 1.22 mm to (78.1, 165.9)
- moved D25 1.21 mm to (95.1, 130.1)
- moved CH25 1.21 mm to (99.7, 130.1)
- moved CH23 1.10 mm to (99.7, 148.0)
- moved D23 1.10 mm to (95.0, 148.0)
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Routing:
- net Net-(U2-P1.15): track 117.2 -> 127.6 mm, vias 6 -> 3
- net Net-(U2-P1.13): track 99.2 -> 106.6 mm, vias 4 -> 5
- net Net-(D21-K): track 84.9 -> 78.1 mm, vias 1 -> 4
- net Net-(U2-P1.11): track 89.5 -> 95.3 mm
- net Net-(U2-AIN7/P0.31): track 59.5 -> 63.8 mm, vias 1 -> 0
- net Net-(D24-A): track 28.6 -> 31.4 mm
- net Net-(D20-A): track 28.7 -> 31.5 mm
- net Net-(D25-A): track 28.7 -> 31.4 mm
- net Net-(D26-A): track 28.7 -> 31.5 mm
- net Net-(Brd1-SCL): track 23.7 -> 25.7 mm
- net Net-(D22-A): track 30.1 -> 32.1 mm
- net Net-(D20-K): track 61.6 -> 63.5 mm, vias 1 -> 2
- net Net-(U2-AIN5/P0.29): track 61.7 -> 60.1 mm, vias 1 -> 0
- net Net-(D21-A): track 30.1 -> 31.5 mm
- net Net-(D23-A): track 30.2 -> 31.5 mm
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