File: pcb/pipar_point/pipar_point.kicad_sch (KiCad schematic)
At the start: 92 parts, among them Q1 AO3416 N-channel MOSFET, SW1 SW_Wuerth_450301014042, SW2 CK_KMS2xxG, U1 Seeeduino Xiao nRF52840, U2 74HC595

Commit message: starts work on t460s board
Other:
- added sheet T460S Trackpoint schematic (t460s_trackpoint.kicad_sch)
Changed lines of the file:
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@@
+		)
+	)
+	(sheet
+		(at 134.62 93.98)
+		(size 52.07 43.18)
+		(fields_autoplaced yes)
+		(stroke
+			(width 0.1524)
+			(type solid)
+		)
+		(fill
+			(color 0 0 0 0.0000)
+		)
+		(property "Sheetname" "T460S Trackpoint schematic"
+			(at 134.62 93.2684 0)
+			(effects
+				(font
+					(size 1.27 1.27)
+				)
+				(justify left bottom)
+			)
+		)
+		(property "Sheetfile" "t460s_trackpoint.kicad_sch"
+			(at 134.62 137.7446 0)
+			(effects
+				(font
+					(size 1.27 1.27)
+				)
+				(justify left top)
+			)
+		)
+		(instances
+			(project "pipar_point"
+				(path "/a3c92014-e327-4265-9fa8-d88c7e42ce9f"
+					(page "2")
+				)
+			)
 		)
 	)

Commit message: starts work on t460s board 2
Parts:
- added C3: 0.1uF, Capacitor_SMD:C_0805_2012Metric_Pad1.18x1.45mm_HandSolder, symbol Device:C_Small
Connections:
- net +3V3: now also C3.1
- net GND: now also C3.2
Changed lines of the file:
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@@
 	)
 	(junction
+		(at 101.6 99.06)
+		(diameter 0)
+		(color 0 0 0 0)
+	)
+	(junction
 		(at 43.18 43.18)
 		(diameter 0)
@@
 	(wire
 		(pts
+			(xy 116.84 99.06) (xy 113.03 99.06)
+		)
+		(stroke
+			(width 0)
+			(type default)
+		)
+	)
+	(wire
+		(pts
 			(xy 104.14 33.02) (xy 104.14 53.34)
 		)
@@
 	(wire
 		(pts
+			(xy 101.6 97.79) (xy 101.6 99.06)
+		)
+		(stroke
+			(width 0)
+			(type default)
+		)
+	)
+	(wire
+		(pts
 			(xy 162.56 66.04) (xy 162.56 60.96)
 		)
@@
 	(wire
 		(pts
+			(xy 107.95 99.06) (xy 101.6 99.06)
+		)
+		(stroke
+			(width 0)
+			(type default)
+		)
+	)
+	(wire
+		(pts
 			(xy 162.56 45.72) (xy 162.56 40.64)
 		)
@@
 	(symbol
 		(lib_id "power:+3V3")
-		(at 101.6 99.06 0)
+		(at 101.6 97.79 0)
 		(unit 1)
 		(exclude_from_sim no)
@@
 		(dnp no)
 		(property "Reference" "#PWR011"
-			(at 101.6 102.87 0)
+			(at 101.6 101.6 0)
 			(effects
 				(font
@@
 		)
 		(property "Value" "+3V3"
-			(at 105.156 99.06 0)
+			(at 105.156 97.79 0)
 			(effects
 				(font
@@
 		)
 		(property "Footprint" ""
-			(at 101.6 99.06 0)
+			(at 101.6 97.79 0)
 			(effects
 				(font
@@
 		)
 		(property "Datasheet" ""
-			(at 101.6 99.06 0)
+			(at 101.6 97.79 0)
 			(effects
 				(font
@@
 		)
 		(property "Description" "Power symbol creates a global label with name \"+3V3\""
-			(at 101.6 99.06 0)
+			(at 101.6 97.79 0)
 			(effects
 				(font
@@
 	)
 	(symbol
+		(lib_id "Device:C_Small")
+		(at 110.49 99.06 90)
+		(unit 1)
+		(exclude_from_sim no)
+		(in_bom yes)
+		(on_board yes)
+		(dnp no)
+		(property "Reference" "C3"
+			(at 110.49 96.774 90)
+			(effects
+				(font
+					(size 1.27 1.27)
+				)
+			)
+		)
+		(property "Value" "0.1uF"
+			(at 110.4963 95.25 90)
+			(effects
+				(font
+					(size 1.27 1.27)
+				)
+			)
+		)
+		(property "Footprint" "Capacitor_SMD:C_0805_2012Metric_Pad1.18x1.45mm_HandSolder"
+			(at 110.49 99.06 0)
+			(effects
+				(font
+					(size 1.27 1.27)
+				)
+				(hide yes)
+			)
+		)
+		(property "Datasheet" "~"
+			(at 110.49 99.06 0)
+			(effects
+				(font
+					(size 1.27 1.27)
+				)
+				(hide yes)
+			)
+		)
+		(property "Description" "Unpolarized capacitor, small symbol"
+			(at 110.49 99.06 0)
+			(effects
+				(font
+					(size 1.27 1.27)
+				)
+				(hide yes)
+			)
+		)
+		(pin "2"
+		)
+		(pin "1"
+		)
+		(instances
+			(project ""
+				(path "/a3c92014-e327-4265-9fa8-d88c7e42ce9f"
+					(reference "C3")
+					(unit 1)
+				)
+			)
+		)
+	)
+	(symbol
 		(lib_id "Device:D")
 		(at 93.98 39.37 90)
@@
 					(unit 1)
 				)
+			)
+		)
+	)
+	(symbol
+		(lib_id "PCM_4ms_Power-symbol:GND")
+		(at 116.84 99.06 0)
+		(unit 1)
+		(exclude_from_sim no)
+		(in_bom yes)
+		(on_board yes)
+		(dnp no)
+		(fields_autoplaced yes)
+		(property "Reference" "#PWR021"
+			(at 116.84 105.41 0)
+			(effects
+				(font
+					(size 1.27 1.27)
+				)
+				(hide yes)
+			)
+		)
+		(property "Value" "GND"
+			(at 116.84 104.14 0)
+			(effects
+				(font
+					(size 1.27 1.27)
+				)
+			)
+		)
+		(property "Footprint" ""
+			(at 116.84 99.06 0)
+			(effects
+				(font
+					(size 1.27 1.27)
+				)
+				(hide yes)
+			)
+		)
+		(property "Datasheet" ""
+			(at 116.84 99.06 0)
+			(effects
+				(font
+					(size 1.27 1.27)
+				)
+				(hide yes)
+			)
+		)
+		(property "Description" ""
+			(at 116.84 99.06 0)
+			(effects
+				(font
+					(size 1.27 1.27)
+				)
+				(hide yes)
+			)
+		)
+		(pin "1"
+		)
+		(instances
+			(project ""
+				(path "/a3c92014-e327-4265-9fa8-d88c7e42ce9f"
+					(reference "#PWR021")
+					(unit 1)
+				)

Commit message: start work on pipar point again
Parts:
- removed C3: 0.1uF, Capacitor_SMD:C_0805_2012Metric_Pad1.18x1.45mm_HandSolder, symbol Device:C_Small
- removed CH1, CH10, CH11, CH12, CH13, CH14, CH15, CH16, CH17, CH18, CH2, CH3, CH4, CH5, CH6, CH7, CH8, CH9: KSwitch, choc:SW_Hotswap_Kailh_Choc_V1V2_Reverse_LED_1.00u, symbol marbastlib-choc:choc_v1_SW_HS_CPG135001S30
- removed D1, D10, D11, D12, D13, D14, D15, D16, D17, D18, D2, D3, D4, D5, D6, D7, D8, D9: D, Diode_SMD:D_SOD-323_HandSoldering, symbol Device:D
- removed LED1, LED10, LED11, LED12, LED13, LED14, LED15, LED16, LED17, LED18, LED2, LED3, LED4, LED5, LED6, LED7, LED8, LED9: ~, LED_SMD:LED_0805_2012Metric, symbol LED:IR26-21C_L110_TR8
- removed Q1: AO3416 N-channel MOSFET, Package_TO_SOT_SMD:SOT-23, symbol Device:Q_NMOS_GSD
- removed R1, R10, R11, R12, R13, R14, R15, R16, R17, R18, R2, R3, R4, R5, R6, R7, R8, R9: 100, Resistor_SMD:R_0805_2012Metric, symbol Device:R
- removed R19: 4.7k, Resistor_SMD:R_0805_2012Metric, symbol PCM_4ms_Resistor:10m_1206_250mW
- removed SW1: SW_Wuerth_450301014042, Button_Switch_SMD:SW_SPDT_PCM12, symbol Switch:SW_Wuerth_450301014042
- removed SW2: CK_KMS2xxG, Button_Switch_SMD:SW_SPST_CK_KMS2xxGP, symbol Switch:CK_KMS2xxG
- removed T460s1: ~, Reversible-KB:Trackpoint_T460s_Board_no_flip, symbol Trackpoint:T460s
- removed TP1: BAT-, TestPoint:TestPoint_THTPad_2.0x2.0mm_Drill1.0mm, symbol Connector:TestPoint
- removed TP2: BAT+, TestPoint:TestPoint_THTPad_D2.0mm_Drill1.0mm, symbol Connector:TestPoint
- removed U1: Seeeduino Xiao nRF52840, Seeed Studio XIAO Series Library:XIAO-nRF52840-Sense-14P-2.54-21X17.8MM, symbol marbastlib-promicroish:Seeeduino_Xiao_nRF52840
- removed U10, U11, U12, U13, U4, U6, U8, U9: ~, choc:Solder Nut, symbol Trackpoint:Solder_Nut
- removed U2: 74HC595, 74HC595PW:SOP65P640X110-16N, symbol 74xx:74HC595
- removed U3: ~, choc:Trackpoint_Connector, symbol Trackpoint:Connector
- removed U5: ~, choc:Trackpoint_T460s_Stick, symbol Trackpoint:Sensor
- removed U7: ~, Art:Salt, symbol Trackpoint:Solder_Nut
Connections:
- no-connect marks 11 -> 0
Other:
- removed sheet T460S Trackpoint schematic
- added sheet Trackpointer (T460s.kicad_sch)

Commit message: more pipar poimt progress
Other:
- added sheet Keymatrix (keymatrix.kicad_sch)
- added sheet Keymatrix_left (keymatrix.kicad_sch)
- added sheet nRF52840 (nRF52840.kicad_sch)
- added sheet nRF52840_left (nRF52840.kicad_sch)
- sheet Trackpointer ports: added none; removed GND
- note added: "Left half"
- note added: "Right half"

Commit message: pipar point panelized
Parts:
- added AE1: Antenna, Mikoto:2.4GHz-meander-antenna-v2-right, symbol Device:Antenna
- added AE2: Antenna, Mikoto:2.4GHz-meander-antenna-v2, symbol Device:Antenna
- added FID50, FID51, FID52, FID53: Fiducial, Fiducial:Fiducial_0.5mm_Mask1.5mm, symbol Mechanical:Fiducial
- added H50, H51, H52, H53, H54, H55, H56, H57, H58, H59: MouseBite, mouse-bite:mouse-bite-5mm-10mm, symbol Mechanical:MountingHole
- added H62, H63, H74, H75, H76, H77: MountingHole, MountingHole:MountingHole_2.1mm, symbol Mechanical:MountingHole
Connections:
- new net nRF52840/Ant: AE1.1 (A)
- new net nRF52840_left/Ant: AE2.1 (A)
Other:
- sheet nRF52840 ports: added Ant; removed none
- sheet nRF52840_left ports: added Ant; removed none

Commit message: finish macropad
Parts:
- added FID54, FID55, FID56, FID57: Fiducial, Fiducial:Fiducial_0.5mm_Mask1.5mm, symbol Mechanical:Fiducial
- added H112, H113, H114, H115, H116, H66, H67, H68, H69, H70: MountingHole, MountingHole:MountingHole_2.2mm_M2_DIN965, symbol Mechanical:MountingHole
- added H118, H119, H120, H121: MountingHole, Keyboard:SMTSO_M2_C4_2+C2.7_1.5, symbol Mechanical:MountingHole
- renumbered AE2 to AE50, AE1 to AE52, H54 to H52, H56 to H53, H58 to H54, H52 to H55, H53 to H56, H55 to H57, H57 to H58, H62 to H60, H63 to H61, H74 to H62, H75 to H63, H76 to H64, H77 to H65
Other:
- added sheet Keymatrix_Macropad (keymatrix_macropad.kicad_sch)
- added sheet nRF52840_XIAO_Macropad (nrf52840_xiao.kicad_sch)
- moved on the sheet: AE50, AE52

Commit message: pipar point v1, prototype
Parts:
- AE50: footprint Mikoto:2.4GHz-meander-antenna-v2 -> Mikoto:2.4GHz-meander-antenna-v2-right
Changed lines of the file:
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@@
+	)
+	(symbol
+		(lib_id "Mechanical:MountingHole")
+		(at 215.9 36.83 0)
+		(unit 1)
+		(exclude_from_sim yes)
+		(in_bom no)
+		(on_board yes)
+		(dnp no)
+		(fields_autoplaced yes)
+		(property "Reference" "H69"
+			(at 218.44 35.5599 0)
+			(effects
+				(font
+					(size 1.27 1.27)
+				)
+				(justify left)
+			)
+		)
+		(property "Value" "MountingHole"
+			(at 218.44 38.0999 0)
+			(effects
+				(font
+					(size 1.27 1.27)
+				)
+				(justify left)
+			)
+		)
+		(property "Footprint" "MountingHole:MountingHole_2.2mm_M2_DIN965"
+			(at 215.9 36.83 0)
+			(effects
+				(font
+					(size 1.27 1.27)
+				)
+				(hide yes)
+			)
+		)
+		(property "Datasheet" "~"
+			(at 215.9 36.83 0)
+			(effects
+				(font
+					(size 1.27 1.27)
+				)
+				(hide yes)
+			)
+		)
+		(property "Description" "Mounting Hole without connection"
+			(at 215.9 36.83 0)
+			(effects
+				(font
+					(size 1.27 1.27)
+				)
+				(hide yes)
+			)
+		)
+		(instances
+			(project "pipar_point"
+				(path "/33180bf6-a8cb-4957-933e-07c9e2251da8"
+					(reference "H69")
+					(unit 1)
+				)
+			)
+		)
+	)
+	(symbol
+		(lib_id "Mechanical:MountingHole")
+		(at 22.86 44.45 0)
+		(unit 1)
+		(exclude_from_sim yes)
+		(in_bom no)
+		(on_board yes)
+		(dnp no)
+		(fields_autoplaced yes)
+		(property "Reference" "H116"
+			(at 25.4 43.1799 0)
+			(effects
+				(font
+					(size 1.27 1.27)
+				)
+				(justify left)
+			)
+		)
+		(property "Value" "MountingHole"
+			(at 25.4 45.7199 0)
+			(effects
+				(font
+					(size 1.27 1.27)
+				)
+				(justify left)
+			)
+		)
+		(property "Footprint" "MountingHole:MountingHole_2.2mm_M2_DIN965"
+			(at 22.86 44.45 0)
+			(effects
+				(font
+					(size 1.27 1.27)
+				)
+				(hide yes)
+			)
+		)
+		(property "Datasheet" "~"
+			(at 22.86 44.45 0)
+			(effects
+				(font
+					(size 1.27 1.27)
+				)
+				(hide yes)
+			)
+		)
+		(property "Description" "Mounting Hole without connection"
+			(at 22.86 44.45 0)
+			(effects
+				(font
+					(size 1.27 1.27)
+				)
+				(hide yes)
+			)
+		)
+		(instances
+			(project "pipar_point"
+				(path "/33180bf6-a8cb-4957-933e-07c9e2251da8"
+					(reference "H116")
+					(unit 1)
+				)
+			)
+		)
+	)
+	(symbol
+		(lib_id "Mechanical:Fiducial")
+		(at 106.68 142.24 0)
+		(unit 1)
+		(exclude_from_sim yes)
+		(in_bom no)
+		(on_board yes)
+		(dnp no)
+		(fields_autoplaced yes)
+		(property "Reference" "FID51"
+			(at 109.22 140.9699 0)
+			(effects
+				(font
+					(size 1.27 1.27)
+				)
+				(justify left)
+			)
+		)
+		(property "Value" "Fiducial"
+			(at 109.22 143.5099 0)
+			(effects
+				(font
+					(size 1.27 1.27)
+				)
+				(justify left)
+			)
+		)
+		(property "Footprint" "Fiducial:Fiducial_0.5mm_Mask1.5mm"
+			(at 106.68 142.24 0)
+			(effects
+				(font
+					(size 1.27 1.27)
+				)
+				(hide yes)
+			)
+		)
+		(property "Datasheet" "~"
+			(at 106.68 142.24 0)
+			(effects
+				(font
+					(size 1.27 1.27)
+				)
+				(hide yes)
+			)
+		)
+		(property "Description" "Fiducial Marker"
+			(at 106.68 142.24 0)
+			(effects
+				(font
+					(size 1.27 1.27)
+				)
+				(hide yes)
+			)
+		)
+		(instances
+			(project "pipar_point"
+				(path "/33180bf6-a8cb-4957-933e-07c9e2251da8"
+					(reference "FID51")
+					(unit 1)
+				)
+			)
+		)
 	)
 	(symbol
@@
 			)
 		)
-		(property "Footprint" "Mikoto:2.4GHz-meander-antenna-v2"
+		(property "Footprint" "Mikoto:2.4GHz-meander-antenna-v2-right"
 			(at 73.66 46.99 0)
 			(effects
@@
 					(unit 1)
 				)
-			)
-		)
-	)
-	(symbol
-		(lib_id "Mechanical:MountingHole")
-		(at 215.9 36.83 0)
-		(unit 1)
-		(exclude_from_sim yes)
-		(in_bom no)
-		(on_board yes)
-		(dnp no)
-		(fields_autoplaced yes)
-		(property "Reference" "H69"
-			(at 218.44 35.5599 0)
-			(effects
-				(font
-					(size 1.27 1.27)
-				)
-				(justify left)
-			)
-		)
-		(property "Value" "MountingHole"
-			(at 218.44 38.0999 0)
-			(effects
-				(font
-					(size 1.27 1.27)
-				)
-				(justify left)
-			)
-		)
-		(property "Footprint" "MountingHole:MountingHole_2.2mm_M2_DIN965"
-			(at 215.9 36.83 0)
-			(effects
-				(font
-					(size 1.27 1.27)
-				)
-				(hide yes)
-			)
-		)
-		(property "Datasheet" "~"
-			(at 215.9 36.83 0)
-			(effects
-				(font
-					(size 1.27 1.27)
-				)
-				(hide yes)
-			)
-		)
-		(property "Description" "Mounting Hole without connection"
-			(at 215.9 36.83 0)
-			(effects
-				(font
-					(size 1.27 1.27)
-				)
-				(hide yes)
-			)
-		)
-		(instances
-			(project "pipar_point"
-				(path "/33180bf6-a8cb-4957-933e-07c9e2251da8"
-					(reference "H69")
-					(unit 1)
-				)
-			)
-		)
-	)
-	(symbol
-		(lib_id "Mechanical:MountingHole")
-		(at 22.86 44.45 0)
-		(unit 1)
-		(exclude_from_sim yes)
-		(in_bom no)
-		(on_board yes)
-		(dnp no)
-		(fields_autoplaced yes)
-		(property "Reference" "H116"
-			(at 25.4 43.1799 0)
-			(effects
-				(font
-					(size 1.27 1.27)
-				)
-				(justify left)
-			)
-		)
-		(property "Value" "MountingHole"
-			(at 25.4 45.7199 0)
-			(effects
-				(font
-					(size 1.27 1.27)
-				)
-				(justify left)
-			)
-		)
-		(property "Footprint" "MountingHole:MountingHole_2.2mm_M2_DIN965"
-			(at 22.86 44.45 0)
-			(effects
-				(font
-					(size 1.27 1.27)
-				)
-				(hide yes)
-			)
-		)
-		(property "Datasheet" "~"
-			(at 22.86 44.45 0)
-			(effects
-				(font
-					(size 1.27 1.27)
-				)
-				(hide yes)
-			)
-		)
-		(property "Description" "Mounting Hole without connection"
-			(at 22.86 44.45 0)
-			(effects
-				(font
-					(size 1.27 1.27)
-				)
-				(hide yes)
-			)
-		)
-		(instances
-			(project "pipar_point"
-				(path "/33180bf6-a8cb-4957-933e-07c9e2251da8"
-					(reference "H116")
-					(unit 1)
-				)
-			)
-		)
-	)
-	(symbol
-		(lib_id "Mechanical:Fiducial")
-		(at 106.68 142.24 0)
-		(unit 1)
-		(exclude_from_sim yes)
-		(in_bom no)
-		(on_board yes)
-		(dnp no)
-		(fields_autoplaced yes)
-		(property "Reference" "FID51"
-			(at 109.22 140.9699 0)
-			(effects
-				(font
-					(size 1.27 1.27)
-				)
-				(justify left)
-			)
-		)
-		(property "Value" "Fiducial"
-			(at 109.22 143.5099 0)
-			(effects
-				(font
-					(size 1.27 1.27)
-				)
-				(justify left)
-			)
-		)
-		(property "Footprint" "Fiducial:Fiducial_0.5mm_Mask1.5mm"
-			(at 106.68 142.24 0)
-			(effects
-				(font
-					(size 1.27 1.27)
-				)
-				(hide yes)
-			)
-		)
-		(property "Datasheet" "~"
-			(at 106.68 142.24 0)
-			(effects
-				(font
-					(size 1.27 1.27)
-				)
-				(hide yes)
-			)
-		)
-		(property "Description" "Fiducial Marker"
-			(at 106.68 142.24 0)
-			(effects
-				(font
-					(size 1.27 1.27)
-				)
-				(hide yes)
-			)
-		)
-		(instances
-			(project "pipar_point"
-				(path "/33180bf6-a8cb-4957-933e-07c9e2251da8"
-					(reference "FID51")
-					(unit 1)
-				)
