File: pcb/pipar_point/pipar_point.kicad_pcb (KiCad board)
At the start: 2 copper layers, 145.3 x 110.3 mm, 116 parts, among them Q1 AO3416 N-channel MOSFET, SW1 SW_Wuerth_450301014042, SW2 CK_KMS2xxG, U1 Seeeduino Xiao nRF52840, U2 74HC595

Commit message: moves the through hole away from pad
Parts:
- moved U4 0.17 mm to (200.7, 50.2)
- moved U5 0.17 mm to (197.4, 59.1)
- moved U6 0.17 mm to (194.2, 68.1)
Changed lines of the file:
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@@
 	(footprint "choc:Solder Nut"
 		(layer "F.Cu")
-		(at 200.763496 50.356872 5)
+		(at 200.669999 50.210003 5)
 		(property "Reference" "U4"
 			(at 0 -0.5 5)
@@
 	(footprint "choc:Trackpoint_T460s_Stick"
 		(layer "F.Cu")
-		(at 197.514306 59.283949 -20)
+		(at 197.420809 59.13708 -20)
 		(property "Reference" "U5"
 			(at 0 12.7 -20)
@@
 	(footprint "choc:Solder Nut"
 		(layer "F.Cu")
-		(at 194.265111 68.211063 5)
+		(at 194.171614 68.064194 5)
 		(property "Reference" "U6"
 			(at 0 -0.5 5)

Commit message: starts work on t460s board
Parts:
- moved D7 1.93 mm to (130.5, 42.8)
- moved R7 1.93 mm to (130.5, 42.8)
- moved CH11 1.93 mm to (162.2, 56.5)
- moved CH10 1.93 mm to (162.2, 39.2)
- moved LED11 1.93 mm to (162.2, 51.9) (x2)
- moved D17 1.93 mm to (197.6, 78.5)
- moved LED9 1.93 mm to (142.1, 71.6) (x2)
- moved D1 1.93 mm to (92.1, 132.0)
- moved R1 1.93 mm to (92.1, 132.0)
- moved CH5 1.93 mm to (122.1, 63.8)
- moved R18 1.93 mm to (190.3, 94.1)
- moved SW2 1.93 mm to (215.5, 52.7) (x2)
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Routing:
- net ROW0: track 333.0 -> 331.2 mm
- net LEDOut: track 494.0 -> 492.3 mm
