File: pcb/pipar_point/pipar_point.kicad_pcb (KiCad board)
At the start: 2 copper layers, 145.3 x 110.3 mm, 116 parts, among them Q1 AO3416 N-channel MOSFET, SW1 SW_Wuerth_450301014042, SW2 CK_KMS2xxG, U1 Seeeduino Xiao nRF52840, U2 74HC595

Commit message: starts work on t460s board 2
Parts:
- added C3: 0.1uF, Capacitor_SMD:C_0805_2012Metric_Pad1.18x1.45mm_HandSolder, F.Cu at (173.4, 100.2)
- added C3: 0.1uF, Capacitor_SMD:C_0805_2012Metric_Pad1.18x1.45mm_HandSolder, B.Cu at (148.9, 100.0)
- moved U12 16.6 mm to (124.8, 84.0)
- moved U8 10.0 mm to (177.3, 28.8)
- moved U10 10.0 mm to (124.8, 116.3)
- moved U11 9.98 mm to (180.7, 116.3)
- moved U9 9.93 mm to (153.4, 25.6)
- moved D4 9.87 mm to (114.7, 38.2)
- moved R4 9.87 mm to (114.7, 38.2)
- moved LED12 9.87 mm to (165.4, 59.7) (x2)
- moved LED2 9.87 mm to (114.8, 103.0) (x2)
- moved D16 9.87 mm to (210.3, 48.9)
- moved R16 9.87 mm to (210.3, 48.9)
- moved LED1 9.87 mm to (99.8, 113.5) (x2)
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Connections:
- net +3V8 renamed Net-(SW1-A)
- net GND renamed Earth
Routing:
- net LEDOut: track 492.3 -> 497.2 mm
- net COL0: track 112.3 -> 115.0 mm
- net Earth: track 241.2 -> 243.3 mm
- net COL5: track 121.4 -> 122.7 mm
- net COL1: track 130.5 -> 131.7 mm
- net ROW1: track 291.7 -> 292.9 mm
- net ROW2: track 244.3 -> 245.2 mm
- net COL2: track 135.7 -> 136.6 mm
- net ROW0: track 331.2 -> 332.2 mm
- net COL4: track 126.7 -> 127.4 mm
- net +3V3: track 664.4 -> 664.9 mm
- added copper zone on B.Cu, net Earth
- added copper zone on F.Cu, net Earth

Commit message: adds lights
Parts:
- removed the U1 at (195.7, 109.1) (x2)
- added U1: Seeeduino Xiao nRF52840, Seeed Studio XIAO Series Library:XIAO-nRF52840-Sense-14P-2.54-21X17.8MM, F.Cu at (196.5, 109.8)
- added U1: Seeeduino Xiao nRF52840, Seeed Studio XIAO Series Library:XIAO-nRF52840-Sense-14P-2.54-21X17.8MM, B.Cu at (196.5, 109.8)
- moved CH15 1.81 mm to (183.7, 70.8)
- moved LED9 1.81 mm to (143.4, 62.6)
- moved LED2 1.81 mm to (113.1, 103.4) (x2)
- moved D5 1.81 mm to (114.5, 55.9)
- moved R5 1.81 mm to (114.5, 55.9)
- moved D8 1.81 mm to (133.2, 51.0)
- moved R8 1.81 mm to (133.2, 51.0)
- moved LED11 1.81 mm to (163.5, 42.9) (x2)
- moved LED10 1.81 mm to (163.5, 25.6) (x2)
- moved D10 1.81 mm to (154.4, 30.4)
- moved R10 1.81 mm to (154.4, 30.4)
- moved R19 1.81 mm to (183.9, 96.9)
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Routing:
- net LEDOut: track 497.2 -> 493.5 mm
- net Earth: track 243.3 -> 239.7 mm, vias 13 -> 15
- net ROW2: track 245.2 -> 248.7 mm
- net +3V3: track 664.9 -> 668.4 mm
- net ROW1: track 292.9 -> 295.8 mm
- net ROW0: track 332.2 -> 334.8 mm
- net MOSI: track 79.8 -> 82.5 mm
- net LEDTrig: track 25.9 -> 28.5 mm
- net  SCK: track 68.6 -> 71.2 mm
- net MISO: track 72.1 -> 74.8 mm
- net TPData: track 38.8 -> 40.0 mm
- net TPCLK: track 31.1 -> 32.3 mm
- net TPRST: track 35.5 -> 36.7 mm
- net BAT+: track 99.9 -> 100.5 mm
- net Net-(U1-RST): track 81.8 -> 81.7 mm, vias 7 -> 8
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Other:
- board size 145.3 x 110.3 mm -> 144.6 x 110.3 mm
