File: pcb/pipar_point/nrf52840_xiao.kicad_sch (KiCad schematic)
At the start: 10 parts, among them Q52 AO3416 N-channel MOSFET, SW54 Reset, SW55 SW_SPST, U64 Seeeduino Xiao nRF52840

Commit message: pipar point v1, prototype
Parts:
- U64: footprint Keyboard:XIAO-nRF52840-Sense-14P-2.54-21X17.8MM -> Keyboard:XIAO-nRF52840-Sense-14P-2.54-21X17.8MM-noNFC
Connections:
- no-connect marks 0 -> 2
Changed lines of the file:
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@@
 		(color 0 0 0 0)
+	)
+	(no_connect
+		(at 124.46 97.79)
+	)
+	(no_connect
+		(at 121.92 97.79)
 	)
 	(polyline
@@
 			)
 		)
-		(property "Footprint" "Keyboard:XIAO-nRF52840-Sense-14P-2.54-21X17.8MM"
+		(property "Footprint" "Keyboard:XIAO-nRF52840-Sense-14P-2.54-21X17.8MM-noNFC"
 			(at 116.84 114.3 0)
 			(effects
