File: pcb/pipar_point/keymatrix.kicad_sch (KiCad schematic)
At the start: 100 parts

Commit message: finish macropad
Parts:
- renumbered D90 to D54, D91 to D55, D92 to D56, D93 to D57, D94 to D58, D95 to D59, D96 to D60, D97 to D61, D98 to D62, D99 to D63, D100 to D64, D101 to D65, D102 to D66, D103 to D67, D104 to D68, D105 to D69, D106 to D70, D107 to D71, D108 to D72, D109 to D73, H90 to H72, H91 to H73, H92 to H74, H93 to H75, H94 to H76, H95 to H77, H96 to H78, H97 to H79, H98 to H80, H99 to H81, H100 to H82, H101 to H83, H102 to H84, H103 to H85, H104 to H86, H105 to H87, H106 to H88, H107 to H89, H108 to H90, H109 to H91, KHS90 to KHS50, KHS91 to KHS51, KHS92 to KHS52, KHS93 to KHS53, KHS94 to KHS54, KHS95 to KHS55, KHS96 to KHS56, KHS97 to KHS57, KHS98 to KHS58, KHS99 to KHS59, KHS100 to KHS60, KHS101 to KHS61, KHS102 to KHS62, KHS103 to KHS63, KHS104 to KHS64, KHS105 to KHS65, KHS106 to KHS66, KHS107 to KHS67, KHS108 to KHS68, KHS109 to KHS69, LED90 to LED50, LED91 to LED51, LED92 to LED52, LED93 to LED53, LED94 to LED54, LED95 to LED55, LED96 to LED56, LED97 to LED57, LED98 to LED58, LED99 to LED59, LED100 to LED60, LED101 to LED61, LED102 to LED62, LED103 to LED63, LED104 to LED64, LED105 to LED65, LED106 to LED66, LED107 to LED67, LED108 to LED68, LED109 to LED69, LR90 to LR50, LR91 to LR51, LR92 to LR52, LR93 to LR53, LR94 to LR54, LR95 to LR55, LR96 to LR56, LR97 to LR57, LR98 to LR58, LR99 to LR59, LR100 to LR60, LR101 to LR61, LR102 to LR62, LR103 to LR63, LR104 to LR64, LR105 to LR65, LR106 to LR66, LR107 to LR67, LR108 to LR68, LR109 to LR69

Commit message: Fixes diode footprint to be sod-523, removes text
Parts:
- D54, D55, D56, D57, D58, D59, D60, D61, D62, D63, D64, D65, D66, D67, D68, D69, D70, D71, D72, D73: footprint Diode_SMD:D_0402_1005Metric -> Diode_SMD:D_SOD-523
Changed lines of the file:
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@@
 			)
 		)
-		(property "Footprint" "Diode_SMD:D_0402_1005Metric"
+		(property "Footprint" "Diode_SMD:D_SOD-523"
 			(at 118.11 73.66 90)
 			(effects
@@
 			)
 		)
-		(property "Footprint" "Diode_SMD:D_0402_1005Metric"
+		(property "Footprint" "Diode_SMD:D_SOD-523"
 			(at 118.11 119.38 90)
 			(effects
@@
 			)
 		)
-		(property "Footprint" "Diode_SMD:D_0402_1005Metric"
+		(property "Footprint" "Diode_SMD:D_SOD-523"
 			(at 118.11 96.52 90)
 			(effects
@@
 			)
 		)
-		(property "Footprint" "Diode_SMD:D_0402_1005Metric"
+		(property "Footprint" "Diode_SMD:D_SOD-523"
 			(at 163.83 119.38 90)
 			(effects
@@
 			)
 		)
-		(property "Footprint" "Diode_SMD:D_0402_1005Metric"
+		(property "Footprint" "Diode_SMD:D_SOD-523"
 			(at 163.83 73.66 90)
 			(effects
@@
 			)
 		)
-		(property "Footprint" "Diode_SMD:D_0402_1005Metric"
+		(property "Footprint" "Diode_SMD:D_SOD-523"
 			(at 209.55 96.52 90)
 			(effects
@@
 			)
 		)
-		(property "Footprint" "Diode_SMD:D_0402_1005Metric"
+		(property "Footprint" "Diode_SMD:D_SOD-523"
 			(at 72.39 96.52 90)
 			(effects
@@
 			)
 		)
-		(property "Footprint" "Diode_SMD:D_0402_1005Metric"
+		(property "Footprint" "Diode_SMD:D_SOD-523"
 			(at 163.83 96.52 90)
 			(effects
@@
 			)
 		)
-		(property "Footprint" "Diode_SMD:D_0402_1005Metric"
+		(property "Footprint" "Diode_SMD:D_SOD-523"
 			(at 186.69 73.66 90)
 			(effects
@@
 			)
 		)
-		(property "Footprint" "Diode_SMD:D_0402_1005Metric"
+		(property "Footprint" "Diode_SMD:D_SOD-523"
 			(at 140.97 96.52 90)
 			(effects
@@
 			)
 		)
-		(property "Footprint" "Diode_SMD:D_0402_1005Metric"
+		(property "Footprint" "Diode_SMD:D_SOD-523"
 			(at 140.97 119.38 90)
 			(effects
@@
 			)
 		)
-		(property "Footprint" "Diode_SMD:D_0402_1005Metric"
+		(property "Footprint" "Diode_SMD:D_SOD-523"
 			(at 209.55 119.38 90)
 			(effects
@@
 			)
 		)
-		(property "Footprint" "Diode_SMD:D_0402_1005Metric"
+		(property "Footprint" "Diode_SMD:D_SOD-523"
 			(at 95.25 119.38 90)
 			(effects
@@
 			)
 		)
-		(property "Footprint" "Diode_SMD:D_0402_1005Metric"
+		(property "Footprint" "Diode_SMD:D_SOD-523"
 			(at 95.25 96.52 90)
 			(effects
@@
 			)
 		)
-		(property "Footprint" "Diode_SMD:D_0402_1005Metric"
+		(property "Footprint" "Diode_SMD:D_SOD-523"
 			(at 95.25 73.66 90)
 			(effects
@@
 			)
 		)
-		(property "Footprint" "Diode_SMD:D_0402_1005Metric"
+		(property "Footprint" "Diode_SMD:D_SOD-523"
 			(at 72.39 73.66 90)
 			(effects
@@
 			)
 		)
-		(property "Footprint" "Diode_SMD:D_0402_1005Metric"
+		(property "Footprint" "Diode_SMD:D_SOD-523"
 			(at 72.39 119.38 90)
 			(effects
@@
 			)
 		)
-		(property "Footprint" "Diode_SMD:D_0402_1005Metric"
+		(property "Footprint" "Diode_SMD:D_SOD-523"
 			(at 140.97 73.66 90)
 			(effects
@@
 			)
 		)
-		(property "Footprint" "Diode_SMD:D_0402_1005Metric"
+		(property "Footprint" "Diode_SMD:D_SOD-523"
 			(at 186.69 119.38 90)
 			(effects
@@
 			)
 		)
-		(property "Footprint" "Diode_SMD:D_0402_1005Metric"
+		(property "Footprint" "Diode_SMD:D_SOD-523"
 			(at 186.69 96.52 90)
 			(effects

Commit message: start fixing footprints
Parts:
- LED50, LED51, LED52, LED53, LED54, LED55, LED56, LED57, LED58, LED59, LED60, LED61, LED62, LED63, LED64, LED65, LED66, LED67, LED68, LED69: footprint LED_SMD:LED_0402_1005Metric -> LED_SMD:LED_0603_1608Metric
Changed lines of the file:
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@@
 			)
 		)
-		(property "Footprint" "LED_SMD:LED_0402_1005Metric"
+		(property "Footprint" "LED_SMD:LED_0603_1608Metric"
 			(at 199.39 91.44 90)
 			(effects
@@
 			)
 		)
-		(property "Footprint" "LED_SMD:LED_0402_1005Metric"
+		(property "Footprint" "LED_SMD:LED_0603_1608Metric"
 			(at 153.67 91.44 90)
 			(effects
@@
 			)
 		)
-		(property "Footprint" "LED_SMD:LED_0402_1005Metric"
+		(property "Footprint" "LED_SMD:LED_0603_1608Metric"
 			(at 62.23 91.44 90)
 			(effects
@@
 			)
 		)
-		(property "Footprint" "LED_SMD:LED_0402_1005Metric"
+		(property "Footprint" "LED_SMD:LED_0603_1608Metric"
 			(at 107.95 91.44 90)
 			(effects
@@
 			)
 		)
-		(property "Footprint" "LED_SMD:LED_0402_1005Metric"
+		(property "Footprint" "LED_SMD:LED_0603_1608Metric"
 			(at 176.53 68.58 90)
 			(effects
@@
 			)
 		)
-		(property "Footprint" "LED_SMD:LED_0402_1005Metric"
+		(property "Footprint" "LED_SMD:LED_0603_1608Metric"
 			(at 62.23 68.58 90)
 			(effects
@@
 			)
 		)
-		(property "Footprint" "LED_SMD:LED_0402_1005Metric"
+		(property "Footprint" "LED_SMD:LED_0603_1608Metric"
 			(at 107.95 114.3 90)
 			(effects
@@
 			)
 		)
-		(property "Footprint" "LED_SMD:LED_0402_1005Metric"
+		(property "Footprint" "LED_SMD:LED_0603_1608Metric"
 			(at 85.09 91.44 90)
 			(effects
@@
 			)
 		)
-		(property "Footprint" "LED_SMD:LED_0402_1005Metric"
+		(property "Footprint" "LED_SMD:LED_0603_1608Metric"
 			(at 130.81 114.3 90)
 			(effects
@@
 			)
 		)
-		(property "Footprint" "LED_SMD:LED_0402_1005Metric"
+		(property "Footprint" "LED_SMD:LED_0603_1608Metric"
 			(at 130.81 68.58 90)
 			(effects
@@
 			)
 		)
-		(property "Footprint" "LED_SMD:LED_0402_1005Metric"
+		(property "Footprint" "LED_SMD:LED_0603_1608Metric"
 			(at 176.53 91.44 90)
 			(effects
@@
 			)
 		)
-		(property "Footprint" "LED_SMD:LED_0402_1005Metric"
+		(property "Footprint" "LED_SMD:LED_0603_1608Metric"
 			(at 153.67 68.58 90)
 			(effects
@@
 			)
 		)
-		(property "Footprint" "LED_SMD:LED_0402_1005Metric"
+		(property "Footprint" "LED_SMD:LED_0603_1608Metric"
 			(at 62.23 114.3 90)
 			(effects
@@
 			)
 		)
-		(property "Footprint" "LED_SMD:LED_0402_1005Metric"
+		(property "Footprint" "LED_SMD:LED_0603_1608Metric"
 			(at 107.95 68.58 90)
 			(effects
@@
 			)
 		)
-		(property "Footprint" "LED_SMD:LED_0402_1005Metric"
+		(property "Footprint" "LED_SMD:LED_0603_1608Metric"
 			(at 130.81 91.44 90)
 			(effects
@@
 			)
 		)
-		(property "Footprint" "LED_SMD:LED_0402_1005Metric"
+		(property "Footprint" "LED_SMD:LED_0603_1608Metric"
 			(at 85.09 68.58 90)
 			(effects
@@
 			)
 		)
-		(property "Footprint" "LED_SMD:LED_0402_1005Metric"
+		(property "Footprint" "LED_SMD:LED_0603_1608Metric"
 			(at 176.53 114.3 90)
 			(effects
@@
 			)
 		)
-		(property "Footprint" "LED_SMD:LED_0402_1005Metric"
+		(property "Footprint" "LED_SMD:LED_0603_1608Metric"
 			(at 199.39 114.3 90)
 			(effects
@@
 			)
 		)
-		(property "Footprint" "LED_SMD:LED_0402_1005Metric"
+		(property "Footprint" "LED_SMD:LED_0603_1608Metric"
 			(at 85.09 114.3 90)
 			(effects
@@
 			)
 		)
-		(property "Footprint" "LED_SMD:LED_0402_1005Metric"
+		(property "Footprint" "LED_SMD:LED_0603_1608Metric"
 			(at 153.67 114.3 90)
 			(effects
