File: pcb/pipar_point/nRF52840.kicad_sch (KiCad schematic)
At the start: 75 parts, among them J53 Conn_02x04_Odd_Even, P1 USB-C, Q1 AO3416 N-channel MOSFET, SW1 Reset, U1 BQ21040DBVR, U11 BQ24075RGT, U2 nRF52840, U3 ESDR0502NMUTAG, U7 XC6220B331MR, U9 MAX17048, Y1 32.768 kHz, Y2 32MHz

Commit message: more progress on pipar point
Parts:
- removed C67: 1uF, footprints:Capacitor_0402_1005M-nosilk, symbol Device:C_Small
- removed C68, C69: 4.7uF, footprints:Capacitor_0402_1005M-nosilk, symbol Device:C_Small
- removed D7: PMEG4010CEJ, footprints:D_SOD-323F-nosilk, symbol Device:D_Schottky_Small
- removed D8: ORANGE, footprints:LED_0402_1005Metric-nosilk, symbol Device:LED_Small
- removed F1: 500mA hold, footprints:Fuse_0402_1005Metric, symbol Device:Polyfuse_Small
- removed R25, R27, R28: 10k, footprints:Resistor_0402_1005M-nosilk, symbol Device:R_Small
- removed R26: 3.9k, footprints:Resistor_0402_1005M-nosilk, symbol Device:R_Small
- removed U11: BQ24075RGT, footprints:VQFN-16-1EP_3x3mm_P0.5mm_EP1.6x1.6mm, symbol Battery_Management:BQ24075RGT
Connections:
- net WirelessCharging: now reaches C15.1, D2.1 (K), U1.6 (VIN)
- no-connect marks 26 -> 23
Other:
- note added: "40mA"
- note removed: "Z, Z: 0mA (off) 0, Z: 100mA Z, 0: 250mA 0, 0: 350mA"
- moved on the sheet: D2, SW1, TP5, TP6

Commit message: update pipar point traces and add more connection pads
Parts:
- removed C14, C15: 1uF, Capacitor_SMD:C_0402_1005Metric, symbol Device:C_Small
- removed D1: CHG, LED_SMD:LED_0603_1608Metric, symbol Device:LED_Small
- removed D2: B5819W SL, Diode_SMD:D_SOD-323, symbol Device:D_Schottky_Small
- removed R2, R4: 10k, Resistor_SMD:R_0402_1005Metric, symbol Device:R_Small
- removed R3: 2.7k, Resistor_SMD:R_0603_1608Metric, symbol Device:R_Small
- removed U1: BQ21040DBVR, Mikoto:SOT95P280X145-6N, symbol bq21040:BQ21040DBVR
- added C67, C69: 4.7uF, Capacitor_SMD:C_0402_1005Metric, symbol Device:C_Small
- added D7: B5819WT, Diode_SMD:D_SOD-523, symbol Device:D_Schottky_Small
- added D9: CHG, LED_SMD:LED_0402_1005Metric, symbol Device:LED_Small
- added R25: 10k, Resistor_SMD:R_0402_1005Metric, symbol Device:R_Small
- added R27: 470, Resistor_SMD:R_0402_1005Metric, symbol Device:R_Small
- added TP11: W_GND, TestPoint:TestPoint_Pad_2.5x2.5mm, symbol Connector:TestPoint
- added TP9: W_VBUS, TestPoint:TestPoint_Pad_2.5x2.5mm, symbol Connector:TestPoint
- added U53: MCP73831-2-MC, Package_DFN_QFN:DFN-8-1EP_3x2mm_P0.5mm_EP1.7x1.4mm, symbol Battery_Management:MCP73831-2-MC
- D22: value BLUE -> CAPS; footprint LED_SMD:LED_0603_1608Metric -> LED_SMD:LED_0402_1005Metric
- D3: footprint LED_SMD:LED_0603_1608Metric -> LED_SMD:LED_0402_1005Metric
Connections:
- net GND: now also C67.2, C69.2, R25.2, TP11.1, U53.6 (V_{SS})
- net VBAT: now also C69.1, U53.3 (V_{BAT}), U53.4 (V_{BAT})
- net VBUS: now also D7.2 (A)
- new net: D9.1 (K), R27.1
- new net: R27.2, U53.5 (STAT)
- new net: R25.1, U53.8 (PROG)
- new net W_VBUS: C67.1, D7.1 (K), D9.2 (A), TP9.1, U53.1 (V_{DD}), U53.2 (V_{DD})
Other:
- note added: "VBAT: 1000/10kR = 100mA"
- note removed: "40mA"
- note removed: "ISET: 540/2700 = 200mA"

Commit message: one side is done
Connections:
- net VBUS: no longer C1.2, J53.2 (Pin_2), U2.AD2 (VBUS)
- net W_VBUS: now also C1.2, J53.2 (Pin_2), U2.AD2 (VBUS)
Changed lines of the file:
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@@
+		)
+	)
+	(label "W_VBUS"
+		(at 156.21 39.37 180)
+		(effects
+			(font
+				(size 1.27 1.27)
+			)
+			(justify right bottom)
 		)
 	)
@@
 		)
 	)
+	(label "W_VBUS"
+		(at 91.44 203.2 0)
+		(effects
+			(font
+				(size 1.27 1.27)
+			)
+			(justify left bottom)
+		)
+	)
 	(label "VBUS"
 		(at 292.1 160.02 0)
@@
 		)
 	)
-	(label "VBUS"
-		(at 156.21 39.37 90)
-		(effects
-			(font
-				(size 1.27 1.27)
-			)
-			(justify left bottom)
-		)
-	)
 	(label "VBAT"
 		(at 321.31 130.81 0)
@@
 		)
 	)
-	(label "VBUS"
-		(at 91.44 203.2 0)
-		(effects
-			(font
-				(size 1.27 1.27)
-			)
-			(justify left bottom)
-		)
-	)

Commit message: pipar point panelized
Parts:
- removed AE1: Antenna, Mikoto:2.4GHz-meander-antenna-v2, symbol Device:Antenna
- added H60: Logo, Art:Salt-smallest, symbol Mechanical:MountingHole
- added H64, H66, H68, H70, H72: MountingHole, MountingHole:MountingHole_2.2mm_M2_DIN965, symbol Mechanical:MountingHole
- added SW50: SW_SPST, Button_Switch_SMD:SW_SPDT_PCM12, symbol Switch:SW_SPST
Connections:
- net VBAT: now also SW50.1 (A); no longer TP5.1
- net ANT renamed Ant
- new net: SW50.2 (B), TP5.1
Other:
- moved on the sheet: TP5, TP6

Commit message: finish macropad
Parts:
- removed H64, H66, H68, H70, H72: MountingHole, MountingHole:MountingHole_2.2mm_M2_DIN965, symbol Mechanical:MountingHole
- renumbered C10 to C62, C11 to C63, C21 to C64, C22 to C65, C12 to C66, C7 to C67, C6 to C68, C5 to C69, C4 to C70, C1 to C71, C2 to C72, C3 to C73, C8 to C74, C9 to C75, C13 to C76, C16 to C77, C65 to C78, C23 to C79, C17 to C80, C18 to C81, C19 to C82, C20 to C83, C24 to C84, C67 to C85, C69 to C86, C49 to C87, C62 to C88, D3 to D50, D22 to D51, D7 to D52, D9 to D53, H60 to H71, J53 to J51, L4 to L50, L1 to L51, L2 to L52, L3 to L53, NT1 to NT50, P1 to P50, Q1 to Q50, R1 to R66, R8 to R67, R9 to R68, R10 to R69, R5 to R70, R31 to R71, R11 to R72, R39 to R73, R25 to R74, R27 to R75, R6 to R76, R7 to R77, R23 to R78, SW1 to SW51, TP5 to TP50, TP6 to TP51, TP9 to TP52, TP11 to TP53, U2 to U54, U9 to U55, U53 to U56, U3 to U57, U7 to U58, Y2 to Y51, Y1 to Y52

Commit message: pipar point v1, prototype
Parts:
- P50: footprint Connector_USB:USB_C_Receptacle_HRO_TYPE-C-31-M-12 -> Keyboard:USB_C_Receptacle_HRO_TYPE-C-31-M-16
Changed lines of the file:
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@@
 			)
 		)
-		(property "Footprint" "Connector_USB:USB_C_Receptacle_HRO_TYPE-C-31-M-12"
+		(property "Footprint" "Keyboard:USB_C_Receptacle_HRO_TYPE-C-31-M-16"
 			(at 274.32 175.26 0)
 			(effects

Commit message: start fixing footprints
Parts:
- D50, D51, D53: footprint LED_SMD:LED_0402_1005Metric -> LED_SMD:LED_0603_1608Metric
Changed lines of the file:
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@@
 			)
 		)
-		(property "Footprint" "LED_SMD:LED_0402_1005Metric"
+		(property "Footprint" "LED_SMD:LED_0603_1608Metric"
 			(at 223.52 160.02 90)
 			(effects
@@
 			)
 		)
-		(property "Footprint" "LED_SMD:LED_0402_1005Metric"
+		(property "Footprint" "LED_SMD:LED_0603_1608Metric"
 			(at 304.8 116.84 90)
 			(effects
@@
 			)
 		)
-		(property "Footprint" "LED_SMD:LED_0402_1005Metric"
+		(property "Footprint" "LED_SMD:LED_0603_1608Metric"
 			(at 223.52 151.13 90)
 			(effects

Commit message: fix esd routing
Connections:
- net USB_D-: now also U57.4 (D-); no longer U57.6 (VBUS)
- net VBUS: now also U57.6 (VBUS); no longer U57.4 (D-)
Changed lines of the file:
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@@
-		)
-	)
-	(label "USB_D-"
-		(at 289.56 200.66 180)
-		(effects
-			(font
-				(size 1.27 1.27)
-			)
-			(justify right bottom)
 		)
 	)
@@
 		)
 	)
-	(label "VBUS"
-		(at 289.56 198.12 180)
-		(effects
-			(font
-				(size 1.27 1.27)
-			)
-			(justify right bottom)
-		)
-	)
 	(label "VDDH"
 		(at 327.66 161.29 180)
@@
 		)
 	)
+	(label "USB_D-"
+		(at 289.56 198.12 180)
+		(effects
+			(font
+				(size 1.27 1.27)
+			)
+			(justify right bottom)
+		)
+	)
 	(label "CAPS_LED"
 		(at 186.69 135.89 0)
@@
 		)
 	)
+	(label "VBUS"
+		(at 289.56 200.66 180)
+		(effects
+			(font
+				(size 1.27 1.27)
+			)
+			(justify right bottom)
+		)
+	)
