File: pcb/pipar_point/pipar_point_trackpoint/pipar_point_trackpoint.kicad_sch (KiCad schematic)
At the start: 32 parts, among them J1 Conn_02x04, Y1 Crystal_GND2_Small

Commit message: working on trackpoint
Connections:
- net GND: now also R6.1, R7.2
- net at C1.1, C2.2, C3.1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: now also U1.28 (P3.3)
- net at U1.15 (DEC): no longer U1.24 (INT0/P1.0)
- net at U1.18 (XYS): no longer U1.21 (P1.2)
Changed lines of the file:
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@@
 	(paper "A4")
+	(junction
+		(at 148.59 82.55)
+		(diameter 0)
+		(color 0 0 0 0)
+	)
+	(junction
+		(at 219.71 35.56)
+		(diameter 0)
+		(color 0 0 0 0)
+	)
 	(junction
 		(at 237.49 41.91)
@@
 	(wire
 		(pts
+			(xy 121.92 104.14) (xy 119.38 104.14)
+		)
+		(stroke
+			(width 0)
+			(type default)
+		)
+	)
+	(wire
+		(pts
 			(xy 153.67 88.9) (xy 153.67 93.98)
 		)
@@
 	(wire
 		(pts
-			(xy 109.22 104.14) (xy 109.22 114.3)
+			(xy 219.71 33.02) (xy 219.71 35.56)
 		)
 		(stroke
@@
 	(wire
 		(pts
+			(xy 267.97 29.21) (xy 267.97 62.23)
+		)
+		(stroke
+			(width 0)
+			(type default)
+		)
+	)
+	(wire
+		(pts
 			(xy 231.14 40.64) (xy 231.14 35.56)
 		)
@@
 	(wire
 		(pts
-			(xy 93.98 107.95) (xy 101.6 107.95)
-		)
-		(stroke
-			(width 0)
-			(type default)
-		)
-	)
-	(wire
-		(pts
 			(xy 231.14 73.66) (xy 231.14 78.74)
 		)
@@
 	(wire
 		(pts
-			(xy 86.36 104.14) (xy 86.36 114.3)
-		)
-		(stroke
-			(width 0)
-			(type default)
-		)
-	)
-	(wire
-		(pts
 			(xy 266.7 81.28) (xy 266.7 33.02)
 		)
@@
 	(wire
 		(pts
+			(xy 273.05 29.21) (xy 267.97 29.21)
+		)
+		(stroke
+			(width 0)
+			(type default)
+		)
+	)
+	(wire
+		(pts
 			(xy 205.74 48.26) (xy 205.74 41.91)
 		)
@@
 	(wire
 		(pts
-			(xy 93.98 104.14) (xy 93.98 107.95)
-		)
-		(stroke
-			(width 0)
-			(type default)
-		)
-	)
-	(wire
-		(pts
 			(xy 231.14 88.9) (xy 231.14 78.74)
 		)
@@
 	(wire
 		(pts
-			(xy 101.6 107.95) (xy 101.6 104.14)
-		)
-		(stroke
-			(width 0)
-			(type default)
-		)
-	)
-	(wire
-		(pts
 			(xy 205.74 35.56) (xy 205.74 40.64)
 		)
@@
 	(wire
 		(pts
-			(xy 86.36 114.3) (xy 109.22 114.3)
-		)
-		(stroke
-			(width 0)
-			(type default)
-		)
-	)
-	(wire
-		(pts
 			(xy 215.9 71.12) (xy 210.82 71.12)
 		)
@@
 	(wire
 		(pts
+			(xy 121.92 82.55) (xy 148.59 82.55)
+		)
+		(stroke
+			(width 0)
+			(type default)
+		)
+	)
+	(wire
+		(pts
 			(xy 203.2 90.17) (xy 203.2 114.3)
 		)
@@
 		(pts
 			(xy 205.74 41.91) (xy 200.66 41.91)
+		)
+		(stroke
+			(width 0)
+			(type default)
+		)
+	)
+	(wire
+		(pts
+			(xy 267.97 62.23) (xy 116.84 62.23)
+		)
+		(stroke
+			(width 0)
+			(type default)
+		)
+	)
+	(wire
+		(pts
+			(xy 121.92 82.55) (xy 121.92 104.14)
 		)
 		(stroke
@@
 					(unit 1)
 				)
+			)
+		)
+	)
+	(symbol
+		(lib_id "power:GND")
+		(at 219.71 33.02 180)
+		(unit 1)
+		(exclude_from_sim no)
+		(in_bom yes)
+		(on_board yes)
+		(dnp no)
+		(fields_autoplaced yes)
+		(property "Reference" "#PWR02"
+			(at 219.71 26.67 0)
+			(effects
+				(font
+					(size 1.27 1.27)
+				)
+				(hide yes)
+			)
+		)
+		(property "Value" "GND"
+			(at 219.71 27.94 0)
+			(effects
+				(font
+					(size 1.27 1.27)
+				)
+			)
+		)
+		(property "Footprint" ""
+			(at 219.71 33.02 0)
+			(effects
+				(font
+					(size 1.27 1.27)
+				)
+				(hide yes)
+			)
+		)
+		(property "Datasheet" ""
+			(at 219.71 33.02 0)
+			(effects
+				(font
+					(size 1.27 1.27)
+				)
+				(hide yes)
+			)
+		)
+		(property "Description" "Power symbol creates a global label with name \"GND\" , ground"
+			(at 219.71 33.02 0)
+			(effects
+				(font
+					(size 1.27 1.27)
+				)
+				(hide yes)
+			)
+		)
+		(pin "1"
+		)
+		(instances
+			(project ""
+				(path "/81c7d85e-7490-4ec7-8863-b12337cd9cc9"
+					(reference "#PWR02")
+					(unit 1)
+				)
