File: pcb/pipar_sool_pnp/pipar_sool_pnp.kicad_pcb (KiCad board)
At the start: 2 copper layers, 142.4 x 110.5 mm, 170 parts, among them SW1 SW_Wuerth_450301014042, SW2 SW_Wuerth_450301014042, U1 Seeeduino Xiao nRF52840, U2 Seeeduino Xiao nRF52840

Commit message: Further changes to placement
Parts:
- removed the CH1 at (183.2, 87.2)
- removed the CH10 at (246.0, -0.29)
- removed the CH11 at (246.0, 17.0)
- removed the CH12 at (246.0, 34.2)
- removed the CH13 at (269.2, 5.89)
- removed the CH14 at (267.7, 23.1)
- removed the CH15 at (266.2, 40.3)
- removed the CH16 at (297.0, 27.0)
- removed the CH17 at (289.7, 42.7)
- removed the CH18 at (282.4, 58.3)
- removed the CH2 at (198.1, 76.7)
- removed the CH3 at (213.1, 66.2)
- removed the CH4 at (204.4, 7.15)
- removed the CH5 at (205.9, 24.3)
- removed the CH6 at (207.4, 41.5)
- removed the CH7 at (223.3, 2.33)
- removed the CH8 at (224.8, 19.5)
- removed the CH9 at (226.3, 36.7)
- moved H16 287.1 mm to (211.2, 79.7), turned to -25 degrees
- moved CH16 285.4 mm to (206.9, 83.1), turned to -25 degrees
- moved CH34 284.8 mm to (211.4, 85.2), turned to 155 degrees
- moved H17 279.9 mm to (203.9, 95.4), turned to -25 degrees
- moved CH17 278.2 mm to (199.6, 98.7), turned to -25 degrees
- moved CH35 277.6 mm to (204.2, 100.8), turned to 155 degrees
- moved H18 272.7 mm to (196.7, 111.0), turned to -25 degrees
- moved CH18 271.0 mm to (192.3, 114.3), turned to -25 degrees
- moved CH36 270.4 mm to (196.9, 116.5), turned to 155 degrees
- moved H13 260.2 mm to (183.5, 58.6), turned to -5 degrees
- moved CH31 259.8 mm to (185.5, 63.6), turned to 175 degrees
- moved CH13 259.8 mm to (180.6, 63.2), turned to -5 degrees
- moved CH30 258.9 mm to (162.8, 91.8)
- moved H12 258.9 mm to (160.3, 86.9)
- moved CH12 258.9 mm to (157.8, 91.8)
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Routing:
- net (no net): vias 126 -> 0

Commit message: Finish PnP position files
Parts:
- removed the D1 at (90.2, 145.2) (x2)
- removed the D10 at (151.2, 52.6) (x2)
- removed the D11 at (151.3, 69.9) (x2)
- removed the D12 at (151.4, 87.1) (x2)
- removed the D13 at (174.5, 58.0) (x2)
- removed the D14 at (173.0, 75.1) (x2)
- removed the D15 at (171.5, 92.3) (x2)
- removed the D16 at (203.0, 76.1) (x2)
- removed the D17 at (195.7, 91.7) (x2)
- removed the D18 at (188.4, 107.3) (x2)
- removed the D2 at (105.2, 134.7) (x2)
- removed the D3 at (120.1, 124.3) (x2)
- removed the D4 at (109.7, 60.8) (x2)
- removed the D5 at (111.3, 78.0) (x2)
- removed the D6 at (112.7, 95.2) (x2)
- removed the D7 at (128.6, 56.0) (x2)
- removed the D8 at (130.0, 73.2) (x2)
- removed the D9 at (131.6, 90.4) (x2)
- removed the SW1 at (220.1, 69.5) (x2)
- removed the U1 at (191.3, 133.7) (x2)
- removed the U2 at (118.8, 107.8)
- removed the U3 at (148.7, 48.3)
- removed U4 (x2): ~, MountingHole:MountingHole_2.2mm_M2
- removed the U6 at (176.3, 140.3)
- removed the U7 at (157.5, 123.0) (x2)
- moved SW1 333.1 mm to (221.0, 74.2), turned to 155 degrees
- moved SW2 333.1 mm to (221.0, 74.2), turned to -25 degrees
- moved TP2 315.7 mm to (214.3, 73.1), turned to -25 degrees
- moved TP1 306.0 mm to (209.2, 70.7), turned to -25 degrees
- moved U8 289.0 mm to (158.5, 127.7)
- moved U8 289.0 mm to (158.4, 127.7)
- moved D16 285.2 mm to (203.9, 80.8), turned to -115 degrees
- moved D34 285.2 mm to (203.9, 80.8), turned to -115 degrees
- moved D17 275.2 mm to (196.6, 96.4), turned to -115 degrees
- moved D35 275.2 mm to (196.6, 96.4), turned to -115 degrees
- moved D18 265.4 mm to (189.3, 112.1), turned to -115 degrees
- moved D36 265.4 mm to (189.3, 112.1), turned to -115 degrees
- moved D13 258.2 mm to (175.4, 62.7), turned to -95 degrees
- moved D31 258.2 mm to (175.4, 62.7), turned to -95 degrees
- moved D14 253.0 mm to (173.9, 79.8), turned to -95 degrees
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