File: pcb/pipar_sool_pnp/pipar_sool_pnp.kicad_sch (KiCad schematic)
At the start: 102 parts, among them SW1 SW_Wuerth_450301014042, SW2 SW_Wuerth_450301014042, U1 Seeeduino Xiao nRF52840, U2 Seeeduino Xiao nRF52840

Commit message: Finish PnP position files
Parts:
- U8: now left out of the parts list
Changed lines of the file:
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@@
 		(unit 1)
 		(exclude_from_sim no)
-		(in_bom yes)
+		(in_bom no)
 		(on_board yes)
 		(dnp no)
