File: pcb/pipar_sool/pipar_sool.kicad_pcb (KiCad board)
At the start: 2 copper layers, 139.4 x 109.8 mm, 109 parts, among them M2 MountingHole_2.2mm_M2, SW1 SW_Wuerth_450301014042

Commit message: Recreated Sool & Pipar for production run
Parts:
- removed ? (x44): , 
- removed the D1 at (20.3, 105.5)
- removed the D1 at (29.3, 121.1)
- removed the D10 at (94.9, 25.5)
- removed the D10 at (76.9, 25.5)
- removed the D11 at (94.9, 43.2)
- removed the D11 at (76.9, 43.2)
- removed the D12 at (94.9, 61.0)
- removed the D12 at (76.9, 61.0)
- removed the D13 at (118.6, 32.0)
- removed the D13 at (100.7, 30.5)
- removed the D14 at (117.0, 49.7)
- removed the D14 at (99.1, 48.2)
- removed the D15 at (115.5, 67.4)
- removed the D15 at (97.6, 65.9)
- removed the D16 at (146.0, 56.5)
- removed the D16 at (129.7, 48.9)
- removed the D17 at (138.5, 72.6)
- removed the D17 at (122.2, 65.0)
- removed the D18 at (131.0, 88.7)
- removed the D18 at (114.7, 81.1)
- removed the D2 at (35.7, 96.6)
- removed the D2 at (44.6, 112.2)
- removed the D3 at (51.0, 87.7)
- removed the D3 at (60.0, 103.3)
- removed the D4 at (51.9, 35.0)
- removed the D4 at (34.0, 36.6)
- removed the D5 at (53.5, 52.7)
- removed the D5 at (35.6, 54.3)
- removed the D6 at (55.0, 70.4)
- removed the D6 at (37.1, 72.0)
- removed the D7 at (71.7, 30.2)
- removed the D7 at (53.8, 31.7)
- removed the D8 at (73.2, 47.9)
- removed the D8 at (55.3, 49.4)
- removed the D9 at (74.8, 65.6)
- removed the D9 at (56.9, 67.1)
- removed M2 (x5): MountingHole_2.2mm_M2, MountingHole:MountingHole_2.2mm_M2
- removed REF** (x2): Salt & Pepper, Art:Salt
- removed the SW1 at (143.5, 42.9) (x2)
- added D1: D, Diode_SMD:Nexperia_CFP3_SOD-123W, F.Cu at (67.6, 140.1)
- added D1: D, Diode_SMD:Nexperia_CFP3_SOD-123W, B.Cu at (67.6, 140.1)
- added D10: D, Diode_SMD:Nexperia_CFP3_SOD-123W, F.Cu at (128.6, 47.5)
- added D10: D, Diode_SMD:Nexperia_CFP3_SOD-123W, B.Cu at (128.6, 47.5)
- added D11: D, Diode_SMD:Nexperia_CFP3_SOD-123W, F.Cu at (128.6, 64.8)
- added D11: D, Diode_SMD:Nexperia_CFP3_SOD-123W, B.Cu at (128.6, 64.8)
- added D12: D, Diode_SMD:Nexperia_CFP3_SOD-123W, F.Cu at (128.7, 81.9)
- added D12: D, Diode_SMD:Nexperia_CFP3_SOD-123W, B.Cu at (128.7, 81.9)
- added D13: D, Diode_SMD:Nexperia_CFP3_SOD-123W, F.Cu at (151.8, 52.8)
- added D13: D, Diode_SMD:Nexperia_CFP3_SOD-123W, B.Cu at (151.8, 52.8)
- added D14: D, Diode_SMD:Nexperia_CFP3_SOD-123W, F.Cu at (150.4, 70.0)
- added D14: D, Diode_SMD:Nexperia_CFP3_SOD-123W, B.Cu at (150.4, 70.0)
- added D15: D, Diode_SMD:Nexperia_CFP3_SOD-123W, F.Cu at (148.9, 87.2)
- added D15: D, Diode_SMD:Nexperia_CFP3_SOD-123W, B.Cu at (148.9, 87.2)
- added D16: D, Diode_SMD:Nexperia_CFP3_SOD-123W, F.Cu at (180.3, 70.9)
- added D16: D, Diode_SMD:Nexperia_CFP3_SOD-123W, B.Cu at (180.3, 70.9)
- added D17: D, Diode_SMD:Nexperia_CFP3_SOD-123W, F.Cu at (173.1, 86.6)
- added D17: D, Diode_SMD:Nexperia_CFP3_SOD-123W, B.Cu at (173.1, 86.6)
- added D18: D, Diode_SMD:Nexperia_CFP3_SOD-123W, F.Cu at (165.8, 102.2)
- added D18: D, Diode_SMD:Nexperia_CFP3_SOD-123W, B.Cu at (165.8, 102.2)
- added D2: D, Diode_SMD:Nexperia_CFP3_SOD-123W, F.Cu at (82.6, 129.6)
- added D2: D, Diode_SMD:Nexperia_CFP3_SOD-123W, B.Cu at (82.6, 129.6)
- added D3: D, Diode_SMD:Nexperia_CFP3_SOD-123W, F.Cu at (97.5, 119.2)
- added D3: D, Diode_SMD:Nexperia_CFP3_SOD-123W, B.Cu at (97.5, 119.2)
- added D4: D, Diode_SMD:Nexperia_CFP3_SOD-123W, F.Cu at (87.1, 55.7)
- added D4: D, Diode_SMD:Nexperia_CFP3_SOD-123W, B.Cu at (87.1, 55.7)
- added D5: D, Diode_SMD:Nexperia_CFP3_SOD-123W, F.Cu at (88.6, 72.9)
- added D5: D, Diode_SMD:Nexperia_CFP3_SOD-123W, B.Cu at (88.6, 72.9)
- added D6: D, Diode_SMD:Nexperia_CFP3_SOD-123W, F.Cu at (90.1, 90.1)
- added D6: D, Diode_SMD:Nexperia_CFP3_SOD-123W, B.Cu at (90.1, 90.1)
- added D7: D, Diode_SMD:Nexperia_CFP3_SOD-123W, F.Cu at (106.0, 50.9)
- added D7: D, Diode_SMD:Nexperia_CFP3_SOD-123W, B.Cu at (106.0, 50.9)
- added D8: D, Diode_SMD:Nexperia_CFP3_SOD-123W, F.Cu at (107.4, 68.1)
- added D8: D, Diode_SMD:Nexperia_CFP3_SOD-123W, B.Cu at (107.4, 68.1)
- added D9: D, Diode_SMD:Nexperia_CFP3_SOD-123W, F.Cu at (109.0, 85.2)
- added D9: D, Diode_SMD:Nexperia_CFP3_SOD-123W, B.Cu at (109.0, 85.2)
- added SW1: SW_Wuerth_450301014042, Button_Switch_SMD:SW_SPDT_PCM12, F.Cu at (197.5, 64.4)
- added SW1: SW_Wuerth_450301014042, Button_Switch_SMD:SW_SPDT_PCM12, B.Cu at (197.5, 64.4)
- added U1: Seeeduino Xiao nRF52840, Seeed Studio XIAO Series Library:XIAO-nRF52840-Sense-14P-2.54-21X17.8MM, F.Cu at (168.7, 128.6)
- added U1: Seeeduino Xiao nRF52840, Seeed Studio XIAO Series Library:XIAO-nRF52840-Sense-14P-2.54-21X17.8MM, B.Cu at (168.7, 128.6)
- added U2: ~, MountingHole:MountingHole_2.2mm_M2, F.Cu at (96.1, 102.6)
- added U3: ~, MountingHole:MountingHole_2.2mm_M2, F.Cu at (126.0, 43.2)
- added U4: ~, MountingHole:MountingHole_2.2mm_M2, F.Cu at (178.6, 58.6)
- added U5: ~, MountingHole:MountingHole_2.2mm_M2, F.Cu at (96.1, 135.2)
- added U6: ~, MountingHole:MountingHole_2.2mm_M2, F.Cu at (153.6, 135.2)
- added U7: ~, Art:Salt, F.Cu at (134.9, 117.9)
- added U7: ~, Art:Salt, B.Cu at (134.9, 117.9)
- TP1: footprint TestPoint:TestPoint_THTPad_D2.0mm_Drill1.0mm -> TestPoint:TestPoint_THTPad_2.0x2.0mm_Drill1.0mm
- TP2: footprint TestPoint:TestPoint_THTPad_2.0x2.0mm_Drill1.0mm -> TestPoint:TestPoint_THTPad_D2.0mm_Drill1.0mm
- moved TP2 98.1 mm to (190.7, 63.3), turned to 65 degrees
- moved TP1 96.7 mm to (185.6, 60.9), turned to 65 degrees
- moved CH4 55.8 mm to (96.0, 54.7)
- moved CH10 55.7 mm to (137.7, 47.3)
- moved CH5 55.6 mm to (97.5, 71.9)
- moved CH11 55.5 mm to (137.7, 64.5)
- moved CH13 55.4 mm to (160.8, 53.5)
- moved CH6 55.4 mm to (99.0, 89.1)
- moved CH18 55.4 mm to (174.0, 105.9)
- moved CH17 55.3 mm to (181.3, 90.3)
- moved CH12 55.3 mm to (137.7, 81.8)
- moved CH16 55.3 mm to (188.6, 74.6)
- moved CH14 55.3 mm to (159.3, 70.7)
- moved CH15 55.1 mm to (157.8, 87.8)
- moved CH7 55.0 mm to (114.9, 49.9)
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Routing:
- net Net-(SW1-C): track 90.4 -> 10.1 mm
- net GND: track 50.0 -> 123.5 mm, vias 3 -> 24
- net Net-(D12-K): track 220.8 -> 178.6 mm, vias 14 -> 7
- net Net-(U1-P0.28): track 146.3 -> 109.7 mm
- net Net-(U1-P0.29): track 163.9 -> 128.4 mm
- net Net-(U1-P0.03): track 129.3 -> 95.0 mm
- net Net-(U1-P0.04): track 178.8 -> 144.5 mm
- net Net-(U1-P0.05): track 193.3 -> 162.4 mm
- net Net-(D11-K): track 253.2 -> 236.5 mm, vias 14 -> 7
- net Net-(D1-K): track 312.1 -> 296.6 mm, vias 14 -> 7
- net Net-(U1-P1.11): track 174.3 -> 166.8 mm, vias 4 -> 6
- net Net-(SW1-B): track 110.0 -> 111.3 mm, vias 5 -> 3
- net unconnected-(SW1-A-Pad3): track 8.43 -> 9.67 mm
- net Net-(D2-A): track 27.5 -> 26.9 mm, vias 1 -> 2
- net Net-(D5-A): track 27.4 -> 26.9 mm, vias 1 -> 2
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Other:
- board size 139.4 x 109.8 mm -> 142.4 x 110.5 mm
- board text added: "+"
- board text added: "-"
- board text added: "Left Side"
- board text added: "Right Side"
- board text removed: "BAT+"
- board text removed: "BAT-"
- board text removed: "Right side"

Commit message: Adds PCBWay zip and adds on off hints
Other:
- board text added: "O"
- board text added: "|"
Changed lines of the file:
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@@
 		(fp_arc
 			(start 2.500004 2.199999)
-			(mid 2.060661 3.26066)
+			(mid 2.06066 3.260659)
 			(end 0.999998 3.699998)
 			(stroke
@@
 		(fp_arc
 			(start 2.500004 2.199999)
-			(mid 2.060661 3.26066)
+			(mid 2.06066 3.260659)
 			(end 0.999998 3.699998)
 			(stroke
@@
 		(fp_arc
 			(start 8.9 8.5)
-			(mid 8.314211 9.914215)
+			(mid 8.31421 9.914211)
 			(end 6.899998 10.500006)
 			(stroke
@@
 		(fp_arc
 			(start 2.500004 2.199999)
-			(mid 2.060661 3.26066)
+			(mid 2.06066 3.260659)
 			(end 0.999998 3.699998)
 			(stroke
@@
 		(fp_arc
 			(start 2.500004 2.199999)
-			(mid 2.060661 3.26066)
+			(mid 2.06066 3.260659)
 			(end 0.999998 3.699998)
 			(stroke
@@
 		)
 	)
+	(gr_text "|"
+		(at 193.23 62.91 -25)
+		(layer "B.SilkS")
+		(effects
+			(font
+				(size 1.5 1.5)
+				(thickness 0.1)
+			)
+			(justify left bottom mirror)
+		)
+	)
 	(gr_text "-"
 		(at 184.71 59.25 65)
@@
 		)
 	)
+	(gr_text "O"
+		(at 202.59 67.55 -25)
+		(layer "B.SilkS")
+		(effects
+			(font
+				(size 1.5 1.5)
+				(thickness 0.1)
+			)
+			(justify left bottom mirror)
+		)
+	)
 	(gr_text "Right Side"
 		(at 131.98 92.01 0)
@@
 		)
 	)
+	(gr_text "|"
+		(at 203.22 66.02 155)
+		(layer "F.SilkS")
+		(effects
+			(font
+				(size 1.5 1.5)
+				(thickness 0.1)
+			)
+			(justify left bottom)
+		)
+	)
 	(gr_text "+"
 		(at 189.1 63.49 65)
@@
 		(layer "F.SilkS")
 		(effects
+			(font
+				(size 1.5 1.5)
+				(thickness 0.1)
+			)
+			(justify left bottom)
+		)
+	)
+	(gr_text "O"
+		(at 193.997091 61.44393 155)
+		(layer "F.SilkS")
+		(effects

Commit message: start of creating newer models
Parts:
- removed the D1 at (67.6, 140.1) (x2)
- removed the D10 at (128.6, 47.5) (x2)
- removed the D11 at (128.6, 64.8) (x2)
- removed the D12 at (128.7, 81.9) (x2)
- removed the D13 at (151.8, 52.8) (x2)
- removed the D14 at (150.4, 70.0) (x2)
- removed the D15 at (148.9, 87.2) (x2)
- removed the D16 at (180.3, 70.9) (x2)
- removed the D17 at (173.1, 86.6) (x2)
- removed the D18 at (165.8, 102.2) (x2)
- removed the D2 at (82.6, 129.6) (x2)
- removed the D3 at (97.5, 119.2) (x2)
- removed the D4 at (87.1, 55.7) (x2)
- removed the D5 at (88.6, 72.9) (x2)
- removed the D6 at (90.1, 90.1) (x2)
- removed the D7 at (106.0, 50.9) (x2)
- removed the D8 at (107.4, 68.1) (x2)
- removed the D9 at (109.0, 85.2) (x2)
- removed the SW1 at (197.5, 64.4) (x2)
- removed the U1 at (168.7, 128.6) (x2)
- removed the U7 at (134.9, 117.9) (x2)
- added CH19: KSwitch, Keyboard:Kailh_HS_Socket, F.Cu at (50.6, 144.3)
- added CH20: KSwitch, Keyboard:Kailh_HS_Socket, F.Cu at (65.2, 134.1)
- added CH21: KSwitch, Keyboard:Kailh_HS_Socket, F.Cu at (79.7, 123.9)
- added CH22: KSwitch, Keyboard:Kailh_HS_Socket, F.Cu at (68.4, 64.3)
- added CH23: KSwitch, Keyboard:Kailh_HS_Socket, F.Cu at (69.9, 81.0)
- added CH24: KSwitch, Keyboard:Kailh_HS_Socket, F.Cu at (71.4, 97.7)
- added CH25: KSwitch, Keyboard:Kailh_HS_Socket, F.Cu at (87.3, 59.5)
- added CH26: KSwitch, Keyboard:Kailh_HS_Socket, F.Cu at (88.8, 76.2)
- added CH27: KSwitch, Keyboard:Kailh_HS_Socket, F.Cu at (90.2, 92.9)
- added CH28: KSwitch, Keyboard:Kailh_HS_Socket, F.Cu at (109.6, 56.7)
- added CH29: KSwitch, Keyboard:Kailh_HS_Socket, F.Cu at (109.6, 73.5)
- added CH30: KSwitch, Keyboard:Kailh_HS_Socket, F.Cu at (109.6, 90.2)
- added CH31: KSwitch, Keyboard:Kailh_HS_Socket, F.Cu at (131.6, 62.5)
- added CH32: KSwitch, Keyboard:Kailh_HS_Socket, F.Cu at (130.2, 79.2)
- added CH33: KSwitch, Keyboard:Kailh_HS_Socket, F.Cu at (128.7, 95.9)
- added CH34: KSwitch, Keyboard:Kailh_HS_Socket, F.Cu at (158.0, 83.3)
- added CH35: KSwitch, Keyboard:Kailh_HS_Socket, F.Cu at (151.0, 98.5)
- added CH36: KSwitch, Keyboard:Kailh_HS_Socket, F.Cu at (143.9, 113.7)
- added D1: D, Diode_SMD:D_0402_1005Metric, F.Cu at (43.9, 143.0)
- added D10: D, Diode_SMD:D_0402_1005Metric, F.Cu at (104.8, 51.8)
- added D11: D, Diode_SMD:D_0402_1005Metric, F.Cu at (104.8, 68.6)
- added D12: D, Diode_SMD:D_0402_1005Metric, F.Cu at (104.8, 85.3)
- added D13: D, Diode_SMD:D_0402_1005Metric, F.Cu at (127.2, 57.2)
- added D14: D, Diode_SMD:D_0402_1005Metric, F.Cu at (125.8, 73.9)
- added D15: D, Diode_SMD:D_0402_1005Metric, F.Cu at (124.3, 90.6)
- added D16: D, Diode_SMD:D_0402_1005Metric, F.Cu at (155.7, 76.9)
- added D17: D, Diode_SMD:D_0402_1005Metric, F.Cu at (148.7, 92.1)
- added D18: D, Diode_SMD:D_0402_1005Metric, F.Cu at (141.6, 107.3)
- added D19: D, Diode_SMD:D_0402_1005Metric, B.Cu at (43.9, 143.0)
- added D2: D, Diode_SMD:D_0402_1005Metric, F.Cu at (58.4, 132.8)
- added D20: D, Diode_SMD:D_0402_1005Metric, B.Cu at (58.4, 132.8)
- added D21: D, Diode_SMD:D_0402_1005Metric, B.Cu at (73.0, 122.7)
- added D22: D, Diode_SMD:D_0402_1005Metric, B.Cu at (63.2, 59.9)
- added D23: D, Diode_SMD:D_0402_1005Metric, B.Cu at (64.7, 76.6)
- added D24: D, Diode_SMD:D_0402_1005Metric, B.Cu at (66.2, 93.3)
- added D25: D, Diode_SMD:D_0402_1005Metric, B.Cu at (82.1, 55.1)
- added D26: D, Diode_SMD:D_0402_1005Metric, B.Cu at (83.6, 71.8)
- added D27: D, Diode_SMD:D_0402_1005Metric, B.Cu at (85.0, 88.5)
- added D28: D, Diode_SMD:D_0402_1005Metric, B.Cu at (104.8, 51.8)
- added D29: D, Diode_SMD:D_0402_1005Metric, B.Cu at (104.8, 68.6)
- added D3: D, Diode_SMD:D_0402_1005Metric, F.Cu at (73.0, 122.7)
- added D30: D, Diode_SMD:D_0402_1005Metric, B.Cu at (104.8, 85.3)
- added D31: D, Diode_SMD:D_0402_1005Metric, B.Cu at (127.2, 57.2)
- added D32: D, Diode_SMD:D_0402_1005Metric, B.Cu at (125.8, 73.9)
- added D33: D, Diode_SMD:D_0402_1005Metric, B.Cu at (124.3, 90.6)
- added D34: D, Diode_SMD:D_0402_1005Metric, B.Cu at (155.7, 76.9)
- added D35: D, Diode_SMD:D_0402_1005Metric, B.Cu at (148.7, 92.1)
- added D36: D, Diode_SMD:D_0402_1005Metric, B.Cu at (141.6, 107.3)
- added D4: D, Diode_SMD:D_0402_1005Metric, F.Cu at (63.2, 59.9)
- added D5: D, Diode_SMD:D_0402_1005Metric, F.Cu at (64.7, 76.6)
- added D6: D, Diode_SMD:D_0402_1005Metric, F.Cu at (66.2, 93.3)
- added D7: D, Diode_SMD:D_0402_1005Metric, F.Cu at (82.1, 55.1)
- added D8: D, Diode_SMD:D_0402_1005Metric, F.Cu at (83.6, 71.8)
- added D9: D, Diode_SMD:D_0402_1005Metric, F.Cu at (85.0, 88.5)
- added H1: MountingHole, Keyboard:Kailh_socket_PG1350_reversible_Holes, F.Cu at (49.9, 138.9)
- added H10: MountingHole, Keyboard:Kailh_socket_PG1350_reversible_Holes, F.Cu at (112.1, 51.9)
- added H11: MountingHole, Keyboard:Kailh_socket_PG1350_reversible_Holes, F.Cu at (112.1, 68.6)
- added H12: MountingHole, Keyboard:Kailh_socket_PG1350_reversible_Holes, F.Cu at (112.1, 85.3)
- added H13: MountingHole, Keyboard:Kailh_socket_PG1350_reversible_Holes, F.Cu at (134.5, 57.9)
- added H14: MountingHole, Keyboard:Kailh_socket_PG1350_reversible_Holes, F.Cu at (133.1, 74.6)
- added H15: MountingHole, Keyboard:Kailh_socket_PG1350_reversible_Holes, F.Cu at (131.6, 91.3)
- added H16: MountingHole, Keyboard:Kailh_socket_PG1350_reversible_Holes, F.Cu at (162.4, 80.0)
- added H17: MountingHole, Keyboard:Kailh_socket_PG1350_reversible_Holes, F.Cu at (155.3, 95.2)
- added H18: MountingHole, Keyboard:Kailh_socket_PG1350_reversible_Holes, F.Cu at (148.2, 110.4)
- added H2: MountingHole, Keyboard:Kailh_socket_PG1350_reversible_Holes, F.Cu at (64.4, 128.7)
- added H3: MountingHole, Keyboard:Kailh_socket_PG1350_reversible_Holes, B.Cu at (79.0, 118.5)
- added H4: MountingHole, Keyboard:Kailh_socket_PG1350_reversible_Holes, F.Cu at (70.5, 59.3)
- added H5: MountingHole, Keyboard:Kailh_socket_PG1350_reversible_Holes, F.Cu at (72.0, 76.0)
- added H6: MountingHole, Keyboard:Kailh_socket_PG1350_reversible_Holes, F.Cu at (73.4, 92.7)
- added H7: MountingHole, Keyboard:Kailh_socket_PG1350_reversible_Holes, F.Cu at (89.4, 54.5)
- added H8: MountingHole, Keyboard:Kailh_socket_PG1350_reversible_Holes, F.Cu at (90.8, 71.2)
- added H9: MountingHole, Keyboard:Kailh_socket_PG1350_reversible_Holes, F.Cu at (92.3, 87.9)
- added LED1: ~, LED_SMD:LED_0402_1005Metric_Pad0.77x0.64mm_HandSolder, B.Cu at (46.8, 134.4)
- added LED10: ~, LED_SMD:LED_0402_1005Metric_Pad0.77x0.64mm_HandSolder, B.Cu at (112.1, 46.4)
- added LED11: ~, LED_SMD:LED_0402_1005Metric_Pad0.77x0.64mm_HandSolder, B.Cu at (112.1, 63.2)
- added LED12: ~, LED_SMD:LED_0402_1005Metric_Pad0.77x0.64mm_HandSolder, B.Cu at (112.1, 79.9)
- added LED13: ~, LED_SMD:LED_0402_1005Metric_Pad0.77x0.64mm_HandSolder, B.Cu at (135.0, 52.5)
- added LED14: ~, LED_SMD:LED_0402_1005Metric_Pad0.77x0.64mm_HandSolder, B.Cu at (133.6, 69.2)
- added LED15: ~, LED_SMD:LED_0402_1005Metric_Pad0.77x0.64mm_HandSolder, B.Cu at (132.1, 85.9)
- added LED16: ~, LED_SMD:LED_0402_1005Metric_Pad0.77x0.64mm_HandSolder, B.Cu at (164.7, 75.1)
- added LED17: ~, LED_SMD:LED_0402_1005Metric_Pad0.77x0.64mm_HandSolder, B.Cu at (157.6, 90.3)
- added LED18: ~, LED_SMD:LED_0402_1005Metric_Pad0.77x0.64mm_HandSolder, B.Cu at (150.5, 105.5)
- added LED19: ~, LED_SMD:LED_0402_1005Metric_Pad0.77x0.64mm_HandSolder, F.Cu at (46.8, 134.4)
- added LED2: ~, LED_SMD:LED_0402_1005Metric_Pad0.77x0.64mm_HandSolder, B.Cu at (61.3, 124.2)
- added LED20: ~, LED_SMD:LED_0402_1005Metric_Pad0.77x0.64mm_HandSolder, F.Cu at (61.3, 124.2)
- added LED21: ~, LED_SMD:LED_0402_1005Metric_Pad0.77x0.64mm_HandSolder, F.Cu at (75.9, 114.0)
- added LED22: ~, LED_SMD:LED_0402_1005Metric_Pad0.77x0.64mm_HandSolder, F.Cu at (70.1, 53.9)
- added LED23: ~, LED_SMD:LED_0402_1005Metric_Pad0.77x0.64mm_HandSolder, F.Cu at (71.5, 70.6)
- added LED24: ~, LED_SMD:LED_0402_1005Metric_Pad0.77x0.64mm_HandSolder, F.Cu at (73.0, 87.3)
- added LED25: ~, LED_SMD:LED_0402_1005Metric_Pad0.77x0.64mm_HandSolder, F.Cu at (88.9, 49.0)
- added LED26: ~, LED_SMD:LED_0402_1005Metric_Pad0.77x0.64mm_HandSolder, F.Cu at (90.4, 65.8)
- added LED27: ~, LED_SMD:LED_0402_1005Metric_Pad0.77x0.64mm_HandSolder, F.Cu at (91.9, 82.4)
- added LED28: ~, LED_SMD:LED_0402_1005Metric_Pad0.77x0.64mm_HandSolder, F.Cu at (112.1, 46.4)
- added LED29: ~, LED_SMD:LED_0402_1005Metric_Pad0.77x0.64mm_HandSolder, F.Cu at (112.1, 63.2)
- added LED3: ~, LED_SMD:LED_0402_1005Metric_Pad0.77x0.64mm_HandSolder, B.Cu at (75.9, 114.0)
- added LED30: ~, LED_SMD:LED_0402_1005Metric_Pad0.77x0.64mm_HandSolder, F.Cu at (112.1, 79.9)
- added LED31: ~, LED_SMD:LED_0402_1005Metric_Pad0.77x0.64mm_HandSolder, F.Cu at (135.0, 52.5)
- added LED32: ~, LED_SMD:LED_0402_1005Metric_Pad0.77x0.64mm_HandSolder, F.Cu at (133.6, 69.2)
- added LED33: ~, LED_SMD:LED_0402_1005Metric_Pad0.77x0.64mm_HandSolder, F.Cu at (132.1, 85.9)
- added LED34: ~, LED_SMD:LED_0402_1005Metric_Pad0.77x0.64mm_HandSolder, F.Cu at (164.7, 75.1)
- added LED35: ~, LED_SMD:LED_0402_1005Metric_Pad0.77x0.64mm_HandSolder, F.Cu at (157.6, 90.3)
- added LED36: ~, LED_SMD:LED_0402_1005Metric_Pad0.77x0.64mm_HandSolder, F.Cu at (150.5, 105.5)
- added LED4: ~, LED_SMD:LED_0402_1005Metric_Pad0.77x0.64mm_HandSolder, B.Cu at (70.1, 53.9)
- added LED5: ~, LED_SMD:LED_0402_1005Metric_Pad0.77x0.64mm_HandSolder, B.Cu at (71.5, 70.6)
- added LED6: ~, LED_SMD:LED_0402_1005Metric_Pad0.77x0.64mm_HandSolder, B.Cu at (73.0, 87.3)
- added LED7: ~, LED_SMD:LED_0402_1005Metric_Pad0.77x0.64mm_HandSolder, B.Cu at (88.9, 49.0)
- added LED8: ~, LED_SMD:LED_0402_1005Metric_Pad0.77x0.64mm_HandSolder, B.Cu at (90.4, 65.8)
- added LED9: ~, LED_SMD:LED_0402_1005Metric_Pad0.77x0.64mm_HandSolder, B.Cu at (91.9, 82.4)
- added Q1: AO3416 N-channel MOSFET, Package_TO_SOT_SMD:SOT-23, F.Cu at (38.1, 108.8)
- added Q2: AO3416 N-channel MOSFET, Package_TO_SOT_SMD:SOT-23, B.Cu at (38.1, 108.8)
- added R1: 100, Resistor_SMD:R_0402_1005Metric_Pad0.72x0.64mm_HandSolder, B.Cu at (47.6, 135.6)
- added R10: 100, Resistor_SMD:R_0402_1005Metric_Pad0.72x0.64mm_HandSolder, B.Cu at (112.1, 47.9)
- added R11: 100, Resistor_SMD:R_0402_1005Metric_Pad0.72x0.64mm_HandSolder, B.Cu at (112.1, 64.7)
- added R12: 100, Resistor_SMD:R_0402_1005Metric_Pad0.72x0.64mm_HandSolder, B.Cu at (112.1, 81.4)
- added R13: 100, Resistor_SMD:R_0402_1005Metric_Pad0.72x0.64mm_HandSolder, B.Cu at (134.9, 54.0)
- added R14: 100, Resistor_SMD:R_0402_1005Metric_Pad0.72x0.64mm_HandSolder, B.Cu at (133.5, 70.7)
- added R15: 100, Resistor_SMD:R_0402_1005Metric_Pad0.72x0.64mm_HandSolder, B.Cu at (132.0, 87.4)
- added R16: 100, Resistor_SMD:R_0402_1005Metric_Pad0.72x0.64mm_HandSolder, B.Cu at (164.1, 76.5)
- added R17: 100, Resistor_SMD:R_0402_1005Metric_Pad0.72x0.64mm_HandSolder, B.Cu at (157.0, 91.7)
- added R18: 100, Resistor_SMD:R_0402_1005Metric_Pad0.72x0.64mm_HandSolder, B.Cu at (149.9, 106.9)
- added R19: 4.7k, Resistor_SMD:R_0402_1005Metric_Pad0.72x0.64mm_HandSolder, F.Cu at (40.6, 108.8)
- added R2: 100, Resistor_SMD:R_0402_1005Metric_Pad0.72x0.64mm_HandSolder, B.Cu at (62.2, 125.4)
- added R20: 100, Resistor_SMD:R_0402_1005Metric_Pad0.72x0.64mm_HandSolder, F.Cu at (47.6, 135.6)
- added R21: 100, Resistor_SMD:R_0402_1005Metric_Pad0.72x0.64mm_HandSolder, F.Cu at (62.2, 125.4)
- added R22: 100, Resistor_SMD:R_0402_1005Metric_Pad0.72x0.64mm_HandSolder, F.Cu at (76.7, 115.2)
- added R23: 100, Resistor_SMD:R_0402_1005Metric_Pad0.72x0.64mm_HandSolder, F.Cu at (70.2, 55.4)
- added R24: 100, Resistor_SMD:R_0402_1005Metric_Pad0.72x0.64mm_HandSolder, F.Cu at (71.7, 72.1)
- added R25: 100, Resistor_SMD:R_0402_1005Metric_Pad0.72x0.64mm_HandSolder, F.Cu at (73.1, 88.8)
- added R26: 100, Resistor_SMD:R_0402_1005Metric_Pad0.72x0.64mm_HandSolder, F.Cu at (89.1, 50.5)
- added R27: 100, Resistor_SMD:R_0402_1005Metric_Pad0.72x0.64mm_HandSolder, F.Cu at (90.5, 67.3)
- added R28: 100, Resistor_SMD:R_0402_1005Metric_Pad0.72x0.64mm_HandSolder, F.Cu at (92.0, 83.9)
- added R29: 100, Resistor_SMD:R_0402_1005Metric_Pad0.72x0.64mm_HandSolder, F.Cu at (112.1, 47.9)
- added R3: 100, Resistor_SMD:R_0402_1005Metric_Pad0.72x0.64mm_HandSolder, B.Cu at (76.7, 115.2)
- added R30: 100, Resistor_SMD:R_0402_1005Metric_Pad0.72x0.64mm_HandSolder, F.Cu at (112.1, 64.7)
- added R31: 100, Resistor_SMD:R_0402_1005Metric_Pad0.72x0.64mm_HandSolder, F.Cu at (112.1, 81.4)
- added R32: 100, Resistor_SMD:R_0402_1005Metric_Pad0.72x0.64mm_HandSolder, F.Cu at (134.9, 54.0)
- added R33: 100, Resistor_SMD:R_0402_1005Metric_Pad0.72x0.64mm_HandSolder, F.Cu at (133.5, 70.7)
- added R34: 100, Resistor_SMD:R_0402_1005Metric_Pad0.72x0.64mm_HandSolder, F.Cu at (132.0, 87.4)
- added R35: 100, Resistor_SMD:R_0402_1005Metric_Pad0.72x0.64mm_HandSolder, F.Cu at (164.1, 76.5)
- added R36: 100, Resistor_SMD:R_0402_1005Metric_Pad0.72x0.64mm_HandSolder, F.Cu at (157.0, 91.7)
- added R37: 100, Resistor_SMD:R_0402_1005Metric_Pad0.72x0.64mm_HandSolder, F.Cu at (149.9, 106.9)
- added R38: 4.7k, Resistor_SMD:R_0402_1005Metric_Pad0.72x0.64mm_HandSolder, B.Cu at (40.6, 108.8)
- added R4: 100, Resistor_SMD:R_0402_1005Metric_Pad0.72x0.64mm_HandSolder, B.Cu at (70.2, 55.4)
- added R5: 100, Resistor_SMD:R_0402_1005Metric_Pad0.72x0.64mm_HandSolder, B.Cu at (71.7, 72.1)
- added R6: 100, Resistor_SMD:R_0402_1005Metric_Pad0.72x0.64mm_HandSolder, B.Cu at (73.1, 88.8)
- added R7: 100, Resistor_SMD:R_0402_1005Metric_Pad0.72x0.64mm_HandSolder, B.Cu at (89.1, 50.5)
- added R8: 100, Resistor_SMD:R_0402_1005Metric_Pad0.72x0.64mm_HandSolder, B.Cu at (90.5, 67.3)
- added R9: 100, Resistor_SMD:R_0402_1005Metric_Pad0.72x0.64mm_HandSolder, B.Cu at (92.0, 83.9)
- added SW1: PowerSwitch, Button_Switch_SMD:SW_SPDT_PCM12, F.Cu at (171.9, 68.5)
- added SW2: PowerSwitch, Button_Switch_SMD:SW_SPDT_PCM12, B.Cu at (171.9, 68.5)
- added SW3: BUTTON-4P, Keyboard:SW4-SMD-2.8-2.6X1.6X0.53MM, B.Cu at (149.0, 132.4)
- added SW4: BUTTON-4P, Keyboard:SW4-SMD-2.8-2.6X1.6X0.53MM, F.Cu at (149.0, 132.4)
- added U1: ~, Keyboard:Solder Nut, F.Cu at (67.5, 108.1)
- added U7: Seeeduino Xiao nRF52840, Keyboard:XIAO-nRF52840-Sense-14P-2.54-21X17.8MM, F.Cu at (143.1, 132.4)
- added U8: Seeeduino Xiao nRF52840, Keyboard:XIAO-nRF52840-Sense-14P-2.54-21X17.8MM, B.Cu at (143.1, 132.4)
- added U9: ~, Art:Salt, B.Cu at (108.7, 122.7)
- CH1, CH10, CH11, CH12, CH13, CH14, CH15, CH16, CH17, CH18, CH2, CH3, CH4, CH5, CH6, CH7, CH8, CH9: footprint keyswitches:Kailh_socket_PG1350_reversible -> Keyboard:Kailh_HS_Socket; moved to B.Cu
- U2, U3, U4, U5: footprint MountingHole:MountingHole_2.2mm_M2 -> Keyboard:Solder Nut
- U6: footprint MountingHole:MountingHole_2.2mm_M2 -> Art:Salt
- moved TP1 147.3 mm to (46.2, 108.4), turned to 0 degrees
- moved TP2 146.0 mm to (51.8, 108.4), turned to 0 degrees
- moved U4 95.7 mm to (128.2, 139.9)
- moved U2 70.9 mm to (153.4, 60.8)
- moved U6 46.6 mm to (108.8, 122.7)
- moved CH16 28.2 mm to (162.6, 85.5), turned to 155 degrees
- moved U5 27.8 mm to (68.7, 139.9)
- moved CH17 27.8 mm to (155.5, 100.7), turned to 155 degrees
- moved CH18 27.4 mm to (148.4, 115.9), turned to 155 degrees
- moved CH13 26.0 mm to (136.6, 62.9), turned to 175 degrees
- moved U3 25.8 mm to (100.5, 47.4)
- moved CH14 25.8 mm to (135.1, 79.6), turned to 175 degrees
- moved CH15 25.6 mm to (133.7, 96.3), turned to 175 degrees
- moved CH10 24.9 mm to (114.6, 56.7), turned to 180 degrees
- moved CH11 24.7 mm to (114.6, 73.5), turned to 180 degrees
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Connections:
- net Net-(U1-P0.03) renamed COL5
- net Net-(U1-P0.04) renamed COL2
- net Net-(U1-P0.05) renamed COL1
- net Net-(U1-P0.28) renamed COL4
- net Net-(U1-P0.29) renamed COL3
- net Net-(U1-P1.11) renamed COL0
- TP2 pad 1: Net-(SW1-C) -> BAT+
Routing:
- net Net-(D1-K): track 296.6 -> 0.00 mm, vias 7 -> 0
- net Net-(D11-K): track 236.5 -> 0.00 mm, vias 7 -> 0
- net Net-(D12-K): track 178.6 -> 0.00 mm, vias 7 -> 0
- net COL0: track 166.8 -> 0.00 mm, vias 6 -> 0
- net COL1: track 162.4 -> 0.00 mm, vias 4 -> 0
- net COL2: track 144.5 -> 0.00 mm, vias 4 -> 0
- net COL3: track 128.4 -> 0.00 mm, vias 4 -> 0
- net GND: track 123.5 -> 6.31 mm, vias 24 -> 1
- net Net-(SW1-B): track 111.3 -> 0.00 mm, vias 3 -> 0
- net COL4: track 109.7 -> 0.00 mm, vias 4 -> 0
- net COL5: track 95.0 -> 0.00 mm, vias 6 -> 0
- net Net-(D8-A): track 27.2 -> 0.00 mm, vias 2 -> 0
- net Net-(D10-A): track 27.2 -> 0.00 mm, vias 2 -> 0
- net Net-(D17-A): track 27.2 -> 0.00 mm, vias 2 -> 0
- net Net-(D16-A): track 27.2 -> 0.00 mm, vias 2 -> 0
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Other:
- board text removed: "+"
- board text removed: "-"
- board text removed: "O"
- board text removed: "|"

Commit message: add changes
Parts:
- moved Q1 108.7 mm to (145.0, 88.8), turned to 65 degrees
- moved Q2 108.7 mm to (145.0, 88.8), turned to 65 degrees
- moved R38 104.8 mm to (143.9, 91.1), turned to -25 degrees
- moved R19 104.8 mm to (143.9, 91.1), turned to 155 degrees
- moved TP1 84.9 mm to (128.2, 130.6)
- moved TP2 78.2 mm to (128.2, 125.4)
Connections:
- U7 pad 11: LEDTrigger -> LEDTrig
- U8 pad 11: LEDTrigger -> LEDTrig
