File: pcb/pipar_sool/pipar_sool.kicad_pcb (KiCad board)
At the start: 2 copper layers, 142.4 x 110.5 mm, 181 parts, among them Q1 AO3416 N-channel MOSFET, Q2 AO3416 N-channel MOSFET, SW1 PowerSwitch, SW2 PowerSwitch, SW3 BUTTON-4P, SW4 BUTTON-4P, U7 Seeeduino Xiao nRF52840, U8 Seeeduino Xiao nRF52840

Commit message: Remove obsolete files and update KiCad project settings for compatibility
Parts:
- H3: moved to F.Cu
- U6, U9: footprint Art:Salt -> Art:Salt-smallest
- moved U9 28.3 mm to (84.1, 136.7), turned to -145 degrees
- moved U6 28.3 mm to (84.1, 136.7), turned to 35 degrees
- moved R38 15.9 mm to (140.8, 106.6)
- moved R19 15.9 mm to (140.8, 106.6)
- moved Q1 15.9 mm to (141.8, 104.3)
- moved Q2 15.9 mm to (141.8, 104.3)
- moved TP1 5.11 mm to (130.7, 135.0)
- moved TP2 5.11 mm to (130.7, 129.9)
- moved D16 3.42 mm to (158.3, 79.2)
- moved LED10 3.42 mm to (114.7, 48.7)
- moved R31 3.42 mm to (114.7, 83.7)
- moved D32 3.42 mm to (128.4, 76.2)
- moved LED35 3.42 mm to (160.2, 92.6)
- moved CH19 3.42 mm to (53.2, 146.5)
- moved H4 3.42 mm to (73.1, 61.5)
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Routing:
- net 3V3: track 0.00 -> 508.1 mm, vias 0 -> 19
- net LEDOut: track 0.00 -> 420.0 mm, vias 0 -> 26
- net ROW0: track 0.00 -> 310.8 mm, vias 0 -> 11
- net ROW1: track 0.00 -> 273.7 mm, vias 0 -> 12
- net ROW2: track 0.00 -> 238.7 mm, vias 0 -> 13
- net BAT+: track 0.00 -> 194.1 mm, vias 0 -> 14
- net COL0: track 0.00 -> 155.8 mm, vias 0 -> 5
- net COL1: track 0.00 -> 149.7 mm, vias 0 -> 9
- net COL2: track 0.00 -> 135.6 mm, vias 0 -> 13
- net COL3: track 0.00 -> 118.8 mm, vias 0 -> 13
- net COL4: track 0.00 -> 105.9 mm, vias 0 -> 13
- net GND: track 6.31 -> 96.8 mm, vias 1 -> 83
- net COL5: track 0.00 -> 82.9 mm, vias 0 -> 13
- net LEDTrig: track 3.44 -> 48.0 mm, vias 0 -> 3
- net 5V: track 0.00 -> 17.7 mm, vias 0 -> 1
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
Commit message: Clean up board
Parts:
- moved U9 90.9 mm to (150.8, 74.9), turned to 135 degrees
- moved U6 90.9 mm to (150.8, 74.9), turned to -45 degrees
- moved U1 4.20 mm to (74.2, 109.5)
- moved U5 2.96 mm to (74.2, 142.0)
- moved U2 2.50 mm to (156.7, 65.4)
- moved CH21 1.16 mm to (83.4, 126.5)
- moved H3 1.16 mm to (82.6, 121.1)
- moved CH3 1.16 mm to (87.5, 123.6)
- moved H7 1.15 mm to (93.0, 57.1)
- moved R11 1.15 mm to (115.8, 67.3)
- moved CH32 1.15 mm to (133.8, 81.8)
- moved SW4 1.15 mm to (152.6, 135.0)
- moved LED29 1.15 mm to (115.8, 65.8)
- moved CH12 1.15 mm to (118.2, 92.8)
- moved CH14 1.15 mm to (138.8, 82.3)
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- renumbered R20 to R19, R21 to R20, R22 to R21, R23 to R22, R24 to R23, R25 to R24, R26 to R25, R27 to R26, R28 to R27, R29 to R28, R30 to R29, R31 to R30, R32 to R31, R33 to R32, R34 to R33, R35 to R34, R36 to R35, R37 to R36, R19 to R39, R38 to R40
Connections:
- SW1 pad 1: BAT+ -> +4V
- SW2 pad 1: BAT+ -> +4V
- U7 pad 16: BAT+ -> +4V
- U8 pad 16: BAT+ -> +4V
Routing:
- net +4V: track 0.00 -> 111.0 mm, vias 0 -> 7
- net BAT+: track 194.1 -> 83.2 mm, vias 14 -> 7
- net COL0: track 155.8 -> 160.7 mm
- net 3V3: track 508.1 -> 512.0 mm
- net ROW0: track 310.8 -> 313.7 mm
- net ROW2: track 238.7 -> 241.4 mm
- net ROW1: track 273.7 -> 276.3 mm
- net COL1: track 149.7 -> 152.2 mm
Other:
- board text added: "+"
- board text added: "-"

Commit message: further improvments and cleanup
Parts:
- added U10: ~, Fiducial:Fiducial_0.5mm_Mask1.5mm, F.Cu at (40.6, 140.8)
- added U11: ~, Fiducial:Fiducial_0.5mm_Mask1.5mm, F.Cu at (181.0, 72.3)
- added U12: ~, Fiducial:Fiducial_0.5mm_Mask1.5mm, B.Cu at (40.6, 140.8)
- added U13: ~, Fiducial:Fiducial_0.5mm_Mask1.5mm, B.Cu at (181.0, 72.3)
- added U14: ~, Fiducial:Fiducial_0.5mm_Mask1.5mm, B.Cu at (63.0, 54.7)
- added U15: ~, Fiducial:Fiducial_0.5mm_Mask1.5mm, F.Cu at (63.0, 54.7)
- moved SW1 4.85 mm to (171.2, 68.9)
- moved SW2 4.85 mm to (171.2, 68.9)
- moved U6 0.15 mm to (150.9, 74.8)
- moved U9 0.15 mm to (150.9, 74.8)
Routing:
- net +4V: track 111.0 -> 105.8 mm
- net BAT+: track 83.2 -> 79.1 mm
- net GND: vias 83 -> 80
- net (no net): vias 4 -> 0
Other:
- board text added: "Pipar & Sool V3"
