File: pcb/pipar_sool/pipar_sool.kicad_pcb (KiCad board)
At the start: 2 copper layers, 142.4 x 110.5 mm, 187 parts, among them Q1 AO3416 N-channel MOSFET, Q2 AO3416 N-channel MOSFET, SW1 PowerSwitch, SW2 PowerSwitch, SW3 BUTTON-4P, SW4 BUTTON-4P, U7 Seeeduino Xiao nRF52840, U8 Seeeduino Xiao nRF52840

Commit message: fill zone improvements
Parts:
- moved U9 89.2 mm to (86.5, 136.5), turned to -145 degrees
- moved U6 89.2 mm to (86.5, 136.5), turned to 35 degrees
- moved U2 0.80 mm to (157.4, 65.7)
- moved R8 0.80 mm to (95.0, 70.1)
- moved H16 0.80 mm to (166.8, 82.9)
- moved CH2 0.80 mm to (73.7, 134.1)
- moved LED7 0.80 mm to (93.4, 51.9)
- moved SW4 0.80 mm to (153.4, 135.2)
- moved LED12 0.80 mm to (116.5, 82.8)
- moved LED35 0.80 mm to (162.0, 93.2)
- moved R6 0.80 mm to (77.6, 91.6)
- moved LED2 0.80 mm to (65.8, 127.0)
- moved D29 0.80 mm to (109.2, 71.5)
- moved U4 0.80 mm to (132.5, 142.3)
- moved CH30 0.80 mm to (114.0, 93.0)
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Routing:
- net 3V3: track 512.0 -> 638.7 mm, vias 19 -> 26
- net GND: track 96.8 -> 187.3 mm, vias 80 -> 40
- net COL0: track 160.7 -> 167.0 mm, vias 5 -> 7
- net ROW0: vias 11 -> 9
- net ROW1: vias 12 -> 10
- net ROW2: vias 13 -> 11
- added copper zone on F.Cu, net 3V3
- removed copper zone on F.Cu, net GND
