File: pcb/pipar_sool/PnP.kicad_sch (KiCad schematic)
At the start: 5 parts, among them Q2 AO3416 N-channel MOSFET, SW2 PowerSwitch, SW4 BUTTON-4P, U8 Seeeduino Xiao nRF52840

Commit message: add changes
Connections:
- net LEDTrigger is gone; now on net LEDTrig: U8.11 (P1.15)
Changed lines of the file:
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@@
 		)
 	)
-	(global_label "LEDTrigger"
+	(global_label "LEDTrig"
 		(shape input)
 		(at 83.82 33.02 0)
@@
 		)
 		(property "Intersheetrefs" "${INTERSHEET_REFS}"
-			(at 92.4295 33.02 0)
+			(at 93.7599 33.02 0)
 			(effects
 				(font

Commit message: Clean up board
Parts:
- renumbered R38 to R40
Connections:
- net BAT+: no longer SW2.1 (B), U8.16 (BAT+)
- new net +4V: SW2.1 (B), U8.16 (BAT+)
