File: pcb/pipar_chip/pipar_chip.kicad_pcb (KiCad board)
At the start: 4 copper layers, 68 x 61.3 mm, 87 parts, among them IC1 MCP1700T-3302E_MAY, J1 Conn_02x03_Odd_Even, J2 USB_C_Receptacle_USB2.0_14P, Q1 AO3400A, SW1 EVP-BB1AAB000, SW2 SW_SPDT, U1 ESDR0502NMUTAG, U2 nPM1100-QDXX, U3 ISP1807-LR-RS

Commit message: update the ESD component to be in bom
Parts:
- added REF**: Solder Nut, Keyboard:Solder Nut, B.Cu at (110.1, 70.4)
Changed lines of the file:
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@@
 		(allow_soldermask_bridges_in_footprints no)
 		(tenting front back)
+		(aux_axis_origin 51.52 88)
+		(grid_origin 51.52 88)
 		(pcbplotparams
 			(layerselection 0x00000000_00000000_55555555_5755f5ff)
@@
 		(sheetname "/")
 		(sheetfile "pipar_chip.kicad_sch")
-		(attr exclude_from_bom)
 		(fp_circle
 			(center -0.75 -0.41)
@@
 		(embedded_fonts no)
 	)
+	(footprint "Keyboard:Solder Nut"
+		(layer "B.Cu")
+		(at 110.12 70.44 180)
+		(property "Reference" "REF**"
+			(at 0 0.5 0)
+			(unlocked yes)
+			(layer "B.SilkS")
+			(effects
+				(font
+					(size 1 1)
+					(thickness 0.1)
+				)
+				(justify mirror)
+			)
+		)
+		(property "Value" "Solder Nut"
+			(at 0 -1 0)
+			(unlocked yes)
+			(layer "B.Fab")
+			(effects
+				(font
+					(size 1 1)
+					(thickness 0.15)
+				)
+				(justify mirror)
+			)
+		)
+		(property "Datasheet" ""
+			(at 0 0 0)
+			(unlocked yes)
+			(layer "B.Fab")
+			(hide yes)
+			(effects
+				(font
+					(size 1 1)
+					(thickness 0.15)
+				)
+				(justify mirror)
+			)
+		)
+		(property "Description" ""
+			(at 0 0 0)
+			(unlocked yes)
+			(layer "B.Fab")
+			(hide yes)
+			(effects
+				(font
+					(size 1 1)
+					(thickness 0.15)
+				)
+				(justify mirror)
+			)
+		)
+		(attr through_hole)
+		(fp_text user "${REFERENCE}"
+			(at 0 -2.5 0)
+			(unlocked yes)
+			(layer "B.Fab")
+			(effects
+				(font
+					(size 1 1)
+					(thickness 0.15)
+				)
+				(justify mirror)
+			)
+		)
+		(pad "1" thru_hole circle
+			(at 0 0 180)
+			(size 4.7 4.7)
+			(drill 3.1)
+			(layers "*.Cu" "*.Mask")
+			(remove_unused_layers no)
+		)
+		(embedded_fonts no)
+	)
 	(footprint "TestPoint:TestPoint_Pad_D1.0mm"
 		(layer "B.Cu")
@@
 	)
 	(segment
-		(start 86.05 33.11)
-		(end 89.09 36.15)
-		(width 0.2032)
-		(layer "F.Cu")
-		(net 26)
-	)
-	(segment
 		(start 75.595 35.495)
 		(end 74.594998 36.495002)
@@
 	)
 	(segment
-		(start 89.09 36.15)
-		(end 89.65 36.15)
-		(width 0.2032)
+		(start 72.377487 36.650005)
+		(end 74.034996 36.650005)
+		(width 0.3048)
 		(layer "F.Cu")
 		(net 26)
 	)
 	(segment
-		(start 72.377487 36.650005)
-		(end 74.034996 36.650005)
-		(width 0.3048)
+		(start 89.65 36.91)
+		(end 85.85 33.11)
+		(width 0.2032)
 		(layer "F.Cu")
 		(net 26)
@@
 	(segment
 		(start 77.98 33.11)
-		(end 86.05 33.11)
+		(end 75.595 35.495)
 		(width 0.2032)
 		(layer "F.Cu")
@@
 	)
 	(segment
-		(start 75.595 35.495)
+		(start 85.85 33.11)
 		(end 77.98 33.11)
 		(width 0.2032)
@@
 	)
 	(via
-		(at 89.65 36.15)
+		(at 89.65 36.91)
 		(size 0.6)
 		(drill 0.3)
@@
 	(segment
 		(start 109.77 33.75)
-		(end 109.77 37.79)
-		(width 0.2032)
-		(layer "B.Cu")
-		(net 26)
-	)
-	(segment
-		(start 113.018575 31.95)
 		(end 111.57 31.95)
 		(width 0.2032)
@@
 	)
 	(segment
-		(start 116.795001 33.766497)
-		(end 116.342397 33.313893)
+		(start 109.77 37.79)
+		(end 109.77 33.75)
 		(width 0.2032)
 		(layer "B.Cu")
@@
 	)
 	(segment
-		(start 116.342397 33.313893)
-		(end 114.382468 33.313893)
+		(start 91.726008 38.986008)
+		(end 108.573992 38.986008)
 		(width 0.2032)
 		(layer "B.Cu")
@@
 	)
 	(segment
-		(start 111.57 31.95)
-		(end 109.77 33.75)
+		(start 114.382468 33.313893)
+		(end 116.342397 33.313893)
 		(width 0.2032)
 		(layer "B.Cu")
@@
 	)
 	(segment
-		(start 89.65 36.91)
-		(end 89.65 36.15)
+		(start 116.342397 33.313893)
+		(end 116.795001 33.766497)
 		(width 0.2032)
 		(layer "B.Cu")
@@
 	)
 	(segment
-		(start 114.382468 33.313893)
+		(start 111.57 31.95)
 		(end 113.018575 31.95)
 		(width 0.2032)
@@
 	)
 	(segment
-		(start 91.726008 38.986008)
-		(end 89.65 36.91)
+		(start 113.018575 31.95)
+		(end 114.382468 33.313893)
 		(width 0.2032)
 		(layer "B.Cu")
@@
 	(segment
 		(start 108.573992 38.986008)
-		(end 91.726008 38.986008)
+		(end 109.77 37.79)
 		(width 0.2032)
 		(layer "B.Cu")
@@
 	)
 	(segment
-		(start 109.77 37.79)
-		(end 108.573992 38.986008)
+		(start 89.65 36.91)
+		(end 91.726008 38.986008)
 		(width 0.2032)
 		(layer "B.Cu")
