File: pcb/pipar_chip/keymatrix.kicad_sch (KiCad schematic)
At the start: 40 parts, among them Q1 AO3400A

Commit message: Pipar Point V3.1
Parts:
- R11: value 1.5k -> 100R
Other:
- note added: "R * N Leds 100R * 12 = 1.2kR per led"
- note removed: "100R * N Leds"
Changed lines of the file:
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@@
 		)
 	)
-	(text "100R * N Leds"
+	(text "R * N Leds\n100R * 12 = 1.2kR per led"
 		(exclude_from_sim no)
-		(at 81.026 80.772 0)
+		(at 74.676 79.502 0)
 		(effects
 			(font
@@
 			)
 		)
-		(property "Value" "1.5k"
+		(property "Value" "100R"
 			(at 86.36 85.0899 0)
 			(effects
