File: pcb/pipar_chip/pipar_chip.kicad_sch (KiCad schematic)
At the start: 47 parts, among them IC1 MCP1700T-3302E_MAY, J1 Conn_02x03_Odd_Even, J2 USB_C_Receptacle_USB2.0_14P, SW1 EVP-BB1AAB000, SW2 SW_SPDT, U1 ESDR0502NMUTAG, U2 nPM1100-QDXX, U3 ISP1807-LR-RS

Commit message: Pipar Point V3.1
Parts:
- added R7, R8: 1.5k, Resistor_SMD:R_0603_1608Metric, symbol Device:R_Small
Connections:
- net VSYS: now also R7.2, R8.2; no longer D3.2 (A), D4.2 (A)
- new net: D3.2 (A), R7.1
- new net: D4.2 (A), R8.1
Other:
- moved on the sheet: D3, D4
