File: pcb/pipar_point_v3/pipar_point_v3.kicad_pcb (KiCad board)
At the start: 4 copper layers, 253 parts, among them IC1 MCP1700T-3302E_MAY, IC2 MCP1700T-3302E_MAY, J1 USB_C_Receptacle_USB2.0_16P, J2 USB_C_Receptacle_USB2.0_16P, J3 Conn_02x03_Odd_Even, J4 Conn_02x03_Odd_Even, Q1 AO3400A, Q2 AO3400A, SW1 EVP-BB1AAB000, SW2 EVP-BB1AAB000, SW3 SW_SPDT, SW4 SW_SPDT, U1 ISP1807-LR-RS, U2 ISP1807-LR-RS, U3 MAX17048, U4 ESDR0502NMUTAG, U5 nPM1100-QDXX, U6 MAX17048, U7 ESDR0502NMUTAG, U8 nPM1100-QDXX

Commit message: places more components
Parts:
- added R21: 1.5k, Resistor_SMD:R_0603_1608Metric, F.Cu at (65.0, 112.9)
- added R22: 1.5k, Resistor_SMD:R_0603_1608Metric, F.Cu at (161.5, -44.1)
- added R23: 1.5k, Resistor_SMD:R_0603_1608Metric, F.Cu at (65.0, 115.4)
- added R24: 1.5k, Resistor_SMD:R_0603_1608Metric, F.Cu at (159.8, -44.1)
- moved Q2 93.2 mm to (178.2, -9.36)
- moved R13 93.2 mm to (175.4, -9.36)
- moved R14 93.2 mm to (181.8, -9.36)
- moved C12 71.1 mm to (159.3, -35.4)
- moved U6 70.4 mm to (161.7, -36.2)
- moved C19 51.0 mm to (159.2, -40.8)
- moved C20 51.0 mm to (164.2, -40.8)
- moved IC2 51.0 mm to (161.7, -40.8)
- moved D23 43.8 mm to (161.5, -47.1), turned to -90 degrees
- moved D24 41.4 mm to (159.8, -47.1), turned to -90 degrees
- moved R10 41.3 mm to (165.9, -48.0)
- moved SW4 40.7 mm to (183.8, -67.8), turned to 180 degrees
- moved R12 36.0 mm to (165.9, -49.5), turned to 180 degrees
- moved R11 35.8 mm to (163.9, -46.3), turned to 180 degrees
- moved C15 34.1 mm to (165.1, -53.2), turned to 90 degrees
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Connections:
- net /Side-Right/3.3V renamed /Side-RightDup/3.3V
- net /Side-Right/3VOUT renamed /Side-RightDup/3VOUT
- net /Side-Right/BAT_SCL renamed /Side-RightDup/BAT_SCL
- net /Side-Right/BAT_SDA renamed /Side-RightDup/BAT_SDA
- net /Side-Right/Backlight renamed /Side-RightDup/Backlight
- net /Side-Right/Col0 renamed /Side-RightDup/Col0
- net /Side-Right/Col1 renamed /Side-RightDup/Col1
- net /Side-Right/Col2 renamed /Side-RightDup/Col2
- net /Side-Right/Col3 renamed /Side-RightDup/Col3
- net /Side-Right/Col4 renamed /Side-RightDup/Col4
- net /Side-Right/Col5 renamed /Side-RightDup/Col5
- net /Side-Right/Col6 renamed /Side-RightDup/Col6
- net /Side-Right/Key Matrix/LEDOut renamed /Side-RightDup/Key Matrix/LEDOut
- net /Side-Right/LED_1 renamed /Side-RightDup/LED_1
- net /Side-Right/LED_2 renamed /Side-RightDup/LED_2
- net /Side-Right/LED_3 renamed /Side-RightDup/LED_3
- net /Side-Right/Power/CC1 renamed /Side-RightDup/Power/CC1
- net /Side-Right/Power/CC2 renamed /Side-RightDup/Power/CC2
- net /Side-Right/Power/FUEL_ALRT renamed /Side-RightDup/Power/FUEL_ALRT
- net /Side-Right/Power/LChg renamed /Side-RightDup/Power/LChg
- net /Side-Right/Power/LError renamed /Side-RightDup/Power/LError
- net /Side-Right/Power/VBAT renamed /Side-RightDup/Power/VBAT
- net /Side-Right/RESET renamed /Side-RightDup/RESET
- net /Side-Right/Row0 renamed /Side-RightDup/Row0
- net /Side-Right/Row1 renamed /Side-RightDup/Row1
- net /Side-Right/Row2 renamed /Side-RightDup/Row2
- net /Side-Right/SWDCLK renamed /Side-RightDup/SWDCLK
- net /Side-Right/SWDIO renamed /Side-RightDup/SWDIO
- net /Side-Right/VBUS renamed /Side-RightDup/VBUS
- C18 pad 2: /Side-Right/Power/VSYS -> /Side-RightDup/Power/VSYS
- C19 pad 2: /Side-Right/Power/VSYS -> /Side-RightDup/Power/VSYS
- D21 pad 2: /Side-Left/Power/VSYS -> Net-(D21-A)
- D22 pad 2: /Side-Left/Power/VSYS -> Net-(D22-A)
- D23 pad 2: /Side-Right/Power/VSYS -> Net-(D23-A)
- D24 pad 2: /Side-Right/Power/VSYS -> Net-(D24-A)
- IC2 pad 1: /Side-Right/Power/VSYS -> /Side-RightDup/Power/VSYS
- J2 pad A6: /Side-Right/USB_D+ -> /Side-RightDup/USB_D+
- J2 pad A7: /Side-Right/USB_D- -> /Side-RightDup/USB_D-
- J2 pad B6: /Side-Right/USB_D+ -> /Side-RightDup/USB_D+
- J2 pad B7: /Side-Right/USB_D- -> /Side-RightDup/USB_D-
- TP15 pad 1: /Side-Right/Power/VSYS -> /Side-RightDup/Power/VSYS
- U2 pad 10: /Side-Right/USB_D- -> /Side-RightDup/USB_D-
- U2 pad 8: /Side-Right/USB_D+ -> /Side-RightDup/USB_D+
- U4 pad 2: /Side-Left/USB_D+ -> unconnected-(U4-NC-Pad2)
- U4 pad 3: /Side-Left/USB_D- -> unconnected-(U4-NC-Pad3)
- U7 pad 2: /Side-Right/USB_D+ -> unconnected-(U7-NC-Pad2)
- U7 pad 3: /Side-Right/USB_D- -> unconnected-(U7-NC-Pad3)
- U7 pad 4: /Side-Right/USB_D- -> /Side-RightDup/USB_D-
- U7 pad 5: /Side-Right/USB_D+ -> /Side-RightDup/USB_D+
- U8 pad 16: /Side-Right/Power/VSYS -> /Side-RightDup/Power/VSYS
- U8 pad 19: /Side-Right/USB_D- -> /Side-RightDup/USB_D-
- U8 pad 2: /Side-Right/Power/VSYS -> /Side-RightDup/Power/VSYS
- U8 pad 20: /Side-Right/USB_D+ -> /Side-RightDup/USB_D+
- U8 pad 3: /Side-Right/Power/VSYS -> /Side-RightDup/Power/VSYS
- U8 pad 5: /Side-Right/Power/VSYS -> /Side-RightDup/Power/VSYS
Routing:
- net /Side-RightDup/Power/VSYS: track 0.00 -> 18.1 mm, vias 0 -> 1
- net /Side-RightDup/3VOUT: track 0.00 -> 6.71 mm
- net Net-(U8-SW): track 0.00 -> 3.34 mm
- net Net-(U8-ICHG): track 0.00 -> 3.12 mm
- net Net-(U8-NTC): track 0.00 -> 2.17 mm
- net /Side-RightDup/Power/LChg: track 0.00 -> 1.93 mm
- net Net-(U8-DEC): track 0.00 -> 1.80 mm
- net GND: track 0.65 -> 2.45 mm
- net /Side-RightDup/Power/VBAT: track 0.00 -> 1.75 mm
- net /Side-RightDup/Power/LError: track 0.00 -> 1.66 mm
- net /Side-RightDup/VBUS: track 2.02 -> 3.64 mm
- net Net-(R10-Pad2): track 0.00 -> 1.52 mm
- net Net-(D24-A): track 0.00 -> 1.42 mm
- net Net-(D23-A): track 0.00 -> 1.42 mm

Commit message: Refactor schematic connections and add hierarchical labels
- Removed redundant no_connect entries and updated UUIDs for clarity.
- Added new no_connect entries at specified coordinates.
- Introduced hierarchical labels for "3.3V", "TPClock", "TPData", and "TPRST" with appropriate formatting and positioning.
Parts:
- added U10: ~, Trackpoint:SK8707-01-0C Sensor, B.Cu at (250.9, -24.6)
- added U9: ~, Trackpoint:SK8707-01, B.Cu at (199.8, -4.71)
Connections:
- net /Side-RightDup/3.3V renamed /Side-Right/3.3V
- net /Side-RightDup/3VOUT renamed /Side-Right/3VOUT
- net /Side-RightDup/BAT_SCL renamed /Side-Right/BAT_SCL
- net /Side-RightDup/BAT_SDA renamed /Side-Right/BAT_SDA
- net /Side-RightDup/Backlight renamed /Side-Right/Backlight
- net /Side-RightDup/Col0 renamed /Side-Right/Col0
- net /Side-RightDup/Col1 renamed /Side-Right/Col1
- net /Side-RightDup/Col2 renamed /Side-Right/Col2
- net /Side-RightDup/Col3 renamed /Side-Right/Col3
- net /Side-RightDup/Col4 renamed /Side-Right/Col4
- net /Side-RightDup/Col5 renamed /Side-Right/Col5
- net /Side-RightDup/Col6 renamed /Side-Right/Col6
- net /Side-RightDup/Key Matrix/LEDOut renamed /Side-Right/Key Matrix/LEDOut
- net /Side-RightDup/LED_1 renamed /Side-Right/LED_1
- net /Side-RightDup/LED_2 renamed /Side-Right/LED_2
- net /Side-RightDup/LED_3 renamed /Side-Right/LED_3
- net /Side-RightDup/Power/CC1 renamed /Side-Right/Power/CC1
- net /Side-RightDup/Power/CC2 renamed /Side-Right/Power/CC2
- net /Side-RightDup/Power/FUEL_ALRT renamed /Side-Right/Power/FUEL_ALRT
- net /Side-RightDup/Power/LChg renamed /Side-Right/Power/LChg
- net /Side-RightDup/Power/LError renamed /Side-Right/Power/LError
- net /Side-RightDup/Power/VBAT renamed /Side-Right/Power/VBAT
- net /Side-RightDup/Power/VSYS renamed /Side-Right/Power/VSYS
- net /Side-RightDup/RESET renamed /Side-Right/RESET
- net /Side-RightDup/Row0 renamed /Side-Right/Row0
- net /Side-RightDup/Row1 renamed /Side-Right/Row1
- net /Side-RightDup/Row2 renamed /Side-Right/Row2
- net /Side-RightDup/SWDCLK renamed /Side-Right/SWDCLK
- net /Side-RightDup/SWDIO renamed /Side-Right/SWDIO
- net /Side-RightDup/USB_D+ renamed /Side-Right/USB_D+
- net /Side-RightDup/USB_D- renamed /Side-Right/USB_D-
- net /Side-RightDup/VBUS renamed /Side-Right/VBUS
- U1 pad 2: unconnected-(U1A-P0_09_NFC1-Pad2) -> /Side-Left/TPRST
- U1 pad 3: unconnected-(U1A-P0_12_TRACEDATA1-Pad3) -> /Side-Left/TPData
- U1 pad 5: unconnected-(U1A-P0_14-Pad5) -> /Side-Left/TPClock
- U2 pad 2: unconnected-(U2A-P0_09_NFC1-Pad2) -> /Side-Right/TPRST
- U2 pad 3: unconnected-(U2A-P0_12_TRACEDATA1-Pad3) -> /Side-Right/TPData
- U2 pad 5: unconnected-(U2A-P0_14-Pad5) -> /Side-Right/TPClock
