File: pcb/pipar_point_v3/side.kicad_sch (KiCad schematic)
At the start: 12 parts, among them J3 Conn_02x03_Odd_Even, SW1 EVP-BB1AAB000, U1 ISP1807-LR-RS

Commit message: updates the pinout for the isp1807
Connections:
- net BAT_SCL: now also U1.34 (P0_06)
- net BAT_SDA: now also U1.32 (P0_08)
- net Backlight: now also U1.61 (P1_11)
- net Col0: now also U1.48 (P0_28_AIN4)
- net Col1: now also U1.46 (P0_29_AIN5)
- net Col2: now also U1.44 (P0_30_AIN6)
- net Col3: now also U1.42 (P0_31_AIN7)
- net Col4: now also U1.40 (P0_02_AIN0)
- net Col5: now also U1.38 (P0_03_AIN1)
- net Col6: now also U1.36 (P0_05_AIN3)
- net LED_1: now also U1.52 (P1_14)
- net LED_2: now also U1.59 (P1_12)
- net LED_3: now also U1.50 (P1_06)
- net Row0: now also U1.56 (P1_09_TRACEDATA3)
- net Row1: now also U1.63 (P1_04)
- net Row2: now also U1.54 (P1_05)
- no-connect marks 46 -> 29
Changed lines of the file:
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@@
-	)
-	(no_connect
-		(at 143.51 36.83)
-	)
-	(no_connect
-		(at 143.51 85.09)
 	)
 	(no_connect
@@
 	)
 	(no_connect
-		(at 143.51 46.99)
-	)
-	(no_connect
-		(at 143.51 57.15)
-	)
-	(no_connect
 		(at 143.51 82.55)
 	)
@@
 	)
 	(no_connect
-		(at 143.51 31.75)
-	)
-	(no_connect
-		(at 143.51 67.31)
-	)
-	(no_connect
-		(at 143.51 26.67)
-	)
-	(no_connect
 		(at 234.95 49.53)
 	)
@@
 	)
 	(no_connect
-		(at 143.51 87.63)
-	)
-	(no_connect
 		(at 234.95 90.17)
 	)
@@
 	)
 	(no_connect
-		(at 143.51 44.45)
-	)
-	(no_connect
 		(at 143.51 62.23)
 	)
 	(no_connect
-		(at 143.51 92.71)
-	)
-	(no_connect
 		(at 43.18 48.26)
 	)
@@
 	)
 	(no_connect
-		(at 143.51 72.39)
-	)
-	(no_connect
 		(at 234.95 82.55)
 	)
@@
 	)
 	(no_connect
-		(at 234.95 46.99)
-	)
-	(no_connect
 		(at 143.51 64.77)
 	)
@@
 	)
 	(no_connect
-		(at 234.95 39.37)
-	)
-	(no_connect
 		(at 234.95 77.47)
 	)
@@
 	(no_connect
 		(at 234.95 67.31)
-	)
-	(no_connect
-		(at 234.95 41.91)
-	)
-	(no_connect
-		(at 143.51 39.37)
-	)
-	(no_connect
-		(at 143.51 69.85)
-	)
-	(no_connect
-		(at 143.51 80.01)
 	)
 	(no_connect
@@
 		)
 	)
+	(label "Col5"
+		(at 143.51 26.67 180)
+		(effects
+			(font
+				(size 1.27 1.27)
+			)
+			(justify right bottom)
+		)
+	)
 	(label "BAT_SDA"
 		(at 43.18 44.45 0)
@@
 		)
 	)
+	(label "Col6"
+		(at 143.51 31.75 180)
+		(effects
+			(font
+				(size 1.27 1.27)
+			)
+			(justify right bottom)
+		)
+	)
+	(label "BAT_SCL"
+		(at 234.95 41.91 0)
+		(effects
+			(font
+				(size 1.27 1.27)
+			)
+			(justify left bottom)
+		)
+	)
+	(label "Row2"
+		(at 143.51 69.85 180)
+		(effects
+			(font
+				(size 1.27 1.27)
+			)
+			(justify right bottom)
+		)
+	)
 	(label "LED_1"
 		(at 25.4 121.92 90)
@@
 		)
 	)
+	(label "Col3"
+		(at 143.51 46.99 180)
+		(effects
+			(font
+				(size 1.27 1.27)
+			)
+			(justify right bottom)
+		)
+	)
 	(label "Row0"
 		(at 43.18 68.58 0)
@@
 		)
 	)
+	(label "Row0"
+		(at 143.51 80.01 180)
+		(effects
+			(font
+				(size 1.27 1.27)
+			)
+			(justify right bottom)
+		)
+	)
+	(label "LED_3"
+		(at 143.51 72.39 180)
+		(effects
+			(font
+				(size 1.27 1.27)
+			)
+			(justify right bottom)
+		)
+	)
+	(label "Backlight"
+		(at 143.51 85.09 180)
+		(effects
+			(font
+				(size 1.27 1.27)
+			)
+			(justify right bottom)
+		)
+	)
 	(label "LED_2"
 		(at 35.56 121.92 90)
@@
 		)
 	)
+	(label "LED_1"
+		(at 143.51 92.71 180)
+		(effects
+			(font
+				(size 1.27 1.27)
+			)
+			(justify right bottom)
+		)
+	)
 	(label "Col1"
 		(at 43.18 80.01 0)
@@
 		)
 	)
+	(label "Col2"
+		(at 143.51 44.45 180)
+		(effects
+			(font
+				(size 1.27 1.27)
+			)
+			(justify right bottom)
+		)
+	)
 	(label "3VOUT"
 		(at 66.04 24.13 180)
@@
 		)
 	)
+	(label "Row1"
+		(at 143.51 67.31 180)
+		(effects
+			(font
+				(size 1.27 1.27)
+			)
+			(justify right bottom)
+		)
+	)
+	(label "Col1"
+		(at 143.51 39.37 180)
+		(effects
+			(font
+				(size 1.27 1.27)
+			)
+			(justify right bottom)
+		)
+	)
 	(label "VBUS"
 		(at 193.04 139.7 270)
@@
 		)
 	)
+	(label "Col0"
+		(at 143.51 36.83 180)
+		(effects
+			(font
+				(size 1.27 1.27)
+			)
+			(justify right bottom)
+		)
+	)
+	(label "Col4"
+		(at 234.95 39.37 0)
+		(effects
+			(font
+				(size 1.27 1.27)
+			)
+			(justify left bottom)
+		)
+	)
 	(label "Backlight"
 		(at 43.18 96.52 0)
@@
 		)
 	)
+	(label "BAT_SDA"
+		(at 234.95 46.99 0)
+		(effects
+			(font
+				(size 1.27 1.27)
+			)
+			(justify left bottom)
+		)
+	)
+	(label "LED_2"
+		(at 143.51 87.63 180)
+		(effects
+			(font
+				(size 1.27 1.27)
+			)
+			(justify right bottom)
+		)
+	)

Commit message: Refactor schematic connections and add hierarchical labels
- Removed redundant no_connect entries and updated UUIDs for clarity.
- Added new no_connect entries at specified coordinates.
- Introduced hierarchical labels for "3.3V", "TPClock", "TPData", and "TPRST" with appropriate formatting and positioning.
Connections:
- net TPRST: now reaches U1.2 (P0_09_NFC1)
- net TPData: now reaches U1.3 (P0_12_TRACEDATA1)
- net TPClock: now reaches U1.5 (P0_14)
- no-connect marks 29 -> 26
Changed lines of the file:
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@@
+	)
+	(no_connect
+		(at 234.95 87.63)
+	)
+	(no_connect
+		(at 234.95 54.61)
+	)
+	(no_connect
+		(at 143.51 90.17)
+	)
+	(no_connect
+		(at 143.51 97.79)
+	)
+	(no_connect
+		(at 234.95 72.39)
+	)
+	(no_connect
+		(at 143.51 82.55)
+	)
+	(no_connect
+		(at 143.51 29.21)
 	)
 	(no_connect
@@
 	)
 	(no_connect
-		(at 234.95 87.63)
-	)
-	(no_connect
-		(at 234.95 54.61)
-	)
-	(no_connect
-		(at 143.51 90.17)
-	)
-	(no_connect
-		(at 234.95 72.39)
-	)
-	(no_connect
-		(at 143.51 82.55)
-	)
-	(no_connect
-		(at 143.51 97.79)
-	)
-	(no_connect
-		(at 234.95 49.53)
-	)
-	(no_connect
-		(at 143.51 29.21)
-	)
-	(no_connect
 		(at 234.95 90.17)
 	)
@@
 	)
 	(no_connect
-		(at 234.95 59.69)
-	)
-	(no_connect
 		(at 234.95 82.55)
 	)
@@
 	(no_connect
 		(at 143.51 64.77)
-	)
-	(no_connect
-		(at 234.95 64.77)
 	)
 	(no_connect
@@
 		)
 	)
+	(label "3.3V"
+		(at 54.61 53.34 180)
+		(effects
+			(font
+				(size 1.27 1.27)
+			)
+			(justify right bottom)
+		)
+	)
 	(label "SWDIO"
 		(at 143.51 100.33 180)
@@
 		)
 	)
+	(hierarchical_label "3.3V"
+		(shape bidirectional)
+		(at 54.61 53.34 0)
+		(effects
+			(font
+				(size 1.27 1.27)
+			)
+			(justify left)
+		)
+	)
+	(hierarchical_label "TPClock"
+		(shape bidirectional)
+		(at 234.95 64.77 0)
+		(effects
+			(font
+				(size 1.27 1.27)
+			)
+			(justify left)
+		)
+	)
+	(hierarchical_label "TPData"
+		(shape bidirectional)
+		(at 234.95 59.69 0)
+		(effects
+			(font
+				(size 1.27 1.27)
+			)
+			(justify left)
+		)
+	)
+	(hierarchical_label "TPRST"
+		(shape bidirectional)
+		(at 234.95 49.53 0)
+		(effects
+			(font
+				(size 1.27 1.27)
+			)
+			(justify left)
+		)
+	)

Commit message: more things :)
Connections:
- no-connect marks 26 -> 27
Changed lines of the file:
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@@
+	)
+	(no_connect
+		(at 143.51 57.15)
 	)
 	(no_connect

Commit message: right side routed, progress on left side
Parts:
- removed D47: LED_Small, LED_SMD:LED_0603_1608Metric, symbol Device:LED_Small
- removed R17: 1.5k, Resistor_SMD:R_0603_1608Metric, symbol Device:R_Small
- removed TP1: TestPoint_Probe, TestPoint:TestPoint_Pad_D1.0mm, symbol Connector:TestPoint_Probe
Connections:
- net LED_3: no longer names the net of U1.50 (P1_06)
- no-connect marks 27 -> 28

Commit message: Pipar Point PCB done, maybe
Parts:
- added H43, H45, H47, H49, H65: MouseBite, mouse-bite:mouse-bite-3mm-6mm, symbol Mechanical:MountingHole
- added H54, H56, H58, H60, H62: MountingHole, MountingHole:MountingHole_2.2mm_M2, symbol Mechanical:MountingHole
- H41: value MountingHole -> Art-small
