File: pcb/pipar_point_v3/side.kicad_sch (KiCad schematic)
At the start: 19 parts, among them J3 Conn_02x03_Odd_Even, SW1 EVP-BB1AAB000, U1 ISP1807-LR-RS

Commit message: adds a proper battery connector
Parts:
- D45: Mouser Part Number 743-IN-PIS63BTPR -> 743-S63AT5B
- D46: Mouser Part Number 743-IN-PIS63BTPG -> 743-IN-S63AT5G
Changed lines of the file:
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@@
 			)
 		)
-		(property "Mouser Part Number" "743-IN-PIS63BTPR"
+		(property "Mouser Part Number" "743-S63AT5B"
 			(at 25.4 127 90)
 			(effects
@@
 			)
 		)
-		(property "Mouser Part Number" "743-IN-PIS63BTPG"
+		(property "Mouser Part Number" "743-IN-S63AT5G"
 			(at 35.56 127 90)
 			(effects

Commit message: cleaned up traces on right side, updated bom
Parts:
- D45: value LED_Small -> LED_Blue; Manufacturer_Name Inolux -> (none); Manufacturer_Part_Number IN-PIS63BTPR -> IN-S63AT5B
- D46: value LED_Small -> LED_Green; Manufacturer_Name Inolux -> (none); Manufacturer_Part_Number IN-PIS63BTPG -> IN-S63AT5G
- R15, R16: Manufacturer_Name YAGEO -> (none); Mouser Part Number 603-RC0603FR-071K5L -> 603-RC0603FR-071K5L
- SW1: Manufacturer_Name Panasonic -> (none); Mouser Part Number 667-EVP-BB1AAB000 -> 667-EVP-BB1AAB000
- U1: Manufacturer_Name Insight SiP -> (none); Manufacturer_Part_Number ISP1807-LR-RS -> ISP1807-LR-RS
Changed lines of the file:
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@@
 		(on_board yes)
 		(dnp no)
-		(fields_autoplaced yes)
 		(property "Reference" "D45"
 			(at 27.94 125.6664 90)
@@
 			)
 		)
-		(property "Value" "LED_Small"
-			(at 27.94 128.2064 90)
+		(property "Value" "LED_Blue"
+			(at 27.178 127.508 0)
 			(effects
 				(font
@@
 			)
 		)
-		(property "Manufacturer_Name" "Inolux"
+		(property "Manufacturer_Name" ""
 			(at 25.4 127 90)
 			(effects
@@
 			)
 		)
-		(property "Manufacturer_Part_Number" "IN-PIS63BTPR"
+		(property "Manufacturer_Part_Number" "IN-S63AT5B"
 			(at 25.4 127 90)
 			(effects
@@
 		(on_board yes)
 		(dnp no)
-		(fields_autoplaced yes)
 		(property "Reference" "D46"
 			(at 38.1 125.6664 90)
@@
 			)
 		)
-		(property "Value" "LED_Small"
-			(at 38.1 128.2064 90)
+		(property "Value" "LED_Green"
+			(at 37.338 126.238 0)
 			(effects
 				(font
@@
 				)
 				(justify right)
-				(hide yes)
 			)
 		)
@@
 			)
 		)
-		(property "Manufacturer_Name" "Inolux"
+		(property "Manufacturer_Name" ""
 			(at 35.56 127 90)
 			(effects
@@
 			)
 		)
-		(property "Manufacturer_Part_Number" "IN-PIS63BTPG"
+		(property "Manufacturer_Part_Number" "IN-S63AT5G"
 			(at 35.56 127 90)
 			(effects
@@
 			)
 		)
-		(property "Manufacturer_Name" "Insight SiP"
+		(property "Manufacturer_Name" ""
 			(at 157.48 138.43 90)
 			(effects
@@
 			)
 		)
-		(property "Manufacturer_Part_Number" "ISP1807-LR-RS "
+		(property "Manufacturer_Part_Number" "ISP1807-LR-RS"
 			(at 157.48 138.43 90)
 			(effects
@@
 			)
 		)
-		(property "Manufacturer_Name" "Insight SiP"
+		(property "Manufacturer_Name" ""
 			(at 143.51 26.67 0)
 			(effects
@@
 			)
 		)
-		(property "Manufacturer_Part_Number" "ISP1807-LR-RS "
+		(property "Manufacturer_Part_Number" "ISP1807-LR-RS"
 			(at 143.51 26.67 0)
 			(effects
@@
 			)
 		)
-		(property "Mouser Part Number" "667-EVP-BB1AAB000"
+		(property "Mouser Part Number" " 667-EVP-BB1AAB000"
 			(at 271.78 82.55 0)
 			(effects
@@
 			)
 		)
-		(property "Manufacturer_Name" "Panasonic"
+		(property "Manufacturer_Name" ""
 			(at 271.78 87.63 0)
 			(effects
@@
 			)
 		)
-		(property "Manufacturer_Name" "YAGEO"
+		(property "Manufacturer_Name" ""
 			(at 35.56 134.62 0)
 			(effects
@@
 			)
 		)
-		(property "Mouser Part Number" "603-RC0603FR-071K5L "
+		(property "Mouser Part Number" " 603-RC0603FR-071K5L"
 			(at 35.56 134.62 0)
 			(effects
@@
 			)
 		)
-		(property "Manufacturer_Name" "YAGEO"
+		(property "Manufacturer_Name" ""
 			(at 25.4 134.62 0)
 			(effects
@@
 			)
 		)
-		(property "Mouser Part Number" "603-RC0603FR-071K5L "
+		(property "Mouser Part Number" " 603-RC0603FR-071K5L"
 			(at 25.4 134.62 0)
 			(effects

Commit message: stuff, i dont remember
Connections:
- net 3.3V: now also R15.1, R16.1
- net GND: no longer R15.1, R16.1
- net LED_1: now also D45.1 (K); no longer D45.2 (A)
- net LED_2: now also D46.1 (K); no longer D46.2 (A)
- net at R15.2: now also D45.2 (A); no longer D45.1 (K)
- net at R16.2: now also D46.2 (A); no longer D46.1 (K)
Other:
- moved on the sheet: D45, D46
Changed lines of the file:
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@@
-	)
-	(junction
-		(at 35.56 139.7)
-		(diameter 0)
-		(color 0 0 0 0)
 	)
 	(junction
@@
 	(label "BAT_SCL"
 		(at 43.18 41.91 0)
+		(effects
+			(font
+				(size 1.27 1.27)
+			)
+			(justify left bottom)
+		)
+	)
+	(label "3.3V"
+		(at 35.56 139.7 0)
 		(effects
 			(font
@@
 	)
 	(symbol
-		(lib_id "power:GND")
-		(at 35.56 139.7 0)
-		(unit 1)
-		(exclude_from_sim no)
-		(in_bom yes)
-		(on_board yes)
-		(dnp no)
-		(fields_autoplaced yes)
-		(property "Reference" "#PWR045"
-			(at 35.56 146.05 0)
-			(effects
-				(font
-					(size 1.27 1.27)
-				)
-				(hide yes)
-			)
-		)
-		(property "Value" "GND"
-			(at 35.56 144.78 0)
-			(effects
-				(font
-					(size 1.27 1.27)
-				)
-			)
-		)
-		(property "Footprint" ""
-			(at 35.56 139.7 0)
-			(effects
-				(font
-					(size 1.27 1.27)
-				)
-				(hide yes)
-			)
-		)
-		(property "Datasheet" ""
-			(at 35.56 139.7 0)
-			(effects
-				(font
-					(size 1.27 1.27)
-				)
-				(hide yes)
-			)
-		)
-		(property "Description" "Power symbol creates a global label with name \"GND\" , ground"
-			(at 35.56 139.7 0)
-			(effects
-				(font
-					(size 1.27 1.27)
-				)
-				(hide yes)
-			)
-		)
-		(pin "1"
-		)
-		(instances
-			(project "pipar_point_v3"
-				(path "/ae2abdf3-be75-4a01-9d2e-db16842fefd9/a463a46f-5d6b-469c-a0de-58044b881b04"
-					(reference "#PWR045")
-					(unit 1)
-				)
-				(path "/ae2abdf3-be75-4a01-9d2e-db16842fefd9/b65bf892-a9b9-431e-af85-efaa63e657b0"
-					(reference "#PWR046")
-					(unit 1)
-				)
-			)
-		)
-	)
-	(symbol
 		(lib_name "MountingHole_1")
 		(lib_id "Mechanical:MountingHole")
@@
 		(lib_name "LED_Small_1")
 		(lib_id "Device:LED_Small")
-		(at 25.4 127 90)
+		(at 25.4 127 270)
 		(unit 1)
 		(exclude_from_sim no)
@@
 		(dnp no)
 		(property "Reference" "D45"
-			(at 27.94 125.6664 90)
+			(at 22.86 128.3336 90)
 			(effects
 				(font
@@
 		)
 		(property "Value" "LED_Blue"
-			(at 27.178 127.508 0)
+			(at 23.622 126.492 0)
 			(effects
 				(font
@@
 		(lib_name "LED_Small_1")
 		(lib_id "Device:LED_Small")
-		(at 35.56 127 90)
+		(at 35.56 127 270)
 		(unit 1)
 		(exclude_from_sim no)
@@
 		(dnp no)
 		(property "Reference" "D46"
-			(at 38.1 125.6664 90)
+			(at 33.02 128.3336 90)
 			(effects
 				(font
@@
 		)
 		(property "Value" "LED_Green"
-			(at 37.338 126.238 0)
-			(effects
-				(font
+			(at 39.37 130.302 0)
+			(effects
+				(font

Commit message: changed npm1100 to npm1300 and got rid of some footprints
Connections:
- net 3VOUT is gone; now on net 3.3V: J3.1 (Pin_1), U1.26 (VCC_NRF)
- no-connect marks 28 -> 27
Other:
- sheet Power ports: added VBUSOut; removed 3.0V, FUEL_ALRT, VBUS

Commit message: Adds trackpoint reset GPIO Fix floating led 15 and 35 (mirrored)
Other:
- moved on the sheet: D45, D46, R15, R16

Commit message: Pipar Point V3.1
Parts:
- J3: footprint Connector_PinHeader_2.00mm:PinHeader_2x03_P2.00mm_Vertical -> Keyboard:PinHeader_2x03_P2.00mm_Vertical_DEBUG
Other:
- sheet Power ports: added BAT_IN, BAT_ON; removed none
Changed lines of the file:
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@@
 		(title "Pipar Point")
 		(date "2025-08-29")
-		(rev "V3")
+		(rev "V3.1")
 		(company "Pipar Keyboards")
 	)
@@
 	)
 	(junction
-		(at 66.04 29.21)
-		(diameter 0)
-		(color 0 0 0 0)
-	)
-	(junction
 		(at 208.28 138.43)
 		(diameter 0)
@@
 	)
 	(junction
+		(at 66.04 26.67)
+		(diameter 0)
+		(color 0 0 0 0)
+	)
+	(junction
 		(at 205.74 138.43)
 		(diameter 0)
@@
 	(wire
 		(pts
+			(xy 43.18 52.07) (xy 48.26 52.07)
+		)
+		(stroke
+			(width 0)
+			(type default)
+		)
+	)
+	(wire
+		(pts
 			(xy 35.56 138.43) (xy 35.56 140.97)
 		)
@@
 		)
 	)
+	(wire
+		(pts
+			(xy 43.18 49.53) (xy 48.26 49.53)
+		)
+		(stroke
+			(width 0)
+			(type default)
+		)
+	)
 	(polyline
 		(pts
@@
 	)
 	(label "3.3V"
-		(at 54.61 53.34 180)
+		(at 68.58 53.34 180)
 		(effects
 			(font
@@
 	(hierarchical_label "3.3V"
 		(shape bidirectional)
-		(at 54.61 53.34 0)
+		(at 68.58 53.34 0)
 		(effects
 			(font
@@
 		)
 	)
+	(hierarchical_label "BAT_ON"
+		(shape bidirectional)
+		(at 48.26 52.07 0)
+		(effects
+			(font
+				(size 1.27 1.27)
+			)
+			(justify left)
+		)
+	)
+	(hierarchical_label "BAT_IN"
+		(shape bidirectional)
+		(at 48.26 49.53 0)
+		(effects
+			(font
+				(size 1.27 1.27)
+			)
+			(justify left)
+		)
+	)
 	(hierarchical_label "TPRST"
 		(shape bidirectional)
@@
 			)
 		)
-		(property "Footprint" "Connector_PinHeader_2.00mm:PinHeader_2x03_P2.00mm_Vertical"
+		(property "Footprint" "Keyboard:PinHeader_2x03_P2.00mm_Vertical_DEBUG"
 			(at 71.12 26.67 0)
 			(effects
@@
 	(symbol
 		(lib_id "power:GND")
-		(at 66.04 29.21 0)
+		(at 66.04 26.67 270)
 		(unit 1)
 		(exclude_from_sim no)
@@
 		(fields_autoplaced yes)
 		(property "Reference" "#PWR043"
-			(at 66.04 35.56 0)
+			(at 59.69 26.67 0)
 			(effects
 				(font
@@
 		)
 		(property "Value" "GND"
-			(at 66.04 34.29 0)
+			(at 64.77 22.86 90)
 			(effects
 				(font
@@
 		)
 		(property "Footprint" ""
-			(at 66.04 29.21 0)
+			(at 66.04 26.67 0)
 			(effects
 				(font
@@
 		)
 		(property "Datasheet" ""
-			(at 66.04 29.21 0)
+			(at 66.04 26.67 0)
 			(effects
 				(font
@@
 		)
 		(property "Description" "Power symbol creates a global label with name \"GND\" , ground"
-			(at 66.04 29.21 0)
+			(at 66.04 26.67 0)
 			(effects
 				(font
@@
 				)
 				(path "/ae2abdf3-be75-4a01-9d2e-db16842fefd9/b65bf892-a9b9-431e-af85-efaa63e657b0"
-					(reference "#PWR044")
+					(reference "#PWR0102")
 					(unit 1)
 				)
@@
 			(effects
 				(font
+					(size 1.27 1.27)
+				)
+				(justify right)
+			)
+		)
+		(pin "BAT_IN" bidirectional
+			(at 43.18 49.53 0)
+			(effects
+				(font
+					(size 1.27 1.27)
+				)
+				(justify right)
+			)
+		)
+		(pin "BAT_ON" bidirectional
+			(at 43.18 52.07 0)
+			(effects
+				(font

Commit message: do some work for the dongle
Parts:
- renumbered D45 to D1, D46 to D2, H49 to H10, H65 to H11, H54 to H12, H56 to H13, H58 to H14, H60 to H15, H62 to H16, H41 to H6, H43 to H7, H45 to H8, H47 to H9, J3 to J1, R15 to R4, R16 to R5, SW1 to SW3, TP2 to TP1, U1 to U3
Other:
- moved on the sheet: SW3
