File: pcb/pipar_point_v3/power.kicad_sch (KiCad schematic)
At the start: 30 parts, among them IC1 MCP1700T-3302E_MAY, J1 USB_C_Receptacle_USB2.0_16P, SW3 SW_SPDT, U3 MAX17048, U4 ESDR0502NMUTAG, U5 nPM1100-QDXX

Commit message: updates the pinout for the isp1807
Other:
- moved on the sheet: D21, D22
Changed lines of the file:
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@@
 	)
 	(no_connect
-		(at 71.12 73.66)
+		(at 71.12 71.12)
 	)
 	(no_connect
@@
 	)
 	(no_connect
-		(at 71.12 71.12)
+		(at 71.12 73.66)
 	)
 	(no_connect
@@
 	(wire
 		(pts
-			(xy 198.12 85.09) (xy 198.12 121.92)
+			(xy 198.12 86.36) (xy 198.12 121.92)
 		)
 		(stroke
@@
 	(wire
 		(pts
-			(xy 198.12 77.47) (xy 198.12 80.01)
+			(xy 198.12 77.47) (xy 198.12 81.28)
 		)
 		(stroke
@@
 	(wire
 		(pts
-			(xy 208.28 85.09) (xy 208.28 124.46)
+			(xy 208.28 86.36) (xy 208.28 124.46)
 		)
 		(stroke
@@
 	(wire
 		(pts
-			(xy 208.28 77.47) (xy 208.28 80.01)
+			(xy 208.28 77.47) (xy 208.28 81.28)
 		)
 		(stroke
@@
 		(lib_name "LED_Small_1")
 		(lib_id "Device:LED_Small")
-		(at 198.12 82.55 90)
+		(at 198.12 83.82 90)
 		(unit 1)
 		(exclude_from_sim no)
@@
 		(fields_autoplaced yes)
 		(property "Reference" "D21"
-			(at 200.66 81.2164 90)
+			(at 200.66 82.4864 90)
 			(effects
 				(font
@@
 		)
 		(property "Value" "LED_Small"
-			(at 200.66 83.7564 90)
+			(at 200.66 85.0264 90)
 			(effects
 				(font
@@
 		)
 		(property "Footprint" "LED_SMD:LED_0603_1608Metric"
-			(at 198.12 82.55 90)
+			(at 198.12 83.82 90)
 			(effects
 				(font
@@
 		)
 		(property "Datasheet" "~"
-			(at 198.12 82.55 90)
+			(at 198.12 83.82 90)
 			(effects
 				(font
@@
 		)
 		(property "Description" "Light emitting diode, small symbol"
-			(at 198.12 82.55 0)
+			(at 198.12 83.82 0)
 			(effects
 				(font
@@
 		)
 		(property "Sim.Pin" "1=K 2=A"
-			(at 198.12 82.55 0)
+			(at 198.12 83.82 0)
 			(effects
 				(font
@@
 		)
 		(property "Manufacturer_Name" "Inolux"
-			(at 198.12 82.55 90)
+			(at 198.12 83.82 90)
 			(effects
 				(font
@@
 		)
 		(property "Manufacturer_Part_Number" "IN-PIS63BTPR"
-			(at 198.12 82.55 90)
+			(at 198.12 83.82 90)
 			(effects
 				(font
@@
 		)
 		(property "Mouser Part Number" "743-IN-PIS63BTPR"
-			(at 198.12 82.55 90)
+			(at 198.12 83.82 90)
 			(effects
 				(font
@@
 		(lib_name "LED_Small_1")
 		(lib_id "Device:LED_Small")
-		(at 208.28 82.55 90)
+		(at 208.28 83.82 90)
 		(unit 1)
 		(exclude_from_sim no)
@@
 		(fields_autoplaced yes)
 		(property "Reference" "D22"
-			(at 210.82 81.2164 90)
+			(at 210.82 82.4864 90)
 			(effects
 				(font
@@
 		)
 		(property "Value" "LED_Small"
-			(at 210.82 83.7564 90)
+			(at 210.82 85.0264 90)
 			(effects
 				(font
@@
 		)
 		(property "Footprint" "LED_SMD:LED_0603_1608Metric"
-			(at 208.28 82.55 90)
+			(at 208.28 83.82 90)
 			(effects
 				(font
@@
 		)
 		(property "Datasheet" "~"
-			(at 208.28 82.55 90)
+			(at 208.28 83.82 90)
 			(effects
 				(font
@@
 		)
 		(property "Description" "Light emitting diode, small symbol"
-			(at 208.28 82.55 0)
+			(at 208.28 83.82 0)
 			(effects
 				(font
@@
 		)
 		(property "Sim.Pin" "1=K 2=A"
-			(at 208.28 82.55 0)
+			(at 208.28 83.82 0)
 			(effects
 				(font
@@
 		)
 		(property "Manufacturer_Name" "Inolux"
-			(at 208.28 82.55 90)
+			(at 208.28 83.82 90)
 			(effects
 				(font
@@
 		)
 		(property "Manufacturer_Part_Number" "IN-PIS63BTPG"
-			(at 208.28 82.55 90)
+			(at 208.28 83.82 90)
 			(effects
 				(font
@@
 		)
 		(property "Mouser Part Number" "743-IN-PIS63BTPG"
-			(at 208.28 82.55 90)
+			(at 208.28 83.82 90)
 			(effects
 				(font

Commit message: places more components
Parts:
- added R21, R23: 1.5k, Resistor_SMD:R_0603_1608Metric, symbol Device:R_Small
Connections:
- net VSYS: now also R21.2, R23.2; no longer D21.2 (A), D22.2 (A)
- new net: D21.2 (A), R21.1
- new net: D22.2 (A), R23.1
Other:
- moved on the sheet: D21, D22

Commit message: more things :)
Connections:
- net USB_D+: now also U4.2 (NC)
- net USB_D-: now also U4.3 (NC)
- no-connect marks 8 -> 6
Other:
- moved on the sheet: U4
Changed lines of the file:
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@@
 	)
 	(no_connect
-		(at 71.12 71.12)
-	)
-	(no_connect
 		(at 45.72 63.5)
 	)
@@
 	)
 	(no_connect
-		(at 71.12 73.66)
-	)
-	(no_connect
 		(at 217.17 58.42)
 	)
@@
 	(wire
 		(pts
-			(xy 46.99 76.2) (xy 53.34 76.2)
+			(xy 46.99 76.2) (xy 52.07 76.2)
 		)
 		(stroke
@@
 	(wire
 		(pts
-			(xy 72.39 76.2) (xy 71.12 76.2)
-		)
-		(stroke
-			(width 0)
-			(type solid)
-		)
-	)
-	(wire
-		(pts
-			(xy 52.07 71.12) (xy 53.34 71.12)
-		)
-		(stroke
-			(width 0)
-			(type solid)
-		)
-	)
-	(wire
-		(pts
 			(xy 45.72 53.34) (xy 52.07 53.34)
 		)
@@
 	(wire
 		(pts
-			(xy 49.53 73.66) (xy 53.34 73.66)
+			(xy 49.53 73.66) (xy 52.07 73.66)
 		)
 		(stroke
@@
 	(wire
 		(pts
-			(xy 72.39 77.47) (xy 72.39 76.2)
+			(xy 69.85 77.47) (xy 69.85 76.2)
 		)
 		(stroke
@@
 		)
 	)
+	(label "USB_D-"
+		(at 69.85 73.66 0)
+		(effects
+			(font
+				(size 1.27 1.27)
+			)
+			(justify left bottom)
+		)
+	)
 	(label "CC2"
 		(at 54.61 43.18 0)
@@
 		)
 	)
+	(label "USB_D+"
+		(at 69.85 71.12 0)
+		(effects
+			(font
+				(size 1.27 1.27)
+			)
+			(justify left bottom)
+		)
+	)
 	(label "VBAT"
 		(at 25.4 101.6 0)
@@
 	(symbol
 		(lib_id "mikoto:ESDR0502NMUTAG")
-		(at 62.23 73.66 0)
+		(at 60.96 73.66 0)
 		(unit 1)
 		(exclude_from_sim no)
@@
 		(fields_autoplaced yes)
 		(property "Reference" "U4"
-			(at 57.15 79.9804 0)
+			(at 55.88 79.9804 0)
 			(effects
 				(font
@@
 		)
 		(property "Value" "ESDR0502NMUTAG"
-			(at 62.23 66.8805 0)
+			(at 60.96 66.8805 0)
 			(effects
 				(font
@@
 		)
 		(property "Footprint" "Mikoto:UDFN-6_1.2x1.0mm_P0.4mm"
-			(at 62.23 63.5 0)
+			(at 60.96 63.5 0)
 			(effects
 				(font
@@
 		)
 		(property "Datasheet" "http://www.onsemi.cn/pub_link/Collateral/ESDR0502N-D.PDF"
-			(at 62.23 60.96 0)
+			(at 60.96 60.96 0)
 			(effects
 				(font
@@
 		)
 		(property "Description" ""
-			(at 62.23 73.66 0)
+			(at 60.96 73.66 0)
 			(effects
 				(font
@@
 		)
 		(property "Manufacturer Part" "ESDR0502NMUTBG"
-			(at 62.23 73.66 0)
+			(at 60.96 73.66 0)
 			(effects
 				(font
@@
 		)
 		(property "Sim.Device" ""
-			(at 62.23 73.66 0)
+			(at 60.96 73.66 0)
 			(effects
 				(font
@@
 		)
 		(property "Sim.Pins" ""
-			(at 62.23 73.66 0)
+			(at 60.96 73.66 0)
 			(effects
 				(font
@@
 		)
 		(property "LCSC" "C327480"
-			(at 57.15 79.9804 0)
+			(at 55.88 79.9804 0)
 			(effects
 				(font
@@
 	(symbol
 		(lib_id "power:GND")
-		(at 72.39 77.47 0)
+		(at 69.85 77.47 0)
 		(unit 1)
 		(exclude_from_sim no)
@@
 		(fields_autoplaced yes)
 		(property "Reference" "#PWR012"
-			(at 72.39 83.82 0)
+			(at 69.85 83.82 0)
 			(effects
 				(font
@@
 		)
 		(property "Value" "GND"
-			(at 72.39 82.55 0)
+			(at 69.85 82.55 0)
 			(effects
 				(font
@@
 		)
 		(property "Footprint" ""
-			(at 72.39 77.47 0)
+			(at 69.85 77.47 0)
 			(effects
 				(font
@@
 		)
 		(property "Datasheet" ""
-			(at 72.39 77.47 0)
+			(at 69.85 77.47 0)
 			(effects
 				(font
@@
 		)
 		(property "Description" "Power symbol creates a global label with name \"GND\" , ground"
-			(at 72.39 77.47 0)
+			(at 69.85 77.47 0)
 			(effects
 				(font

Commit message: adds a proper battery connector
Parts:
- removed TP6: TestPoint, TestPoint:TestPoint_Pad_1.5x1.5mm, symbol Connector:TestPoint
- removed TP7: TestPoint, TestPoint:TestPoint_Pad_D1.5mm, symbol Connector:TestPoint
- added J5: Conn_01x02, Connector_JST:JST_PH_S2B-PH-SM4-TB_1x02-1MP_P2.00mm_Horizontal, symbol Connector_Generic:Conn_01x02
- D21: Mouser Part Number 743-IN-PIS63BTPR -> 743-IN-S63AT5A
- D22: Mouser Part Number 743-IN-PIS63BTPG -> 743-IN-S63AT5G
- J1: Mouser Part Number (none) -> 179-UJ20CHGSMTP16TR
- U3: Mouser Part Number (none) -> 700-MAX17048G+T10
- U4: Mouser Part Number (none) -> 863-ESDR0502NMUTBG; now left out of the parts list
Connections:
- net GND: now also J5.1 (Pin_1)
- net at SW3.2 (B): now also J5.2 (Pin_2)
Changed lines of the file:
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@@
 	)
 	(junction
-		(at 92.71 45.72)
-		(diameter 0)
-		(color 0 0 0 0)
-	)
-	(junction
 		(at 49.53 48.26)
 		(diameter 0)
@@
 	)
 	(junction
+		(at 90.17 39.37)
+		(diameter 0)
+		(color 0 0 0 0)
+	)
+	(junction
 		(at 203.2 55.88)
 		(diameter 0)
@@
 	(wire
 		(pts
+			(xy 96.52 45.72) (xy 105.41 45.72)
+		)
+		(stroke
+			(width 0)
+			(type default)
+		)
+	)
+	(wire
+		(pts
 			(xy 203.2 55.88) (xy 203.2 77.47)
 		)
@@
 	(wire
 		(pts
-			(xy 104.14 45.72) (xy 105.41 45.72)
-		)
-		(stroke
-			(width 0)
-			(type default)
-		)
-	)
-	(wire
-		(pts
 			(xy 203.2 77.47) (xy 198.12 77.47)
 		)
@@
 	(wire
 		(pts
+			(xy 90.17 39.37) (xy 93.98 39.37)
+		)
+		(stroke
+			(width 0)
+			(type default)
+		)
+	)
+	(wire
+		(pts
 			(xy 45.72 53.34) (xy 52.07 53.34)
 		)
@@
 	(wire
 		(pts
+			(xy 96.52 45.72) (xy 96.52 39.37)
+		)
+		(stroke
+			(width 0)
+			(type default)
+		)
+	)
+	(wire
+		(pts
 			(xy 49.53 30.48) (xy 49.53 35.56)
 		)
@@
 			)
 		)
+		(property "Mouser Part Number" "700-MAX17048G+T10"
+			(at 46.99 105.41 0)
+			(effects
+				(font
+					(size 1.27 1.27)
+				)
+				(hide yes)
+			)
+		)
 		(pin "1"
 		)
@@
 	(symbol
 		(lib_id "power:PWR_FLAG")
-		(at 92.71 45.72 0)
+		(at 90.17 39.37 0)
 		(unit 1)
 		(exclude_from_sim no)
@@
 		(on_board yes)
 		(dnp no)
-		(fields_autoplaced yes)
 		(property "Reference" "#FLG02"
-			(at 92.71 43.815 0)
+			(at 90.17 37.465 0)
 			(effects
 				(font
@@
 		)
 		(property "Value" "PWR_FLAG"
-			(at 86.868 43.942 0)
+			(at 87.376 35.56 0)
 			(effects
 				(font
@@
 		)
 		(property "Footprint" ""
-			(at 92.71 45.72 0)
+			(at 90.17 39.37 0)
 			(effects
 				(font
@@
 		)
 		(property "Datasheet" "~"
-			(at 92.71 45.72 0)
+			(at 90.17 39.37 0)
 			(effects
 				(font
@@
 		)
 		(property "Description" "Special symbol for telling ERC where power comes from"
-			(at 92.71 45.72 0)
+			(at 90.17 39.37 0)
 			(effects
 				(font
@@
 	(symbol
 		(lib_id "power:GND")
-		(at 92.71 45.72 0)
+		(at 90.17 39.37 0)
 		(unit 1)
 		(exclude_from_sim no)
@@
 		(fields_autoplaced yes)
 		(property "Reference" "#PWR014"
-			(at 92.71 52.07 0)
+			(at 90.17 45.72 0)
 			(effects
 				(font
@@
 		)
 		(property "Value" "GND"
-			(at 92.71 50.8 0)
+			(at 90.17 44.45 0)
 			(effects
 				(font
@@
 		)
 		(property "Footprint" ""
-			(at 92.71 45.72 0)
+			(at 90.17 39.37 0)
 			(effects
 				(font
@@
 		)
 		(property "Datasheet" ""
-			(at 92.71 45.72 0)
+			(at 90.17 39.37 0)
 			(effects
 				(font
@@
 		)
 		(property "Description" "Power symbol creates a global label with name \"GND\" , ground"
-			(at 92.71 45.72 0)
+			(at 90.17 39.37 0)
 			(effects
 				(font
@@
 		(unit 1)
 		(exclude_from_sim no)
-		(in_bom yes)
+		(in_bom no)
 		(on_board yes)
 		(dnp no)
@@
 			)
 		)
+		(property "Mouser Part Number" "863-ESDR0502NMUTBG"
+			(at 60.96 73.66 0)
+			(effects
+				(font
+					(size 1.27 1.27)
+				)
+				(hide yes)
+			)
+		)
 		(pin "1"
 		)
@@
 	)
 	(symbol
-		(lib_id "Connector:TestPoint")
-		(at 104.14 45.72 90)
-		(unit 1)
-		(exclude_from_sim no)
-		(in_bom no)
-		(on_board yes)
-		(dnp no)
-		(fields_autoplaced yes)
-		(property "Reference" "TP7"
-			(at 101.346 43.942 90)
-			(effects
-				(font
-					(size 1.27 1.27)
-				)
-			)
-		)
-		(property "Value" "TestPoint"
-			(at 101.092 47.498 90)
-			(effects
-				(font
-					(size 1.27 1.27)
-				)
-			)
-		)
-		(property "Footprint" "TestPoint:TestPoint_Pad_D1.5mm"
-			(at 104.14 40.64 0)
-			(effects
-				(font
-					(size 1.27 1.27)
-				)
-				(hide yes)
-			)
-		)
-		(property "Datasheet" "~"
-			(at 104.14 40.64 0)
-			(effects
-				(font
-					(size 1.27 1.27)
-				)
-				(hide yes)
-			)
-		)
-		(property "Description" "test point"
-			(at 104.14 45.72 0)
-			(effects
-				(font
-					(size 1.27 1.27)
-				)
-				(hide yes)
-			)
-		)
-		(pin "1"
-		)
-		(instances
-			(project "pipar_point_v3"
-				(path "/ae2abdf3-be75-4a01-9d2e-db16842fefd9/a463a46f-5d6b-469c-a0de-58044b881b04/70e08d6b-7700-49a1-a6c2-1f04ae3c26db"
-					(reference "TP7")
-					(unit 1)
-				)
-				(path "/ae2abdf3-be75-4a01-9d2e-db16842fefd9/b65bf892-a9b9-431e-af85-efaa63e657b0/70e08d6b-7700-49a1-a6c2-1f04ae3c26db"
-					(reference "TP13")
-					(unit 1)
-				)
-			)
-		)
-	)
-	(symbol
 		(lib_id "power:GND")
 		(at 179.07 114.3 0)
@@
 			)
 		)
-		(property "Mouser Part Number" "743-IN-PIS63BTPR"
+		(property "Mouser Part Number" "743-IN-S63AT5A"
 			(at 198.12 87.63 90)
 			(effects
@@
 	)
 	(symbol
+		(lib_id "Connector_Generic:Conn_01x02")
+		(at 93.98 34.29 90)
+		(unit 1)
+		(exclude_from_sim no)
+		(in_bom yes)
+		(on_board yes)
+		(dnp no)
+		(fields_autoplaced yes)
+		(property "Reference" "J5"
+			(at 99.06 33.0199 90)
+			(effects
+				(font
+					(size 1.27 1.27)
+				)
+				(justify right)
+			)
+		)
+		(property "Value" "Conn_01x02"
+			(at 99.06 35.5599 90)
+			(effects
+				(font
+					(size 1.27 1.27)
+				)
+				(justify right)
+			)
+		)
+		(property "Footprint" "Connector_JST:JST_PH_S2B-PH-SM4-TB_1x02-1MP_P2.00mm_Horizontal"
+			(at 93.98 34.29 0)
+			(effects
+				(font
+					(size 1.27 1.27)
+				)
+				(hide yes)
+			)
+		)
+		(property "Datasheet" "~"
+			(at 93.98 34.29 0)
+			(effects
+				(font
+					(size 1.27 1.27)
+				)
+				(hide yes)
+			)
+		)
+		(property "Description" "Generic connector, single row, 01x02, script generated (kicad-library-utils/schlib/autogen/connector/)"
+			(at 93.98 34.29 0)
+			(effects
+				(font
+					(size 1.27 1.27)
+				)
+				(hide yes)
+			)
+		)
+		(property "Mouser Part Number" "306-S2BPHSM4TBLFSN"
+			(at 93.98 34.29 90)
+			(effects
+				(font
+					(size 1.27 1.27)
+				)
+				(hide yes)
+			)
+		)
+		(pin "1"
+		)
+		(pin "2"
+		)
+		(instances
+			(project ""
+				(path "/ae2abdf3-be75-4a01-9d2e-db16842fefd9/a463a46f-5d6b-469c-a0de-58044b881b04/70e08d6b-7700-49a1-a6c2-1f04ae3c26db"
+					(reference "J5")
+					(unit 1)
+				)
+				(path "/ae2abdf3-be75-4a01-9d2e-db16842fefd9/b65bf892-a9b9-431e-af85-efaa63e657b0/70e08d6b-7700-49a1-a6c2-1f04ae3c26db"
+					(reference "J6")
+					(unit 1)
+				)
+			)
+		)
+	)
+	(symbol
 		(lib_id "power:GND")
 		(at 69.85 77.47 0)
@@
 			)
 		)
+		(property "Mouser Part Number" "179-UJ20CHGSMTP16TR"
+			(at 30.48 50.8 0)
+			(effects
+				(font
+					(size 1.27 1.27)
+				)
+				(hide yes)
+			)
+		)
 		(pin "A7"
 		)
@@
 			)
 		)
-		(property "Mouser Part Number" "743-IN-PIS63BTPG"
+		(property "Mouser Part Number" "743-IN-S63AT5G"
 			(at 208.28 87.63 90)
 			(effects
@@
 					(unit 1)
 				)
-			)
-		)
-	)
-	(symbol
-		(lib_id "Connector:TestPoint")
-		(at 92.71 45.72 270)
-		(unit 1)
-		(exclude_from_sim no)
-		(in_bom no)
-		(on_board yes)
-		(dnp no)
-		(fields_autoplaced yes)
-		(property "Reference" "TP6"
-			(at 88.138 45.974 90)
-			(effects
-				(font
-					(size 1.27 1.27)
-				)
-				(justify left)
-			)
-		)
-		(property "Value" "TestPoint"
-			(at 82.042 47.752 90)
-			(effects
-				(font
-					(size 1.27 1.27)
-				)
-				(justify left)
-			)
-		)
-		(property "Footprint" "TestPoint:TestPoint_Pad_1.5x1.5mm"
-			(at 92.71 50.8 0)
-			(effects
-				(font
-					(size 1.27 1.27)
-				)
-				(hide yes)
-			)
-		)
-		(property "Datasheet" "~"
-			(at 92.71 50.8 0)
-			(effects
-				(font
-					(size 1.27 1.27)
-				)
-				(hide yes)
-			)
-		)
-		(property "Description" "test point"
-			(at 92.71 45.72 0)
-			(effects
-				(font
-					(size 1.27 1.27)
-				)
-				(hide yes)
-			)
-		)
-		(pin "1"
-		)
-		(instances
-			(project "pipar_point_v3"
-				(path "/ae2abdf3-be75-4a01-9d2e-db16842fefd9/a463a46f-5d6b-469c-a0de-58044b881b04/70e08d6b-7700-49a1-a6c2-1f04ae3c26db"
-					(reference "TP6")
-					(unit 1)
-				)
-				(path "/ae2abdf3-be75-4a01-9d2e-db16842fefd9/b65bf892-a9b9-431e-af85-efaa63e657b0/70e08d6b-7700-49a1-a6c2-1f04ae3c26db"
-					(reference "TP12")
-					(unit 1)
-				)
