File: pcb/pipar_point_v3/power.kicad_sch (KiCad schematic)
At the start: 31 parts, among them IC1 MCP1700T-3302E_MAY, J1 USB_C_Receptacle_USB2.0_16P, J5 Conn_01x02, SW3 SW_SPDT, U3 MAX17048, U4 ESDR0502NMUTAG, U5 nPM1100-QDXX

Commit message: cleaned up traces on right side, updated bom
Parts:
- C1: Manufacturer_Name TDK -> (none); Manufacturer_Part_Number C1608X5R1H103K080AA -> CGA3E2X7R1H103K080AA; Mouser Part Number 810-C1608X5R1H103KAA -> 810-CGA3E2X7R1H103K
- C10, C3, C4, C9: Manufacturer_Name YAGEO -> (none); Manufacturer_Part_Number CC0603KRX7R5BB105 -> CGA3E1X7R1V105K080AC; Mouser Part Number 603-CC603KRX7R5BB105 -> 810-CGA3E1X7R1V105KC
- C2: Manufacturer_Name YAGEO -> (none); Manufacturer_Part_Number CC0603KRX7R5BB105 -> C1608X7R1H104K080AA; Mouser Part Number 603-CC603KRX7R5BB105 -> 810-C1608X7R1H104K
- C5, C6, C7, C8: Manufacturer_Name TDK -> (none)
- D21: value LED_Small -> LED_Error; Manufacturer_Name Inolux -> (none); Manufacturer_Part_Number IN-PIS63BTPR -> IN-S63AT5A
- D22: value LED_Small -> LED_Green; Manufacturer_Name Inolux -> (none); Manufacturer_Part_Number IN-PIS63BTPG -> IN-S63AT5G
- IC1: Manufacturer_Name Microchip -> (none)
- J1: Manufacturer_Part_Number (none) -> UJ20-C-H-G-SMT-P16-TR; Mouser Part Number 179-UJ20CHGSMTP16TR -> 179-UJ20CHGSMTP16TR
- J5: Manufacturer_Part_Number (none) -> S2B-PH-SM4-TB(LF)(SN)
- L1: Manufacturer_Name TDK -> (none); Mouser Part Number 810-MLZ2012A2R2WT000 -> 810-MLZ2012A2R2WT000
- R21, R23, R6: Manufacturer_Name YAGEO -> (none); Mouser Part Number 603-RC0603FR-071K5L -> 603-RC0603FR-071K5L
- R3, R4, R5, R7: Manufacturer_Name YAGEO -> (none); Manufacturer_Part_Number 603-RC0603FR-075K1L -> RC0603FR-075K1L; Mouser Part Number 603-RC0603FR-075K1L -> 603-RC0603FR-075K1L
- SW3: Manufacturer_Name C&K -> (none); Manufacturer_Part_Number PCM12SMTBR -> PCM12SMTBR; Mouser Part Number 611-PCM12SMTBR -> 611-PCM12SMTBR
- U3: Manufacturer_Part_Number (none) -> MAX17048G+T10; Mouser Part Number 700-MAX17048G+T10 -> 700-MAX17048G+T10
- U5: Manufacturer_Name Nordic Semiconductor -> (none); Manufacturer_Part_Number NPM1100-QDAA-R -> nPM1100-QDAA-R
Changed lines of the file:
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@@
 			)
 		)
-		(property "Mouser Part Number" "603-CC603KRX7R5BB105"
+		(property "Mouser Part Number" "810-CGA3E1X7R1V105KC"
 			(at 113.03 52.07 90)
 			(effects
@@
 			)
 		)
-		(property "Manufacturer_Name" "YAGEO"
+		(property "Manufacturer_Name" ""
 			(at 113.03 52.07 90)
 			(effects
@@
 			)
 		)
-		(property "Manufacturer_Part_Number" "CC0603KRX7R5BB105"
+		(property "Manufacturer_Part_Number" "CGA3E1X7R1V105K080AC"
 			(at 113.03 52.07 90)
 			(effects
@@
 			)
 		)
-		(property "Manufacturer_Name" "Microchip"
+		(property "Manufacturer_Name" ""
 			(at 243.84 63.5 0)
 			(effects
@@
 			)
 		)
-		(property "Mouser Part Number" "700-MAX17048G+T10"
+		(property "Mouser Part Number" " 700-MAX17048G+T10"
+			(at 46.99 105.41 0)
+			(effects
+				(font
+					(size 1.27 1.27)
+				)
+				(hide yes)
+			)
+		)
+		(property "Manufacturer_Part_Number" " MAX17048G+T10"
 			(at 46.99 105.41 0)
 			(effects
@@
 			)
 		)
-		(property "Manufacturer_Name" "TDK"
+		(property "Manufacturer_Name" ""
 			(at 161.29 83.82 0)
 			(effects
@@
 			)
 		)
-		(property "Mouser Part Number" "603-CC603KRX7R5BB105"
+		(property "Mouser Part Number" "810-CGA3E1X7R1V105KC"
 			(at 213.36 58.42 0)
 			(effects
@@
 			)
 		)
-		(property "Manufacturer_Name" "YAGEO"
+		(property "Manufacturer_Name" ""
 			(at 213.36 58.42 0)
 			(effects
@@
 			)
 		)
-		(property "Manufacturer_Part_Number" "CC0603KRX7R5BB105"
+		(property "Manufacturer_Part_Number" "CGA3E1X7R1V105K080AC"
 			(at 213.36 58.42 0)
 			(effects
@@
 			)
 		)
-		(property "Manufacturer_Name" "YAGEO"
+		(property "Manufacturer_Name" ""
 			(at 67.31 43.18 90)
 			(effects
@@
 			)
 		)
-		(property "Manufacturer_Part_Number" "603-RC0603FR-075K1L"
+		(property "Manufacturer_Part_Number" "RC0603FR-075K1L"
 			(at 67.31 43.18 90)
 			(effects
@@
 			)
 		)
-		(property "Mouser Part Number" "603-RC0603FR-075K1L "
+		(property "Mouser Part Number" "603-RC0603FR-075K1L"
 			(at 67.31 43.18 90)
 			(effects
@@
 			)
 		)
-		(property "Mouser Part Number" "603-CC603KRX7R5BB105"
+		(property "Mouser Part Number" "810-CGA3E1X7R1V105KC"
 			(at 53.34 30.48 90)
 			(effects
@@
 			)
 		)
-		(property "Manufacturer_Name" "YAGEO"
+		(property "Manufacturer_Name" ""
 			(at 53.34 30.48 90)
 			(effects
@@
 			)
 		)
-		(property "Manufacturer_Part_Number" "CC0603KRX7R5BB105"
+		(property "Manufacturer_Part_Number" "CGA3E1X7R1V105K080AC"
 			(at 53.34 30.48 90)
 			(effects
@@
 			)
 		)
-		(property "Mouser Part Number" "810-C1608X5R1H103KAA"
+		(property "Mouser Part Number" "810-CGA3E2X7R1H103K"
 			(at 22.86 77.47 0)
 			(effects
@@
 			)
 		)
-		(property "Manufacturer_Name" "TDK"
+		(property "Manufacturer_Name" ""
 			(at 22.86 77.47 0)
 			(effects
@@
 			)
 		)
-		(property "Manufacturer_Part_Number" "C1608X5R1H103K080AA"
+		(property "Manufacturer_Part_Number" "CGA3E2X7R1H103K080AA"
 			(at 22.86 77.47 0)
 			(effects
@@
 			)
 		)
-		(property "Manufacturer_Name" "YAGEO"
+		(property "Manufacturer_Name" ""
 			(at 67.31 40.64 90)
 			(effects
@@
 			)
 		)
-		(property "Manufacturer_Part_Number" "603-RC0603FR-075K1L"
+		(property "Manufacturer_Part_Number" "RC0603FR-075K1L"
 			(at 67.31 40.64 90)
 			(effects
@@
 			)
 		)
-		(property "Mouser Part Number" "603-RC0603FR-075K1L "
+		(property "Mouser Part Number" "603-RC0603FR-075K1L"
 			(at 67.31 40.64 90)
 			(effects
@@
 			)
 		)
-		(property "Manufacturer_Name" "C&K"
+		(property "Manufacturer_Name" ""
 			(at 110.49 45.72 90)
 			(effects
@@
 			)
 		)
-		(property "Manufacturer_Part_Number" "PCM12SMTBR"
+		(property "Manufacturer_Part_Number" " PCM12SMTBR"
 			(at 110.49 45.72 90)
 			(effects
@@
 			)
 		)
-		(property "Mouser Part Number" "611-PCM12SMTBR "
+		(property "Mouser Part Number" " 611-PCM12SMTBR"
 			(at 110.49 45.72 90)
 			(effects
@@
 			)
 		)
-		(property "Mouser Part Number" "603-CC603KRX7R5BB105"
+		(property "Mouser Part Number" "810-C1608X7R1H104K"
 			(at 27.94 106.68 0)
 			(effects
@@
 			)
 		)
-		(property "Manufacturer_Name" "YAGEO"
+		(property "Manufacturer_Name" ""
 			(at 27.94 106.68 0)
 			(effects
@@
 			)
 		)
-		(property "Manufacturer_Part_Number" "CC0603KRX7R5BB105"
+		(property "Manufacturer_Part_Number" "C1608X7R1H104K080AA"
 			(at 27.94 106.68 0)
 			(effects
@@
 		(on_board yes)
 		(dnp no)
-		(fields_autoplaced yes)
 		(property "Reference" "D21"
 			(at 200.66 86.2964 90)
@@
 			)
 		)
-		(property "Value" "LED_Small"
-			(at 200.66 88.8364 90)
+		(property "Value" "LED_Error"
+			(at 194.056 89.408 90)
 			(effects
 				(font
@@
 			)
 		)
-		(property "Manufacturer_Name" "Inolux"
+		(property "Manufacturer_Name" ""
 			(at 198.12 87.63 90)
 			(effects
@@
 			)
 		)
-		(property "Manufacturer_Part_Number" "IN-PIS63BTPR"
+		(property "Manufacturer_Part_Number" "IN-S63AT5A"
 			(at 198.12 87.63 90)
 			(effects
@@
 			)
 		)
-		(property "Manufacturer_Name" "YAGEO"
+		(property "Manufacturer_Name" ""
 			(at 208.28 82.55 0)
 			(effects
@@
 			)
 		)
-		(property "Mouser Part Number" "603-RC0603FR-071K5L "
+		(property "Mouser Part Number" " 603-RC0603FR-071K5L"
 			(at 208.28 82.55 0)
 			(effects
@@
 			)
 		)
+		(property "Manufacturer_Part_Number" "S2B-PH-SM4-TB(LF)(SN)"
+			(at 93.98 34.29 90)
+			(effects
+				(font
+					(size 1.27 1.27)
+				)
+				(hide yes)
+			)
+		)
 		(pin "1"
 		)
@@
 			)
 		)
-		(property "Mouser Part Number" "603-CC603KRX7R5BB105"
+		(property "Mouser Part Number" "810-CGA3E1X7R1V105KC"
 			(at 252.73 58.42 0)
 			(effects
@@
 			)
 		)
-		(property "Manufacturer_Name" "YAGEO"
+		(property "Manufacturer_Name" ""
 			(at 252.73 58.42 0)
 			(effects
@@
 			)
 		)
-		(property "Manufacturer_Part_Number" "CC0603KRX7R5BB105"
+		(property "Manufacturer_Part_Number" "CGA3E1X7R1V105K080AC"
 			(at 252.73 58.42 0)
 			(effects
@@
 			)
 		)
-		(property "Mouser Part Number" "179-UJ20CHGSMTP16TR"
+		(property "Mouser Part Number" " 179-UJ20CHGSMTP16TR"
+			(at 30.48 50.8 0)
+			(effects
+				(font
+					(size 1.27 1.27)
+				)
+				(hide yes)
+			)
+		)
+		(property "Manufacturer_Part_Number" "UJ20-C-H-G-SMT-P16-TR"
 			(at 30.48 50.8 0)
 			(effects
@@
 			)
 		)
-		(property "Manufacturer_Name" "Nordic Semiconductor"
+		(property "Manufacturer_Name" ""
 			(at 123.19 83.82 0)
 			(effects
@@
 			)
 		)
-		(property "Manufacturer_Part_Number" "NPM1100-QDAA-R"
+		(property "Manufacturer_Part_Number" "nPM1100-QDAA-R"
 			(at 123.19 83.82 0)
 			(effects
@@
 			)
 		)
-		(property "Manufacturer_Name" "TDK"
+		(property "Manufacturer_Name" ""
 			(at 149.86 81.28 0)
 			(effects
@@
 			)
 		)
-		(property "Mouser Part Number" "810-MLZ2012A2R2WT000 "
+		(property "Mouser Part Number" " 810-MLZ2012A2R2WT000"
 			(at 149.86 81.28 0)
 			(effects
@@
 		(on_board yes)
 		(dnp no)
-		(fields_autoplaced yes)
 		(property "Reference" "D22"
 			(at 210.82 86.2964 90)
@@
 			)
 		)
-		(property "Value" "LED_Small"
-			(at 210.82 88.8364 90)
+		(property "Value" "LED_Green"
+			(at 204.216 89.408 90)
 			(effects
 				(font
@@
 			)
 		)
-		(property "Manufacturer_Name" "Inolux"
+		(property "Manufacturer_Name" ""
 			(at 208.28 87.63 90)
 			(effects
@@
 			)
 		)
-		(property "Manufacturer_Part_Number" "IN-PIS63BTPG"
+		(property "Manufacturer_Part_Number" "IN-S63AT5G"
 			(at 208.28 87.63 90)
 			(effects
@@
 			)
 		)
-		(property "Manufacturer_Name" "TDK"
+		(property "Manufacturer_Name" ""
 			(at 179.07 83.82 0)
 			(effects
@@
 			)
 		)
-		(property "Manufacturer_Name" "YAGEO"
+		(property "Manufacturer_Name" ""
 			(at 91.44 105.41 0)
 			(effects
@@
 			)
 		)
-		(property "Mouser Part Number" "603-RC0603FR-071K5L "
+		(property "Mouser Part Number" " 603-RC0603FR-071K5L"
 			(at 91.44 105.41 0)
 			(effects
@@
 			)
 		)
-		(property "Manufacturer_Name" "TDK"
+		(property "Manufacturer_Name" ""
 			(at 170.18 83.82 0)
 			(effects
@@
 			)
 		)
-		(property "Manufacturer_Name" "YAGEO"
+		(property "Manufacturer_Name" ""
 			(at 88.9 85.09 0)
 			(effects
@@
 			)
 		)
-		(property "Manufacturer_Part_Number" "603-RC0603FR-075K1L"
+		(property "Manufacturer_Part_Number" "RC0603FR-075K1L"
 			(at 88.9 85.09 0)
 			(effects
@@
 			)
 		)
-		(property "Mouser Part Number" "603-RC0603FR-075K1L "
+		(property "Mouser Part Number" "603-RC0603FR-075K1L"
 			(at 88.9 85.09 0)
 			(effects
@@
 			)
 		)
-		(property "Manufacturer_Name" "YAGEO"
+		(property "Manufacturer_Name" ""
 			(at 198.12 82.55 0)
 			(effects
@@
 			)
 		)
-		(property "Mouser Part Number" "603-RC0603FR-071K5L "
+		(property "Mouser Part Number" " 603-RC0603FR-071K5L"
 			(at 198.12 82.55 0)
 			(effects
@@
 			)
 		)
-		(property "Manufacturer_Name" "YAGEO"
+		(property "Manufacturer_Name" ""
 			(at 93.98 81.28 90)
 			(effects
@@
 			)
 		)
-		(property "Manufacturer_Part_Number" "603-RC0603FR-075K1L"
+		(property "Manufacturer_Part_Number" "RC0603FR-075K1L"
 			(at 93.98 81.28 90)
 			(effects
@@
 			)
 		)
-		(property "Mouser Part Number" "603-RC0603FR-075K1L "
+		(property "Mouser Part Number" "603-RC0603FR-075K1L"
 			(at 93.98 81.28 90)
 			(effects
@@
 			)
 		)
-		(property "Manufacturer_Name" "TDK"
+		(property "Manufacturer_Name" ""
 			(at 127 48.26 0)
 			(effects

Commit message: stuff, i dont remember
Parts:
- added U11: nPM1300-QEXX, Package_DFN_QFN:QFN-32-1EP_5x5mm_P0.5mm_EP3.6x3.6mm_ThermalVias, symbol PCM_nordic-lib-kicad-npm:nPM1300-QEXX
Changed lines of the file:
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@@
+	)
+	(symbol
+		(lib_id "PCM_nordic-lib-kicad-npm:nPM1300-QEXX")
+		(at 137.16 243.84 0)
+		(unit 1)
+		(exclude_from_sim no)
+		(in_bom yes)
+		(on_board yes)
+		(dnp no)
+		(fields_autoplaced yes)
+		(property "Reference" "U11"
+			(at 137.16 243.84 0)
+			(do_not_autoplace yes)
+			(effects
+				(font
+					(size 1.27 1.27)
+				)
+			)
+		)
+		(property "Value" "nPM1300-QEXX"
+			(at 137.16 246.38 0)
+			(do_not_autoplace yes)
+			(effects
+				(font
+					(size 1.27 1.27)
+				)
+			)
+		)
+		(property "Footprint" "Package_DFN_QFN:QFN-32-1EP_5x5mm_P0.5mm_EP3.6x3.6mm_ThermalVias"
+			(at 137.16 302.26 0)
+			(effects
+				(font
+					(size 1.27 1.27)
+				)
+				(hide yes)
+			)
+		)
+		(property "Datasheet" "https://docs.nordicsemi.com/bundle/ps_npm1300"
+			(at 137.16 299.72 0)
+			(effects
+				(font
+					(size 1.27 1.27)
+				)
+				(hide yes)
+			)
+		)
+		(property "Description" "PMIC, LED Driver, Battery Charger, QFN-32"
+			(at 137.16 297.18 0)
+			(effects
+				(font
+					(size 1.27 1.27)
+				)
+				(hide yes)
+			)
+		)
+		(pin "2"
+		)
+		(pin "23"
+		)
+		(pin "7"
+		)
+		(pin "14"
+		)
+		(pin "24"
+		)
+		(pin "17"
+		)
+		(pin "32"
+		)
+		(pin "25"
+		)
+		(pin "13"
+		)
+		(pin "26"
+		)
+		(pin "9"
+		)
+		(pin "12"
+		)
+		(pin "20"
+		)
+		(pin "22"
+		)
+		(pin "5"
+		)
+		(pin "8"
+		)
+		(pin "10"
+		)
+		(pin "27"
+		)
+		(pin "33"
+		)
+		(pin "21"
+		)
+		(pin "15"
+		)
+		(pin "29"
+		)
+		(pin "30"
+		)
+		(pin "16"
+		)
+		(pin "4"
+		)
+		(pin "31"
+		)
+		(pin "19"
+		)
+		(pin "11"
+		)
+		(pin "3"
+		)
+		(pin "1"
+		)
+		(pin "18"
+		)
+		(pin "6"
+		)
+		(pin "28"
+		)
+		(instances
+			(project ""
+				(path "/ae2abdf3-be75-4a01-9d2e-db16842fefd9/a463a46f-5d6b-469c-a0de-58044b881b04/70e08d6b-7700-49a1-a6c2-1f04ae3c26db"
+					(reference "U11")
+					(unit 1)
+				)
+				(path "/ae2abdf3-be75-4a01-9d2e-db16842fefd9/b65bf892-a9b9-431e-af85-efaa63e657b0/70e08d6b-7700-49a1-a6c2-1f04ae3c26db"
+					(reference "U12")
+					(unit 1)
+				)
+			)
+		)
 	)
 	(symbol

Commit message: changed npm1100 to npm1300 and got rid of some footprints
Parts:
- removed C10, C4, C9: 1uF, Capacitor_SMD:C_0603_1608Metric, symbol Device:C_Small
- removed C5: 2.2uF, Capacitor_SMD:C_0603_1608Metric, symbol Device:C_Small
- removed C6, C7, C8: 10uF, Capacitor_SMD:C_0603_1608Metric, symbol Device:C_Small
- removed D21: LED_Error, LED_SMD:LED_0603_1608Metric, symbol Device:LED_Small
- removed D22: LED_Green, LED_SMD:LED_0603_1608Metric, symbol Device:LED_Small
- removed IC1: MCP1700T-3302E_MAY, SamacSys_Parts:SON65P200X200X90-7N, symbol SamacSys_Parts:MCP1700T-3302E_MAY
- removed L1: 2.2uH, Inductor_SMD:L_0805_2012Metric, symbol Device:L_Small
- removed R21, R23, R6: 1.5k, Resistor_SMD:R_0603_1608Metric, symbol Device:R_Small
- removed R3, R4, R5, R7: 5.1k, Resistor_SMD:R_0603_1608Metric, symbol Device:R_Small
- removed SW3: SW_SPDT, Button_Switch_SMD:SW_SPDT_PCM12, symbol Switch:SW_SPDT
- removed TP10, TP5, TP8, TP9: TestPoint_Probe, TestPoint:TestPoint_Pad_D1.0mm, symbol Connector:TestPoint_Probe
- removed U3: MAX17048, Package_DFN_QFN:TDFN-8-1EP_2x2mm_P0.5mm_EP0.8x1.2mm, symbol mikoto:MAX17048
- removed U5: nPM1100-QDXX, Package_DFN_QFN:QFN-24-1EP_4x4mm_P0.5mm_EP2.6x2.6mm_ThermalVias, symbol PCM_nordic-lib-kicad-npm:nPM1100-QDXX
- added C21: 1uF, Capacitor_SMD:C_0603_1608Metric, symbol Device:C_Small
- added C23: 2.2uF, Capacitor_SMD:C_0603_1608Metric, symbol Device:C_Small
- added C25: 100nF, Capacitor_SMD:C_0603_1608Metric, symbol Device:C_Small
- added C29, C33, C35: 10uF, Capacitor_SMD:C_0603_1608Metric, symbol Device:C_Small
- added D47: LED_Error, LED_SMD:LED_0603_1608Metric, symbol Device:LED_Small
- added D50: LED_Green, LED_SMD:LED_0603_1608Metric, symbol Device:LED_Small
- added L5: 2.2uH, Inductor_SMD:L_0805_2012Metric, symbol Device:L_Small
- added NT1: NetTie_2, NetTie:NetTie-2_THT_Pad0.3mm, symbol Device:NetTie_2
- added R17, R20: 1.5k, Resistor_SMD:R_0603_1608Metric, symbol Device:R_Small
- added R27, R29: 10k, Resistor_SMD:R_0603_1608Metric, symbol Device:R_Small
- added R8: 500k, Resistor_SMD:R_0603_1608Metric, symbol Device:R_Small
- added SW5: SW_SPDT, Button_Switch_SMD:SW_SPDT_PCM12, symbol Switch:SW_SPDT
- added TP1: TestPoint_Probe, TestPoint:TestPoint_Pad_D1.0mm, symbol Connector:TestPoint_Probe
- C2: value 0.1uF -> 1uF; Manufacturer_Part_Number C1608X7R1H104K080AA -> LMK107B7105KA-T; Mouser Part Number 810-C1608X7R1H104K -> 963-LMK107B7105KA-T
- C3: Manufacturer_Part_Number CGA3E1X7R1V105K080AC -> LMK107B7105KA-T; Mouser Part Number 810-CGA3E1X7R1V105KC -> 963-LMK107B7105KA-T
Connections:
- net 3.3V: now also U11.12 (VDDIO), U11.32 (VOUT2), C25.2, C29.2, L5.1, R27.1, R29.1
- net BAT_I2C_SCL: now also U11.14 (SCL), R29.2
- net BAT_I2C_SDA: now also U11.13 (SDA), R27.2
- net CC1: now also U11.23 (CC1)
- net CC2: now also U11.24 (CC2)
- net GND: now also C2.2, U11.17 (VSET1), U11.18 (NTC), U11.2 (PVSS1), U11.28 (LSIN1/VINLDO1), U11.29 (LSOUT1/VOUTLDO1), U11.30 (LSIN2/VINLDO2), U11.31 (LSOUT2/VOUTLDO2), U11.33 (AVSS), C21.2, C23.2, C25.1, C35.1, NT1.2, R8.2; no longer C2.1
- net VBAT: now also U11.19 (VBAT), C23.1, SW5.3 (C); no longer C2.2
- net VBUS: now also U11.21 (VBUS), C21.1
- net VSYS: now also U11.1 (VOUT1), U11.20 (VSYS), U11.4 (PVDD), C33.2, C35.2, R17.2, R20.2
- net at U11.16 (VSET2): now also R8.1
- net VBUSOut: now reaches U11.22 (VBUSOUT)
- net VBUSOut: now also C2.1, TP1.1
- net at U11.25 (LED0): now also D47.1 (K)
- net at U11.26 (LED1): now also D50.1 (K)
- net at U11.5 (SW2): now also L5.2
- net PVSS2: now reaches U11.6 (PVSS2)
- net PVSS2: now also C29.1, C33.1, NT1.1
- net at J5.2 (Pin_2): now also SW5.2 (B)
- new net: D50.2 (A), R20.1
- new net: D47.2 (A), R17.1
- no-connect marks 6 -> 11
Other:
- note added: "VIA to GND"
- note removed: "Battery Fuel Gauge"
- note removed: "note: use internal pullups for these"
- moved on the sheet: U11
