File: pcb/pipar_point_v3/power.kicad_sch (KiCad schematic)
At the start: 24 parts, among them J1 USB_C_Receptacle_USB2.0_16P, J5 Conn_01x02, SW5 SW_SPDT, U11 nPM1300-QEXX, U4 ESDR0502NMUTAG

Commit message: Update pipar_point_v3.zip with latest production files
Parts:
- U11: Manufacturer_Part_Number (none) -> nPM1300-QEAA-R7; Mouser Part Number (none) -> 949-NPM1300-QEAA-R7
Changed lines of the file:
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@@
+			)
+		)
+		(property "Manufacturer_Part_Number" "nPM1300-QEAA-R7"
+			(at 168.91 77.47 0)
+			(effects
+				(font
+					(size 1.27 1.27)
+				)
+				(hide yes)
+			)
+		)
+		(property "Mouser Part Number" "949-NPM1300-QEAA-R7"
+			(at 168.91 77.47 0)
+			(effects
+				(font
+					(size 1.27 1.27)
+				)
+				(hide yes)
 			)
 		)

Commit message: Pipar Point V3.1
Parts:
- removed J5: Conn_01x02, Connector_JST:JST_PH_S2B-PH-SM4-TB_1x02-1MP_P2.00mm_Horizontal, symbol Connector_Generic:Conn_01x02
- removed SW5: SW_SPDT, Button_Switch_SMD:SW_SPDT_PCM12, symbol Switch:SW_SPDT
- added J5: Conn_JST_PH_S2B-PH-SM4-TB_1x02-1MP_P2.00mm_Horizo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, Connector_JST:JST_PH_S2B-PH-SM4-TB_1x02-1MP_P2.00mm_Horizontal, symbol Keyboard:Conn_JST_PH_S2B-PH-SM4-TB_1x02-1MP_P2.00mm_Horizontal
Connections:
- net GND: now also J5.1 (Pin_1), J5.MP
- net VBAT renamed BAT_IN
- new net BAT_ON: J5.2 (Pin_2)
- no-connect marks 11 -> 10

Commit message: do some work for the dongle
Parts:
- renumbered C33 to C10, C35 to C11, C2 to C12, C23 to C13, C29 to C14, C1 to C6, C3 to C7, C21 to C8, C25 to C9, D47 to D25, D50 to D26, J1 to J3, J5 to J4, L5 to L1, R27 to R29, R29 to R30, R17 to R31, R20 to R32, R8 to R33, TP1 to TP3, U4 to U5, U11 to U6

Commit message: feat: add dongle fix: move footprint folders around generates new production files mentions pcbway as the v3 sponsor on silkscreen
Parts:
- J4: Manufacturer_Part_Number (none) -> S2B-PH-SM4-TB(LF)(SN); Mouser Part Number (none) -> 306-S2BPHSM4TBLFSN
Connections:
- net VSYS renamed VSYSOut
Changed lines of the file:
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@@
+	)
+	(junction
+		(at 198.12 31.75)
+		(diameter 0)
+		(color 0 0 0 0)
 	)
 	(junction
@@
 	(wire
 		(pts
+			(xy 198.12 31.75) (xy 217.17 31.75)
+		)
+		(stroke
+			(width 0)
+			(type default)
+		)
+	)
+	(wire
+		(pts
 			(xy 168.91 36.83) (xy 171.45 36.83)
 		)
@@
 		(shape output)
 		(at 217.17 44.45 0)
+		(effects
+			(font
+				(size 1.27 1.27)
+			)
+			(justify left)
+		)
+	)
+	(hierarchical_label "VSYSOut"
+		(shape output)
+		(at 217.17 31.75 0)
 		(effects
 			(font
@@
 			(effects
 				(font
+					(size 1.27 1.27)
+				)
+				(hide yes)
+			)
+		)
+		(property "Manufacturer_Part_Number" "S2B-PH-SM4-TB(LF)(SN)"
+			(at 238.76 115.57 90)
+			(effects
+				(font
+					(size 1.27 1.27)
+				)
+				(hide yes)
+			)
+		)
+		(property "Mouser Part Number" "306-S2BPHSM4TBLFSN"
+			(at 238.76 115.57 90)
+			(effects
+				(font

Commit message: pcb: update manufacturer and Mouser part numbers in schematics
Replace IRLML6344TRPBF (942-IRLML6344TRPBF) with SI2342DS-T1-GE3 (78-SI2342DS-T1-GE3) in keymatrix.kicad_sch.
Correct GRM188R61E106KA73J -> GRM188R61E106KA73D and update corresponding Mouser codes (…KA3J -> …KA3D) in power.kicad_sch.
Parts:
- C10, C11, C14: Manufacturer_Part_Number GRM188R61E106KA73J -> GRM188R61E106KA73D; Mouser Part Number 81-GRM188R61E106KA3J -> 81-GRM188R61E106KA3D
Changed lines of the file:
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@@
 			)
 		)
-		(property "Mouser Part Number" "81-GRM188R61E106KA3J"
+		(property "Mouser Part Number" "81-GRM188R61E106KA3D"
 			(at 198.12 34.29 0)
 			(effects
@@
 			)
 		)
-		(property "Manufacturer_Part_Number" "GRM188R61E106KA73J"
+		(property "Manufacturer_Part_Number" "GRM188R61E106KA73D"
 			(at 198.12 34.29 0)
 			(effects
@@
 			)
 		)
-		(property "Mouser Part Number" "81-GRM188R61E106KA3J"
+		(property "Mouser Part Number" "81-GRM188R61E106KA3D"
 			(at 189.23 34.29 0)
 			(effects
@@
 			)
 		)
-		(property "Manufacturer_Part_Number" "GRM188R61E106KA73J"
+		(property "Manufacturer_Part_Number" "GRM188R61E106KA73D"
 			(at 189.23 34.29 0)
 			(effects
@@
 			)
 		)
-		(property "Mouser Part Number" "81-GRM188R61E106KA3J"
+		(property "Mouser Part Number" "81-GRM188R61E106KA3D"
 			(at 215.9 74.93 0)
 			(effects
@@
 			)
 		)
-		(property "Manufacturer_Part_Number" "GRM188R61E106KA73J"
+		(property "Manufacturer_Part_Number" "GRM188R61E106KA73D"
 			(at 215.9 74.93 0)
 			(effects
