File: pcb/pipar_point_v3/pipar_point_v3.kicad_sch (KiCad schematic)
At the start: 3 parts

Commit message: Right hand side keys
Other:
- added sheet Side-RightDup (side.kicad_sch)
- sheet Side-Right: file side.kicad_sch -> side-right.kicad_sch
Changed lines of the file:
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@@
 			(color 0 0 0 0.0000)
 		)
-		(property "Sheetname" "Side-Right"
+		(property "Sheetname" "Side-RightDup"
 			(at 179.07 24.6884 0)
 			(effects
@@
 				)
 			)
+		)
+	)
+	(sheet
+		(at 116.84 25.4)
+		(size 58.42 101.6)
+		(exclude_from_sim no)
+		(in_bom yes)
+		(on_board yes)
+		(dnp no)
+		(fields_autoplaced yes)
+		(stroke
+			(width 0.1524)
+			(type solid)
+		)
+		(fill
+			(color 0 0 0 0.0000)
+		)
+		(property "Sheetname" "Side-Right"
+			(at 116.84 24.6884 0)
+			(effects
+				(font
+					(size 1.27 1.27)
+				)
+				(justify left bottom)
+			)
+		)
+		(property "Sheetfile" "side-right.kicad_sch"
+			(at 116.84 127.5846 0)
+			(effects
+				(font
+					(size 1.27 1.27)
+				)
+				(justify left top)
+			)
+		)
+		(instances
+			(project "pipar_point_v3"
+				(path "/ae2abdf3-be75-4a01-9d2e-db16842fefd9"
+					(page "8")
+				)
+			)

Commit message: Refactor schematic connections and add hierarchical labels
- Removed redundant no_connect entries and updated UUIDs for clarity.
- Added new no_connect entries at specified coordinates.
- Introduced hierarchical labels for "3.3V", "TPClock", "TPData", and "TPRST" with appropriate formatting and positioning.
Parts:
- added U10: ~, Trackpoint:SK8707-01-0C Sensor, symbol Keyboard:SK8707-01-0C_Sensor
- added U9: ~, Trackpoint:SK8707-01, symbol Keyboard:SK8707-01
Connections:
- new net: U10.1D, U9.1D
- new net: U10.2D, U9.2D
- new net: U10.3D, U9.3D
- new net: U10.4D, U9.4D
- new net GND: U9.1A (GND), U9.7C (GND)
- new net Side-Right/3.3V: U9.5A (VCC)
- new net Side-Right/TPClock: U9.3A (IPD_CLK)
- new net Side-Right/TPData: U9.2A (IPD_DATA)
- no-connect marks 0 -> 10
Other:
- removed sheet Side-RightDup
- sheet Side-Left ports: added 3.3V, TPClock, TPData, TPRST; removed none
- sheet Side-Right: file side-right.kicad_sch -> side.kicad_sch
- sheet Side-Right ports: added 3.3V, TPClock, TPData, TPRST; removed none

Commit message: Pipar Point PCB done, maybe
Parts:
- added FID4: Fiducial, Fiducial:Fiducial_0.5mm_Mask1mm, symbol Mechanical:Fiducial
- added H51, H52, H53: PanelMountingHole, MountingHole:MountingHole_3mm, symbol Mechanical:MountingHole
- added H64, H66: Art, Art:Salt, symbol Mechanical:MountingHole

Commit message: adds a proper battery connector
Parts:
- U10, U9: now left out of the parts list
Changed lines of the file:
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@@
 		(unit 1)
 		(exclude_from_sim no)
-		(in_bom yes)
+		(in_bom no)
 		(on_board yes)
 		(dnp no)
@@
 		(unit 1)
 		(exclude_from_sim no)
-		(in_bom yes)
+		(in_bom no)
 		(on_board yes)
 		(dnp no)

Commit message: Adds trackpoint reset GPIO Fix floating led 15 and 35 (mirrored)
Parts:
- added C4: 100nF, Capacitor_SMD:C_0603_1608Metric, symbol Device:C_Small
- added R3, R4, R5: 10k, Resistor_SMD:R_0603_1608Metric, symbol Device:R_Small
Connections:
- net GND: now also R5.2
- net Side-Right/3.3V: now also C4.2, R3.2, R4.2
- net Side-Right/TPClock: now also R4.1
- net Side-Right/TPData: now also R3.1
- net Side-Right/TPRST: now also U9.4A (IPD_RST), C4.1, R5.1
- no-connect marks 10 -> 8
Other:
- moved on the sheet: U10, U9

Commit message: Pipar Point V3.1
Parts:
- added C5, C6, C7, C8: 100nF, Capacitor_SMD:C_0603_1608Metric, symbol Device:C_Small
- added SW3, SW5: SW_SPDT, Button_Switch_SMD:SW_SPDT_PCM12, symbol Switch:SW_SPDT
Connections:
- net GND: now also C4.1, C5.1, C6.1, C7.1, C8.1
- net Side-Right/3.3V: no longer C4.2
- net Side-Right/TPRST: now also C4.2; no longer C4.1
- net at U10.1D, U9.1D: now also C6.2
- net at U10.2D, U9.2D: now also C5.2
- net at U10.3D, U9.3D: now also C7.2
- net at U10.4D, U9.4D: now also C8.2
- new net Side-Left/BAT_IN: SW5.3 (C)
- new net Side-Left/BAT_ON: SW5.2 (B)
- new net Side-Right/BAT_IN: SW3.1 (A)
- new net Side-Right/BAT_ON: SW3.2 (B)
- no-connect marks 8 -> 10
Other:
- sheet Side-Left ports: added BAT_IN, BAT_ON; removed none
- sheet Side-Right ports: added BAT_IN, BAT_ON; removed none
- moved on the sheet: C4, U10

Commit message: do some work for the dongle
Parts:
- renumbered C8 to C1, C7 to C2, C5 to C3, C6 to C4, C4 to C5, H51 to H1, H52 to H2, H53 to H3, H64 to H4, H66 to H5, R5 to R1, R4 to R2, SW5 to SW1, SW3 to SW2, U10 to U1, U9 to U2
Other:
- added sheet Dongle (dongle.kicad_sch)
- moved on the sheet: C1, C2, C3, C4, C5, FID1, FID2, FID3, FID4, H1, H2, H3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
