File: pcb/pipar_point_v3/pipar_point_v3.kicad_sch (KiCad schematic)
At the start: 21 parts, among them SW1 SW_SPDT, SW2 SW_SPDT

Commit message: feat: add dongle fix: move footprint folders around generates new production files mentions pcbway as the v3 sponsor on silkscreen
Other:
- sheet Dongle ports: added BAT_IN, BAT_ON; removed none
Changed lines of the file:
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@@
 	(wire
 		(pts
+			(xy 124.46 101.6) (xy 124.46 105.41)
+		)
+		(stroke
+			(width 0)
+			(type default)
+		)
+	)
+	(wire
+		(pts
 			(xy 217.17 138.43) (xy 222.25 138.43)
 		)
@@
 	(wire
 		(pts
+			(xy 124.46 105.41) (xy 134.62 105.41)
+		)
+		(stroke
+			(width 0)
+			(type default)
+		)
+	)
+	(wire
+		(pts
 			(xy 256.54 119.38) (xy 257.81 119.38)
 		)
@@
 	(wire
 		(pts
+			(xy 134.62 101.6) (xy 134.62 105.41)
+		)
+		(stroke
+			(width 0)
+			(type default)
+		)
+	)
+	(wire
+		(pts
 			(xy 217.17 140.97) (xy 218.44 140.97)
 		)
@@
 			)
 		)
+		(pin "BAT_IN" bidirectional
+			(at 124.46 101.6 270)
+			(effects
+				(font
+					(size 1.27 1.27)
+				)
+				(justify left)
+			)
+		)
+		(pin "BAT_ON" bidirectional
+			(at 134.62 101.6 270)
+			(effects
+				(font
+					(size 1.27 1.27)
+				)
+				(justify left)
+			)
+		)
