File: pcb/pipar_point_v3/dongle.kicad_sch (KiCad schematic)
At the start: 15 parts, among them J7 Conn_02x03_Odd_Even, SW5 EVP-BB1AAB000, U9 ISP1807-LR-RS

Commit message: feat: add dongle fix: move footprint folders around generates new production files mentions pcbway as the v3 sponsor on silkscreen
Parts:
- added J10, J11: Conn_01x10_Pin, Connector_PinHeader_2.54mm:PinHeader_1x10_P2.54mm_Vertical, symbol Connector:Conn_01x10_Pin
- H52: footprint Art:Salt-smallest -> Art:Salt-8x8
Connections:
- net 3.3V: now also J11.9 (Pin_9)
- net BAT_SCL: now also U9.32 (P0_08), J10.9 (Pin_9); no longer U9.34 (P0_06)
- net BAT_SDA: now also U9.34 (P0_06), J10.10 (Pin_10); no longer U9.32 (P0_08)
- net Backlight: now also J11.8 (Pin_8)
- net Col0: now also J10.2 (Pin_2)
- net Col1: now also J10.3 (Pin_3)
- net Col2: now also J10.4 (Pin_4)
- net Col3: now also J10.5 (Pin_5)
- net Col4: now also J10.6 (Pin_6)
- net Col5: now also J10.7 (Pin_7)
- net Col6: now also J10.8 (Pin_8)
- net GND: now also J10.1 (Pin_1), J11.1 (Pin_1)
- net Row0: now also J11.2 (Pin_2)
- net Row1: now also J11.3 (Pin_3)
- net Row2: now also J11.4 (Pin_4)
- net TPClock: now also J11.7 (Pin_7)
- net TPData: now also J11.6 (Pin_6)
- net TPRST: now also J11.5 (Pin_5)
- new net VSYS: J11.10 (Pin_10)
Other:
- sheet Power ports: added VSYSOut; removed none

Commit message: adds dongle cover part updates production files
Parts:
- added H75, H76: MountingHole, MountingHole:MountingHole_2.2mm_M2, symbol Mechanical:MountingHole
- H53, H74: value MouseBite -> MountingHole; footprint mouse-bite:mouse-bite-3mm-6mm -> MountingHole:MountingHole_2.2mm_M2
