File: pcb/pipar_point_v3/keymatrix.kicad_sch (KiCad schematic)
At the start: 83 parts, among them Q1 AO3400A

Commit message: adds a proper battery connector
Parts:
- D1, D10, D11, D12, D13, D14, D15, D16, D17, D18, D19, D2, D20, D3, D4, D5, D6, D7, D8, D9: Mouser Part Number (none) -> 621-1N4148WT
- KHS1, KHS10, KHS11, KHS12, KHS13, KHS14, KHS15, KHS16, KHS17, KHS18, KHS19, KHS2, KHS20, KHS3, KHS4, KHS5, KHS6, KHS7, KHS8, KHS9: now left out of the parts list
- LED1, LED10, LED11, LED12, LED13, LED14, LED15, LED16, LED17, LED18, LED19, LED2, LED20, LED3, LED4, LED5, LED6, LED7, LED8, LED9: Mouser Part Number (none) -> 743-IN-S63AT5UW

Commit message: cleaned up traces on right side, updated bom
Parts:
- D1, D10, D11, D12, D13, D14, D15, D16, D17, D18, D19, D2, D20, D3, D4, D5, D6, D7, D8, D9: Manufacturer_Part_Number (none) -> 1N4148WT-7
- LED1, LED10, LED11, LED12, LED13, LED14, LED15, LED16, LED17, LED18, LED19, LED2, LED20, LED3, LED4, LED5, LED6, LED7, LED8, LED9: Manufacturer_Part_Number (none) -> IN-S63AT5UW
- Q1: Manufacturer_Name Infineon Technologies -> (none); Manufacturer_Part_Number IRLML6344TRPBF -> IRLML6344TRPBF; Mouser Part Number 942-IRLML6344TRPBF -> 942-IRLML6344TRPBF
- R1: Manufacturer_Name YAGEO -> (none); Manufacturer_Part_Number 603-RC0603FR-075K1L -> RC0603FR-075K1L; Mouser Part Number 603-RC0603FR-075K1L -> 603-RC0603FR-075K1L
- R2: Manufacturer_Name YAGEO -> (none); Mouser Part Number 603-RC0603FR-071K5L -> 603-RC0603FR-071K5L

Commit message: Adds trackpoint reset GPIO Fix floating led 15 and 35 (mirrored)
Connections:
- net LEDOut: now also LED15.1 (K)
Changed lines of the file:
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@@
 	(wire
 		(pts
-			(xy 166.37 125.73) (xy 166.37 129.54)
+			(xy 166.37 120.65) (xy 166.37 129.54)
 		)
 		(stroke

Commit message: Pipar Point V3.1
Parts:
- added R10, R12, R21, R23, R31, R33, R35, R37, R39, R41, R43, R45, R47, R49, R51, R53, R55, R57, R6: 49.9R, Resistor_SMD:R_0603_1608Metric, symbol Device:R_Small
- H1, H10, H11, H12, H13, H14, H15, H16, H17, H18, H19, H2, H20, H3, H4, H5, H6, H7, H8, H9: footprint Keyboard:SwitchHoles_Kailh_Choc_V1V2 -> Keyboard:SwitchHoles_Kailh_Choc_V1
- R2: value 1.5k -> 49.9R; Manufacturer_Part_Number RC0603FR-071K5L -> AC0603FR-0749R9L; Mouser Part Number 603-RC0603FR-071K5L -> 603-AC0603FR-0749R9L
Connections:
- net LEDOut: now also Q1.3 (D); no longer R2.1
- net Vcc: now also R2.2, R10.2, R12.2, R21.2, R23.2, R31.2, R33.2, R35.2, R37.2, R39.2, R41.2, R43.2, R45.2, R47.2, R49.2, R51.2, R53.2, R55.2, R57.2, R6.2; no longer LED1.2 (A), LED10.2 (A), LED11.2 (A), LED12.2 (A), LED13.2 (A), LED14.2 (A), LED15.2 (A), LED16.2 (A), LED17.2 (A), LED18.2 (A), LED19.2 (A), LED2.2 (A), LED20.2 (A), LED3.2 (A), LED4.2 (A), LED5.2 (A), LED6.2 (A), LED7.2 (A), LED8.2 (A), LED9.2 (A)
- new net: LED12.2 (A), R37.1
- new net: LED19.2 (A), R57.1
- new net: LED14.2 (A), R43.1
- new net: LED18.2 (A), R53.1
- new net: LED2.2 (A), R2.1
- new net: LED8.2 (A), R33.1
- new net: LED11.2 (A), R39.1
- new net: LED16.2 (A), R49.1
- new net: LED1.2 (A), R6.1
- new net: LED9.2 (A), R35.1
- new net: LED5.2 (A), R21.1
- new net: LED10.2 (A), R41.1
- new net: LED7.2 (A), R31.1
- new net: LED17.2 (A), R51.1
- new net: LED13.2 (A), R47.1
- new net: LED3.2 (A), R10.1
- new net: LED4.2 (A), R23.1
- new net: LED20.2 (A), R55.1
- new net: LED6.2 (A), R12.1
- new net: LED15.2 (A), R45.1
Other:
- note removed: "100R * N Leds 1.5K is almost 2k"
- moved on the sheet: LED1, LED10, LED11, LED12, LED13, LED14, LED15, LED16, LED17, LED18, LED19, LED2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

Commit message: do some work for the dongle
Parts:
- renumbered D6 to D10, D7 to D11, D8 to D12, D9 to D13, D10 to D14, D11 to D15, D12 to D16, D13 to D17, D14 to D18, D15 to D19, D16 to D20, D17 to D21, D18 to D22, D19 to D23, D20 to D24, D1 to D5, D2 to D6, D3 to D7, D4 to D8, D5 to D9, H1 to H28, H2 to H29, H3 to H30, H4 to H31, H5 to H32, H6 to H33, H7 to H34, H8 to H35, H9 to H36, H10 to H37, H11 to H38, H12 to H39, H13 to H40, H14 to H41, H15 to H42, H16 to H43, H17 to H44, H18 to H45, H19 to H46, H20 to H47, R2 to R10, R10 to R11, R23 to R12, R21 to R13, R12 to R14, R31 to R15, R33 to R16, R35 to R17, R41 to R18, R39 to R19, R37 to R20, R47 to R21, R43 to R22, R45 to R23, R49 to R24, R51 to R25, R53 to R26, R57 to R27, R55 to R28, R1 to R8, R6 to R9

Commit message: pcb: update manufacturer and Mouser part numbers in schematics
Replace IRLML6344TRPBF (942-IRLML6344TRPBF) with SI2342DS-T1-GE3 (78-SI2342DS-T1-GE3) in keymatrix.kicad_sch.
Correct GRM188R61E106KA73J -> GRM188R61E106KA73D and update corresponding Mouser codes (…KA3J -> …KA3D) in power.kicad_sch.
Parts:
- Q1: Manufacturer_Part_Number IRLML6344TRPBF -> SI2342DS-T1-GE3; Mouser Part Number 942-IRLML6344TRPBF -> 78-SI2342DS-T1-GE3
Changed lines of the file:
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@@
 			)
 		)
-		(property "Manufacturer_Part_Number" "IRLML6344TRPBF"
+		(property "Manufacturer_Part_Number" "SI2342DS-T1-GE3"
 			(at 58.42 58.42 90)
 			(effects
@@
 			)
 		)
-		(property "Mouser Part Number" " 942-IRLML6344TRPBF"
+		(property "Mouser Part Number" "78-SI2342DS-T1-GE3"
 			(at 58.42 58.42 90)
 			(effects
