File: pcb/pipar_urchin_unibody/pipar_urchin_unibody.kicad_pcb (KiCad board)
At the start: 2 copper layers, 223.5 x 112.5 mm, 106 parts, among them J1 Conn_02x03_Odd_Even, J2 USB_C_Receptacle_USB2.0_16P, J3 Conn_01x02, J4 Conn_01x04, SW1 EVP-BB1AAB000, SW2 SW_SPDT, U1 ISP1807-LR-RS, U2 ESDR0502NMUTAG, U3 nPM1300-QEXX

Commit message: changed the body to make room for the oled screen
Parts:
- J4: moved to B.Cu
- moved J4 8.25 mm to (141.9, 97.2)
- moved U2 2.92 mm to (138.4, 68.0)
- moved J2 2.92 mm to (138.1, 62.1)
- moved C1 2.92 mm to (134.9, 68.1)
- moved C2 2.92 mm to (144.2, 64.5)
- moved J3 2.92 mm to (148.0, 64.2)
- moved SW2 2.92 mm to (128.3, 61.3)
Routing:
- net /VBAT: track 28.5 -> 32.4 mm
- net /3.3V: track 88.6 -> 91.9 mm
- net /CC2: track 16.1 -> 19.0 mm
- net /USB_D-: track 64.8 -> 67.8 mm
- net /CC1: track 18.3 -> 21.3 mm
- net /VBUS: track 27.2 -> 30.1 mm
- net /USB_D+: track 64.8 -> 67.7 mm
- net /LED_2: track 33.0 -> 34.6 mm
- net /SCL: track 17.5 -> 16.0 mm
- net /SDA: track 17.8 -> 19.3 mm, vias 1 -> 2
- net /LED_1: track 34.4 -> 35.8 mm
- net /SWDCLK: track 27.3 -> 26.7 mm
- net /SWDIO: track 21.9 -> 21.3 mm
- net GND: vias 164 -> 159
Other:
- outline, holes or cut-outs redrawn
- board text added: "SCL"
- board text added: "SDA"

Commit message: Update pipar_urchin_unibody.zip with latest production files
Parts:
- added H1: MountingHole_Pad, MountingHole:MountingHole_2.2mm_M2_DIN965_Pad, F.Cu at (47.9, 98.0)
- added H2: MountingHole_Pad, MountingHole:MountingHole_2.2mm_M2_DIN965_Pad, F.Cu at (53.8, 51.5)
- added H3: MountingHole_Pad, MountingHole:MountingHole_2.2mm_M2_DIN965_Pad, F.Cu at (222.4, 51.5)
- added H4: MountingHole_Pad, MountingHole:MountingHole_2.2mm_M2_DIN965_Pad, F.Cu at (228.3, 98.0)
Routing:
- net /Row2: track 410.2 -> 413.2 mm
Other:
- board text added: "37"

Commit message: moves battery plug down, improves layout
Routing:
- net GND: track 52.6 -> 50.7 mm
Changed lines of the file:
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@@
 		)
 		(pad "2" thru_hole circle
-			(at 1.550001 2.65 15)
+			(at 1.55 2.65 15)
 			(size 2 2)
 			(drill 1)
@@
 		)
 		(pad "1" thru_hole circle
-			(at -1.550001 2.65 345)
+			(at -1.55 2.65 345)
 			(size 2 2)
 			(drill 1)
@@
 		)
 		(pad "2" thru_hole circle
-			(at 1.550001 2.65 15)
+			(at 1.55 2.65 15)
 			(size 2 2)
 			(drill 1)
@@
 		)
 		(pad "1" thru_hole circle
-			(at -1.550001 2.65 345)
+			(at -1.55 2.65 345)
 			(size 2 2)
 			(drill 1)
@@
 		)
 		(pad "2" thru_hole circle
-			(at 1.550001 2.65 15)
+			(at 1.55 2.65 15)
 			(size 2 2)
 			(drill 1)
@@
 		)
 		(pad "1" thru_hole circle
-			(at -1.550001 2.65 345)
+			(at -1.55 2.65 345)
 			(size 2 2)
 			(drill 1)
@@
 		)
 		(pad "1" thru_hole circle
-			(at -1.550001 2.65 345)
+			(at -1.55 2.65 345)
 			(size 2 2)
 			(drill 1)
@@
 		)
 		(pad "2" thru_hole circle
-			(at 1.550001 2.65 15)
+			(at 1.55 2.65 15)
 			(size 2 2)
 			(drill 1)
@@
 		)
 		(pad "1" thru_hole circle
-			(at -1.550001 2.65 345)
+			(at -1.55 2.65 345)
 			(size 2 2)
 			(drill 1)
@@
 		)
 		(pad "2" thru_hole circle
-			(at 1.550001 2.65 15)
+			(at 1.55 2.65 15)
 			(size 2 2)
 			(drill 1)
@@
 		)
 		(pad "2" thru_hole circle
-			(at 1.550001 2.65 15)
+			(at 1.55 2.65 15)
 			(size 2 2)
 			(drill 1)
@@
 		)
 		(pad "1" thru_hole circle
-			(at -1.550001 2.65 345)
+			(at -1.55 2.65 345)
 			(size 2 2)
 			(drill 1)
@@
 		)
 		(pad "1" thru_hole circle
-			(at -1.550001 2.65 345)
+			(at -1.55 2.65 345)
 			(size 2 2)
 			(drill 1)
@@
 		)
 		(pad "1" thru_hole circle
-			(at -1.550001 2.65 345)
+			(at -1.55 2.65 345)
 			(size 2 2)
 			(drill 1)
@@
 		)
 		(pad "2" thru_hole circle
-			(at 1.550001 2.65 15)
+			(at 1.55 2.65 15)
 			(size 2 2)
 			(drill 1)
@@
 		)
 		(pad "2" thru_hole circle
-			(at 1.550001 2.65 15)
+			(at 1.55 2.65 15)
 			(size 2 2)
 			(drill 1)
@@
 		)
 		(pad "1" thru_hole circle
-			(at -1.550001 2.65 345)
+			(at -1.55 2.65 345)
 			(size 2 2)
 			(drill 1)
@@
 		)
 		(pad "2" thru_hole circle
-			(at 1.550001 2.65 15)
+			(at 1.55 2.65 15)
 			(size 2 2)
 			(drill 1)
@@
 		)
 		(pad "1" thru_hole circle
-			(at -1.550001 2.65 345)
+			(at -1.55 2.65 345)
 			(size 2 2)
 			(drill 1)
@@
 		)
 		(pad "2" thru_hole circle
-			(at 1.550001 2.65 15)
+			(at 1.55 2.65 15)
 			(size 2 2)
 			(drill 1)
@@
 		)
 		(pad "1" thru_hole circle
-			(at -1.550001 2.65 345)
+			(at -1.55 2.65 345)
 			(size 2 2)
 			(drill 1)
@@
 		)
 		(pad "1" thru_hole circle
-			(at -1.550001 2.65 345)
+			(at -1.55 2.65 345)
 			(size 2 2)
 			(drill 1)
@@
 		)
 		(pad "2" thru_hole circle
-			(at 1.550001 2.65 15)
+			(at 1.55 2.65 15)
 			(size 2 2)
 			(drill 1)
@@
 		)
 		(pad "2" thru_hole circle
-			(at 1.550001 2.65 15)
+			(at 1.55 2.65 15)
 			(size 2 2)
 			(drill 1)
@@
 		)
 		(pad "2" thru_hole circle
-			(at 1.550001 2.65 15)
+			(at 1.55 2.65 15)
 			(size 2 2)
 			(drill 1)
@@
 		)
 		(pad "1" thru_hole circle
-			(at -1.550001 2.65 345)
+			(at -1.55 2.65 345)
 			(size 2 2)
 			(drill 1)
@@
 		)
 		(pad "2" thru_hole circle
-			(at 1.550001 2.65 15)
+			(at 1.55 2.65 15)
 			(size 2 2)
 			(drill 1)
@@
 		)
 		(pad "1" thru_hole circle
-			(at -1.550001 2.65 345)
+			(at -1.55 2.65 345)
 			(size 2 2)
 			(drill 1)
@@
 		)
 		(pad "1" thru_hole circle
-			(at -1.550001 2.65 345)
+			(at -1.55 2.65 345)
 			(size 2 2)
 			(drill 1)
@@
 		)
 		(pad "2" thru_hole circle
-			(at 1.550001 2.65 15)
+			(at 1.55 2.65 15)
 			(size 2 2)
 			(drill 1)
@@
 	)
 	(segment
+		(start 134.607317 110.816112)
+		(end 134.607316 110.816111)
+		(width 0.2032)
+		(layer "F.Cu")
+		(net 19)
+	)
+	(segment
 		(start 145.111214 63.679477)
 		(end 145.121207 63.669477)
@@
 	)
 	(segment
-		(start 134.607317 110.816112)
-		(end 133.493152 110.816106)
-		(width 0.2032)
-		(layer "F.Cu")
-		(net 19)
-	)
-	(segment
 		(start 141.941116 80.736587)
 		(end 141.951628 80.72608)
@@
 	)
 	(segment
+		(start 134.607316 110.816111)
+		(end 134.607316 110.816107)
+		(width 0.2032)
+		(layer "F.Cu")
+		(net 19)
+	)
+	(segment
 		(start 122.6514 115.677225)
 		(end 122.651399 116.984356)
@@
 	)
 	(segment
-		(start 133.493152 110.816106)
-		(end 133.111397 110.434351)
-		(width 0.2032)
-		(layer "F.Cu")
-		(net 19)
-	)
-	(segment
 		(start 138.001213 68.31948)
 		(end 137.531207 68.789481)
@@
 	)
 	(via
-		(at 133.111397 110.434351)
+		(at 134.607316 110.816107)
 		(size 0.6)
 		(drill 0.3)
@@
 	)
 	(via
-		(at 135.341627 105.386075)
+		(at 135.26 105.33)
 		(size 0.6)
 		(drill 0.3)
@@
 	)
 	(segment
-		(start 135.341625 106.266077)
-		(end 135.341627 105.386075)
-		(width 0.2032)
-		(layer "B.Cu")
-		(net 19)
-	)
-	(segment
-		(start 134.871626 108.21608)
-		(end 135.341625 107.746074)
-		(width 0.2032)
-		(layer "B.Cu")
-		(net 19)
-	)
-	(segment
-		(start 135.341625 107.746074)
-		(end 135.341625 106.266077)
-		(width 0.2032)
+		(start 148.959464 63.497739)
+		(end 148.961216 63.499482)
+		(width 0.4064)
 		(layer "B.Cu")
 		(net 19)
 	)
 	(segment
-		(start 133.111397 110.434351)
-		(end 133.111397 109.976304)
+		(start 134.607316 110.816107)
+		(end 135.26 110.163423)
 		(width 0.2032)
 		(layer "B.Cu")
@@
 	)
 	(segment
-		(start 133.111397 109.976304)
-		(end 134.871626 108.21608)
+		(start 135.26 110.163423)
+		(end 135.26 105.33)
 		(width 0.2032)
 		(layer "B.Cu")
 		(net 19)
-	)
-	(segment
-		(start 148.959464 63.497739)
-		(end 148.961216 63.499482)
-		(width 0.4064)
-		(layer "B.Cu")
-		(net 19)
